Commit message: Add continuous joint parameter to rl dp 5

File: irc_ros_description/urdf/igus_robolink_rl_dp_5.ros2_control.xacro (robot description, xacro)
@@ -74,6 +74,8 @@
     <joint name="joint5">
       <command_interface name="position">
-        <param name="min">{-pi*179/180}</param>
-        <param name="max">{pi*179/180}</param>
+        <xacro:unless value="$(arg continuous_last_joint)">
+          <param name="min">{-pi*179/180}</param>
+          <param name="max">{pi*179/180}</param>
+        </xacro:unless>
       </command_interface>
       <command_interface name="velocity">

File: irc_ros_description/urdf/igus_robolink_rl_dp_5.urdf.xacro (robot description, xacro)
@@ -5,4 +5,6 @@
   <xacro:arg name="use_gripper" default="false" />
   <xacro:arg name="gripper" default="schmalz_ecbpmi" />
+  <!-- Enable continuous rotation on the last joint -->
+  <xacro:arg name="continuous_last_joint" default="true" />
   <xacro:include filename="$(find irc_ros_description)/urdf/igus_robolink_rl_dp_5.xacro" />
   <xacro:include filename="$(find irc_ros_description)/urdf/igus_robolink_rl_dp_5.ros2_control.xacro" />

File: irc_ros_description/urdf/igus_robolink_rl_dp_5.xacro (robot description, xacro)
@@ -1,4 +1,5 @@
 <?xml version="1.0" ?>
-<robot name="igus_robolink_rl_dp_5">
+<robot xmlns:xacro="http://wiki.ros.org/xacro"
+       name="igus_robolink_rl_dp_5" >
   <link name="base_link">
     <visual>
@@ -117,12 +118,22 @@
     </inertial>
   </link>
-  <joint name="joint5" type="revolute">
-    <parent link="link_6"/>
-    <child link="link_7"/>
-    <!-- FIXME The 0.03m offset are most likely caused by the mesh file -->
-    <origin rpy="0.0 0.0 0.0" xyz="0.0 0 0.1785"/>
-    <axis xyz="0 0 1"/>
-    <limit effort="330.0" lower="${-pi*179/180}" upper="${pi*179/180}" velocity="2.16"/>
-  </joint>
+  <xacro:if value="$(arg continuous_last_joint)">
+    <joint name="joint5" type="continuous">
+      <parent link="link_6"/>
+      <child link="link_7"/>
+      <origin rpy="0.0 0.0 0.0" xyz="0.0 0 0.1785"/>
+      <axis xyz="0 0 1"/>
+      <limit effort="330.0" velocity="2.16"/>
+    </joint>
+  </xacro:if>
+  <xacro:unless value="$(arg continuous_last_joint)">
+    <joint name="joint5" type="revolute">
+      <parent link="link_6"/>
+      <child link="link_7"/>
+      <origin rpy="0.0 0.0 0.0" xyz="0.0 0 0.1785"/>
+      <axis xyz="0 0 1"/>
+      <limit effort="330.0" lower="${-pi*179/180}" upper="${pi*179/180}" velocity="2.16"/>
+    </joint>
+  </xacro:unless>
   <link name="link_7">
     <visual>
