Commit message: Adapted ReBeL 6DOF 00 and 01

File: irc_ros_description/urdf/igus_rebel_6dof.urdf.xacro (robot description, xacro)
@@ -6,4 +6,8 @@
   <!-- Gripper selection -->
   <xacro:arg name="gripper" default="ext_dio_gripper" />
+  <!-- Enable continuous rotation on the last joint -->
+  <!-- While the last axis can turn continuously, it is limited here in case a tool with wiring is mounted.
+  If you are certain that no wiring issues can arise you may change this do a continuous joint -->
+  <xacro:arg name="continuous_last_joint" default="true" />
   <!-- TODO -->
   <xacro:arg name="root_link" default="false" />

File: irc_ros_description/urdf/igus_rebel_6dof_00.ros2_control.xacro (robot description, xacro)
@@ -81,8 +81,8 @@
     <joint name="joint6">
       <command_interface name="position">
-        <!-- While the last axis can turn continuously, it is limited here in case a tool with wiring is mounted.
-        If you are certain that no wiring issues can arise you may change this do a continuous joint -->
-        <param name="min">${-pi*179/180}</param>
-        <param name="max">${pi*179/180}</param>
+        <xacro:unless value="$(arg continuous_last_joint)">
+          <param name="min">${-pi*179/180}</param>
+          <param name="max">${pi*179/180}</param>
+        </xacro:unless>
       </command_interface>
       <command_interface name="velocity">

File: irc_ros_description/urdf/igus_rebel_6dof_00.xacro (robot description, xacro)
@@ -144,11 +144,22 @@
     </inertial>
   </link>
-  <joint name="joint6" type="revolute">
-    <parent link="link_7"/>
-    <child link="link_8"/>
-    <origin rpy="0.0 0.0 0.0" xyz="0.0 0 0.1208"/>
-    <axis xyz="0 0 1"/>
-    <limit effort="330.0" lower="${-pi*179/180}" upper="${pi*179/180}" velocity="2.16"/>
-  </joint>
+  <xacro:if value="$(arg continuous_last_joint)">
+  <joint name="joint6" type="continuous">
+      <parent link="link_7"/>
+      <child link="link_8"/>
+      <origin rpy="0.0 0.0 0.0" xyz="0.0 0 0.1208"/>
+      <axis xyz="0 0 1"/>
+      <limit effort="330.0" velocity="2.16"/>
+    </joint>
+  </xacro:if>
+  <xacro:unless value="$(arg continuous_last_joint)">
+    <joint name="joint6" type="revolute">
+      <parent link="link_7"/>
+      <child link="link_8"/>
+      <origin rpy="0.0 0.0 0.0" xyz="0.0 0 0.1208"/>
+      <axis xyz="0 0 1"/>
+      <limit effort="330.0" lower="${-pi*179/180}" upper="${pi*179/180}" velocity="2.16"/>
+    </joint>
+  </xacro:unless>
   <link name="link_8">
     <visual>

File: irc_ros_description/urdf/igus_rebel_6dof_01.ros2_control.xacro (robot description, xacro)
@@ -80,8 +80,8 @@
     <joint name="joint6">
       <command_interface name="position">
-        <!-- While the last axis can turn continuously, it is limited here in case a tool with wiring is mounted.
-        If you are certain that no wiring issues can arise you may change this do a continuous joint -->
-        <param name="min">${-pi*179/180}</param>
-        <param name="max">${pi*179/180}</param>
+        <xacro:unless value="$(arg continuous_last_joint)">
+          <param name="min">${-pi*179/180}</param>
+          <param name="max">${pi*179/180}</param>
+        </xacro:unless>
       </command_interface>
       <command_interface name="velocity">

Commit message: 13 Continuous last joint (#46)
* Add continuous last joint parameter for RL DP 5, ReBeL 4DOF and 6DOF 

* Add missing xacro headers

File: irc_ros_description/urdf/igus_rebel_6dof.urdf.xacro (robot description, xacro)
@@ -6,4 +6,8 @@
   <!-- Gripper selection -->
   <xacro:arg name="gripper" default="ext_dio_gripper" />
+  <!-- Enable continuous rotation on the last join. While the last axis can turn continuously,
+  it is limited here in case a tool with wiring is mounted. If you are certain that no wiring
+  issues can arise you may enable this -->
+  <xacro:arg name="continuous_last_joint" default="false" />
   <!-- TODO -->
   <xacro:arg name="root_link" default="false" />

File: irc_ros_description/urdf/igus_rebel_6dof_00.xacro (robot description, xacro)
@@ -1,4 +1,5 @@
 <?xml version="1.0" ?>
-<robot name="igus_rebel_6dof">
+<robot xmlns:xacro="http://wiki.ros.org/xacro"
+       name="igus_rebel_6dof" >
   <link name="base_link">
     <visual>
@@ -144,11 +145,22 @@
     </inertial>
   </link>
-  <joint name="joint6" type="revolute">
-    <parent link="link_7"/>
-    <child link="link_8"/>
-    <origin rpy="0.0 0.0 0.0" xyz="0.0 0 0.1208"/>
-    <axis xyz="0 0 1"/>
-    <limit effort="330.0" lower="${-pi*179/180}" upper="${pi*179/180}" velocity="2.16"/>
-  </joint>
+  <xacro:if value="$(arg continuous_last_joint)">
+  <joint name="joint6" type="continuous">
+      <parent link="link_7"/>
+      <child link="link_8"/>
+      <origin rpy="0.0 0.0 0.0" xyz="0.0 0 0.1208"/>
+      <axis xyz="0 0 1"/>
+      <limit effort="330.0" velocity="2.16"/>
+    </joint>
+  </xacro:if>
+  <xacro:unless value="$(arg continuous_last_joint)">
+    <joint name="joint6" type="revolute">
+      <parent link="link_7"/>
+      <child link="link_8"/>
+      <origin rpy="0.0 0.0 0.0" xyz="0.0 0 0.1208"/>
+      <axis xyz="0 0 1"/>
+      <limit effort="330.0" lower="${-pi*179/180}" upper="${pi*179/180}" velocity="2.16"/>
+    </joint>
+  </xacro:unless>
   <link name="link_8">
     <visual>

File: irc_ros_description/urdf/igus_rebel_6dof_01.ros2_control.xacro (robot description, xacro)
@@ -1,4 +1,5 @@
 <?xml version="1.0" ?>
-<robot xmlns:xacro="http://www.ros.org/wiki/xacro">
+<robot xmlns:xacro="http://wiki.ros.org/xacro"
+       name="igus_rebel_6dof" >
   <ros2_control name="Rebel" type="system">
     <hardware>
@@ -80,8 +81,8 @@
     <joint name="joint6">
       <command_interface name="position">
-        <!-- While the last axis can turn continuously, it is limited here in case a tool with wiring is mounted.
-        If you are certain that no wiring issues can arise you may change this do a continuous joint -->
-        <param name="min">${-pi*179/180}</param>
-        <param name="max">${pi*179/180}</param>
+        <xacro:unless value="$(arg continuous_last_joint)">
+          <param name="min">${-pi*179/180}</param>
+          <param name="max">${pi*179/180}</param>
+        </xacro:unless>
       </command_interface>
       <command_interface name="velocity">

File: irc_ros_description/urdf/igus_robolink_rl_dp_5.urdf.xacro (robot description, xacro)
@@ -5,4 +5,8 @@
   <xacro:arg name="use_gripper" default="false" />
   <xacro:arg name="gripper" default="schmalz_ecbpmi" />
+  <!-- Enable continuous rotation on the last join. While the last axis can turn continuously,
+  it is limited here in case a tool with wiring is mounted. If you are certain that no wiring
+  issues can arise you may enable this -->
+  <xacro:arg name="continuous_last_joint" default="false" />
   <xacro:include filename="$(find irc_ros_description)/urdf/igus_robolink_rl_dp_5.xacro" />
   <xacro:include filename="$(find irc_ros_description)/urdf/igus_robolink_rl_dp_5.ros2_control.xacro" />
