Commit message: Add prefix to .ros2_control.xacros

File: irc_ros_description/urdf/cpr_platform_medium.ros2_control.xacro (robot description, xacro)
@@ -20,6 +20,6 @@
       </xacro:unless>
     </hardware>
-    <xacro:din_rail_module name="joint_wheel_1" can_id="0x18" gear_scale="33.33" continuous_joint="true" />
-    <xacro:din_rail_module name="joint_wheel_2" can_id="0x28" gear_scale="-33.33" continuous_joint="true" />
+    <xacro:din_rail_module name="${prefix}joint_wheel_1" can_id="0x18" gear_scale="33.33" continuous_joint="true" />
+    <xacro:din_rail_module name="${prefix}joint_wheel_2" can_id="0x28" gear_scale="-33.33" continuous_joint="true" />
   </ros2_control>
 </robot>

File: irc_ros_description/urdf/cpr_platform_medium.urdf.xacro (robot description, xacro)
@@ -7,4 +7,5 @@
   <xacro:arg name="use_cprcanv2" default="false"/>
   <xacro:arg name="use_cri" default="false"/>
+  <xacro:arg name="prefix" default="" />
   <xacro:include filename="$(find irc_ros_description)/urdf/din_rail_module.ros2_control.xacro" />
   <xacro:include filename="$(find irc_ros_description)/urdf/cpr_platform_medium.xacro" />

File: irc_ros_description/urdf/gripper_ext_dio_gripper.ros2_control.xacro (robot description, xacro)
@@ -7,5 +7,5 @@
     <param name="can_socket">can0</param>
   </hardware>
-  <gpio name="dio_ext">
+  <gpio name="${prefix}dio_ext">
     <param name="can_id">0x90</param>
     <command_interface name="digital_output" size="7" data_type="bool" />

File: irc_ros_description/urdf/igus_rebel_4dof.urdf.xacro (robot description, xacro)
@@ -18,4 +18,5 @@
   <!-- TODO -->
   <xacro:arg name="root_link" default="false" />
+  <xacro:arg name="prefix" default="" />
   <xacro:include filename="$(find irc_ros_description)/urdf/igus_rebel_4dof_$(arg rebel_version).xacro" />
   <xacro:include filename="$(find irc_ros_description)/urdf/igus_rebel_4dof_$(arg rebel_version).ros2_control.xacro" />

File: irc_ros_description/urdf/igus_rebel_4dof_00.ros2_control.xacro (robot description, xacro)
@@ -20,15 +20,15 @@
       </xacro:unless>
     </hardware>
-    <xacro:rebel_joint name="joint1" can_id="0x10" position_min="${-pi*179/180}" position_max="${pi*179/180}" gear_scale="-1031.11" />
+    <xacro:rebel_joint name="${prefix}joint1" can_id="0x10" position_min="${-pi*179/180}" position_max="${pi*179/180}" gear_scale="-1031.11" />
     <!-- Position limit difference with iRC files due to 30 degree offset in joint 2 and 3 -->
-    <xacro:rebel_joint name="joint2" can_id="0x20" position_min="${-pi*2/3}" position_max="${pi*2/3}" gear_scale="1031.11" />
-    <xacro:rebel_joint name="joint3" can_id="0x30" position_min="${-pi*2/3}" position_max="${pi*2/3}" gear_scale="1031.11" />
-    <xacro:rebel_joint name="joint4" can_id="0x40" position_min="${-pi*19/36}" position_max="${pi*19/36}" gear_scale="1031.11" continuous_last_joint="$(arg continuous_last_joint)" />
-    <gpio name="dio_base">
+    <xacro:rebel_joint name="${prefix}joint2" can_id="0x20" position_min="${-pi*2/3}" position_max="${pi*2/3}" gear_scale="1031.11" />
+    <xacro:rebel_joint name="${prefix}joint3" can_id="0x30" position_min="${-pi*2/3}" position_max="${pi*2/3}" gear_scale="1031.11" />
+    <xacro:rebel_joint name="${prefix}joint4" can_id="0x40" position_min="${-pi*19/36}" position_max="${pi*19/36}" gear_scale="1031.11" continuous_last_joint="$(arg continuous_last_joint)" />
+    <gpio name="${prefix}dio_base">
       <param name="can_id">0x70</param>
       <command_interface name="digital_output" size="7" data_type="bool" />
       <state_interface name="digital_input" size="7" data_type="bool" />
     </gpio>
-    <gpio name="dio_arm">
+    <gpio name="${prefix}dio_arm">
       <param name="can_id">0x80</param>
       <command_interface name="digital_output" size="2" data_type="bool" />

File: irc_ros_description/urdf/igus_rebel_4dof_01.ros2_control.xacro (robot description, xacro)
@@ -20,14 +20,14 @@
       </xacro:unless>
     </hardware>
-    <xacro:rebel_joint name="joint1" can_id="0x10" position_min="${-pi*179/180}" position_max="${pi*179/180}" gear_scale="-1443.55" />
-    <xacro:rebel_joint name="joint2" can_id="0x20" position_min="${-pi*2/3}" position_max="${pi*2/3}" gear_scale="1443.55" />
-    <xacro:rebel_joint name="joint3" can_id="0x30" position_min="${-pi*2/3}" position_max="${pi*2/3}" gear_scale="1443.55" />
-    <xacro:rebel_joint name="joint4" can_id="0x40" position_min="${-pi*19/36}" position_max="${pi*19/36}" gear_scale="1031.11" continuous_joint="$(arg continuous_last_joint)" />
-    <gpio name="dio_base">
+    <xacro:rebel_joint name="${prefix}joint1" can_id="0x10" position_min="${-pi*179/180}" position_max="${pi*179/180}" gear_scale="-1443.55" />
+    <xacro:rebel_joint name="${prefix}joint2" can_id="0x20" position_min="${-pi*2/3}" position_max="${pi*2/3}" gear_scale="1443.55" />
+    <xacro:rebel_joint name="${prefix}joint3" can_id="0x30" position_min="${-pi*2/3}" position_max="${pi*2/3}" gear_scale="1443.55" />
+    <xacro:rebel_joint name="${prefix}joint4" can_id="0x40" position_min="${-pi*19/36}" position_max="${pi*19/36}" gear_scale="1031.11" continuous_joint="$(arg continuous_last_joint)" />
+    <gpio name="${prefix}dio_base">
       <param name="can_id">0x70</param>
       <command_interface name="digital_output" size="7" data_type="bool" />
       <state_interface name="digital_input" size="7" data_type="bool" />
     </gpio>
-    <gpio name="dio_arm">
+    <gpio name="${prefix}dio_arm">
       <param name="can_id">0x80</param>
       <command_interface name="digital_output" size="2" data_type="bool" />

File: irc_ros_description/urdf/igus_rebel_6dof.urdf.xacro (robot description, xacro)
@@ -18,4 +18,5 @@
   <!-- TODO -->
   <xacro:arg name="root_link" default="false" />
+  <xacro:arg name="prefix" default="" />
   <xacro:include filename="$(find irc_ros_description)/urdf/igus_rebel_6dof_$(arg rebel_version).xacro" />
   <xacro:include filename="$(find irc_ros_description)/urdf/igus_rebel_6dof_$(arg rebel_version).ros2_control.xacro" />

File: irc_ros_description/urdf/igus_rebel_6dof_00.ros2_control.xacro (robot description, xacro)
@@ -20,17 +20,17 @@
       </xacro:unless>
     </hardware>
-    <xacro:rebel_joint name="joint1" can_id="0x10" position_min="${-pi*179/180}" position_max="${pi*179/180}" gear_scale="1031.11" />
+    <xacro:rebel_joint name="${prefix}joint1" can_id="0x10" position_min="${-pi*179/180}" position_max="${pi*179/180}" gear_scale="1031.11" />
     <!-- Position limit difference with iRC files due to 30 degree offset in joint 2 and 3 -->
-    <xacro:rebel_joint name="joint2" can_id="0x20" position_min="${-pi*2/3}" position_max="${pi*2/3}" gear_scale="1031.11" />
-    <xacro:rebel_joint name="joint3" can_id="0x30" position_min="${-pi*2/3}" position_max="${pi*2/3}" gear_scale="1031.11" />
-    <xacro:rebel_joint name="joint4" can_id="0x40" position_min="${-pi*179/180}" position_max="${pi*179/180}" gear_scale="-1031.11" />
-    <xacro:rebel_joint name="joint5" can_id="0x50" position_min="${-pi*19/36}" position_max="${pi*19/36}" gear_scale="1031.11" />
-    <xacro:rebel_joint name="joint6" can_id="0x60" position_min="${-pi*179/180}" position_max="${pi*179/180}" gear_scale="-1031.11" continuous_joint="$(arg continuous_last_joint)" />
-    <gpio name="dio_base">
+    <xacro:rebel_joint name="${prefix}joint2" can_id="0x20" position_min="${-pi*2/3}" position_max="${pi*2/3}" gear_scale="1031.11" />
+    <xacro:rebel_joint name="${prefix}joint3" can_id="0x30" position_min="${-pi*2/3}" position_max="${pi*2/3}" gear_scale="1031.11" />
+    <xacro:rebel_joint name="${prefix}joint4" can_id="0x40" position_min="${-pi*179/180}" position_max="${pi*179/180}" gear_scale="-1031.11" />
+    <xacro:rebel_joint name="${prefix}joint5" can_id="0x50" position_min="${-pi*19/36}" position_max="${pi*19/36}" gear_scale="1031.11" />
+    <xacro:rebel_joint name="${prefix}joint6" can_id="0x60" position_min="${-pi*179/180}" position_max="${pi*179/180}" gear_scale="-1031.11" continuous_joint="$(arg continuous_last_joint)" />
+    <gpio name="${prefix}dio_base">
       <param name="can_id">0x70</param>
       <command_interface name="digital_output" size="7" data_type="bool" />
       <state_interface name="digital_input" size="7" data_type="bool" />
     </gpio>
-    <gpio name="dio_arm">
+    <gpio name="${prefix}dio_arm">
       <param name="can_id">0x80</param>
       <command_interface name="digital_output" size="2" data_type="bool" />

File: irc_ros_description/urdf/igus_rebel_6dof_01.ros2_control.xacro (robot description, xacro)
@@ -20,17 +20,17 @@
       </xacro:unless>
     </hardware>
-    <xacro:rebel_joint name="joint1" can_id="0x10" position_min="${-pi*179/180}" position_max="${pi*179/180}" gear_scale="1443.55" />
+    <xacro:rebel_joint name="${prefix}joint1" can_id="0x10" position_min="${-pi*179/180}" position_max="${pi*179/180}" gear_scale="1443.55" />
     <!-- Position limit difference with iRC files due to 30 degree offset in joint 2 and 3 -->
-    <xacro:rebel_joint name="joint2" can_id="0x20" position_min="${-pi*2/3}" position_max="${pi*2/3}" gear_scale="1443.55" />
-    <xacro:rebel_joint name="joint3" can_id="0x30" position_min="${-pi*2/3}" position_max="${pi*2/3}" gear_scale="1443.55" />
-    <xacro:rebel_joint name="joint4" can_id="0x40" position_min="${-pi*179/180}" position_max="${pi*179/180}" gear_scale="-1443.55" />
-    <xacro:rebel_joint name="joint5" can_id="0x50" position_min="${-pi*19/36}" position_max="${pi*19/36}" gear_scale="1031.11" />
-    <xacro:rebel_joint name="joint6" can_id="0x60" position_min="${-pi*179/180}" position_max="${pi*179/180}" gear_scale="-1031.11" continuous_joint="$(arg continuous_last_joint)" />
-    <gpio name="dio_base">
+    <xacro:rebel_joint name="${prefix}joint2" can_id="0x20" position_min="${-pi*2/3}" position_max="${pi*2/3}" gear_scale="1443.55" />
+    <xacro:rebel_joint name="${prefix}joint3" can_id="0x30" position_min="${-pi*2/3}" position_max="${pi*2/3}" gear_scale="1443.55" />
+    <xacro:rebel_joint name="${prefix}joint4" can_id="0x40" position_min="${-pi*179/180}" position_max="${pi*179/180}" gear_scale="-1443.55" />
+    <xacro:rebel_joint name="${prefix}joint5" can_id="0x50" position_min="${-pi*19/36}" position_max="${pi*19/36}" gear_scale="1031.11" />
+    <xacro:rebel_joint name="${prefix}joint6" can_id="0x60" position_min="${-pi*179/180}" position_max="${pi*179/180}" gear_scale="-1031.11" continuous_joint="$(arg continuous_last_joint)" />
+    <gpio name="${prefix}dio_base">
       <param name="can_id">0x70</param>
       <command_interface name="digital_output" size="7" data_type="bool" />
       <state_interface name="digital_input" size="7" data_type="bool" />
     </gpio>
-    <gpio name="dio_arm">
+    <gpio name="${prefix}dio_arm">
       <param name="can_id">0x80</param>
       <command_interface name="digital_output" size="2" data_type="bool" />

File: irc_ros_description/urdf/igus_rebel_6dof_pre.ros2_control.xacro (robot description, xacro)
@@ -20,10 +20,10 @@
       </xacro:unless>
     </hardware>
-    <xacro:rebel_joint name="joint1" can_id="0x10" position_min="${-pi*179/180}" position_max="${pi*179/180}" gear_scale="1031.11" />
-    <xacro:rebel_joint name="joint2" can_id="0x20" position_min="${-pi*4/9}" position_max="${pi*7/9}" gear_scale="1031.11" />
-    <xacro:rebel_joint name="joint3" can_id="0x30" position_min="${-pi*4/9}" position_max="${pi*7/9}" gear_scale="1031.11" />
-    <xacro:rebel_joint name="joint4" can_id="0x40" position_min="${-pi*179/180}" position_max="${pi*179/180}" gear_scale="-1031.11" />
-    <xacro:rebel_joint name="joint5" can_id="0x50" position_min="${-pi*19/36}" position_max="${pi*19/36}" gear_scale="1031.11" />
-    <xacro:rebel_joint name="joint6" can_id="0x60" position_min="${-pi*179/180}" position_max="${pi*179/180}" gear_scale="-1031.11" continuous_joint="$(arg continuous_last_joint)" />
+    <xacro:rebel_joint name="${prefix}joint1" can_id="0x10" position_min="${-pi*179/180}" position_max="${pi*179/180}" gear_scale="1031.11" />
+    <xacro:rebel_joint name="${prefix}joint2" can_id="0x20" position_min="${-pi*4/9}" position_max="${pi*7/9}" gear_scale="1031.11" />
+    <xacro:rebel_joint name="${prefix}joint3" can_id="0x30" position_min="${-pi*4/9}" position_max="${pi*7/9}" gear_scale="1031.11" />
+    <xacro:rebel_joint name="${prefix}joint4" can_id="0x40" position_min="${-pi*179/180}" position_max="${pi*179/180}" gear_scale="-1031.11" />
+    <xacro:rebel_joint name="${prefix}joint5" can_id="0x50" position_min="${-pi*19/36}" position_max="${pi*19/36}" gear_scale="1031.11" />
+    <xacro:rebel_joint name="${prefix}joint6" can_id="0x60" position_min="${-pi*179/180}" position_max="${pi*179/180}" gear_scale="-1031.11" continuous_joint="$(arg continuous_last_joint)" />
     <!-- Pre version does not have GPIOs -->
   </ros2_control>

File: irc_ros_description/urdf/igus_robolink_rl_dp_5.ros2_control.xacro (robot description, xacro)
@@ -21,9 +21,9 @@
     </hardware>
     <!-- The gear_scale is positive in the iRC files -->
-    <xacro:din_rail_module name="joint1" can_id="0x10" position_min="${-pi*7/9}" position_max="${pi*7/9}" gear_scale="-266.67" referencing_required="true", referencing_priority="5" />
-    <xacro:din_rail_module name="joint2" can_id="0x20" position_min="${-pi*5/18}" position_max="${pi*1/2}" gear_scale="266.67" referencing_required="true", referencing_priority="2" />
-    <xacro:din_rail_module name="joint3" can_id="0x30" position_min="${-pi*41/36}" position_max="${pi*5/36}" gear_scale="277.78" referencing_required="true", referencing_priority="1" />
-    <xacro:din_rail_module name="joint4" can_id="0x40" position_min="${-pi*5/9}" position_max="${pi*5/9}" gear_scale="-266.67" referencing_required="true", referencing_priority="3" />
-    <xacro:din_rail_module name="joint5" can_id="0x50" position_min="${-pi*179/180}" position_max="${pi*179/180}" gear_scale="-155.56" referencing_required="true", referencing_priority="4" continuous_joint="$(arg continuous_last_joint)"/>
+    <xacro:din_rail_module name="${prefix}joint1" can_id="0x10" position_min="${-pi*7/9}" position_max="${pi*7/9}" gear_scale="-266.67" referencing_required="true", referencing_priority="5" />
+    <xacro:din_rail_module name="${prefix}joint2" can_id="0x20" position_min="${-pi*5/18}" position_max="${pi*1/2}" gear_scale="266.67" referencing_required="true", referencing_priority="2" />
+    <xacro:din_rail_module name="${prefix}joint3" can_id="0x30" position_min="${-pi*41/36}" position_max="${pi*5/36}" gear_scale="277.78" referencing_required="true", referencing_priority="1" />
+    <xacro:din_rail_module name="${prefix}joint4" can_id="0x40" position_min="${-pi*5/9}" position_max="${pi*5/9}" gear_scale="-266.67" referencing_required="true", referencing_priority="3" />
+    <xacro:din_rail_module name="${prefix}joint5" can_id="0x50" position_min="${-pi*179/180}" position_max="${pi*179/180}" gear_scale="-155.56" referencing_required="true", referencing_priority="4" continuous_joint="$(arg continuous_last_joint)"/>
   </ros2_control>
 </robot>

File: irc_ros_description/urdf/igus_robolink_rl_dp_5.urdf.xacro (robot description, xacro)
@@ -15,4 +15,5 @@
   issues can arise you may enable this -->
   <xacro:arg name="continuous_last_joint" default="false" />
+  <xacro:arg name="prefix" default="" />
   <xacro:include filename="$(find irc_ros_description)/urdf/igus_robolink_rl_dp_5.xacro" />
   <xacro:include filename="$(find irc_ros_description)/urdf/igus_robolink_rl_dp_5.ros2_control.xacro" />

File: irc_ros_description/urdf/rebel_joint.ros2_control.xacro (robot description, xacro)
@@ -1,5 +1,5 @@
 <?xml version="1.0"?>
 <robot xmlns:xacro="http://www.ros.org/wiki/xacro">
-  <xacro:macro name="rebel_joint" params="name can_id position_min position_max gear_scale continuous_joint=false">
+  <xacro:macro name="rebel_joint" params="name can_id="" position_min=0 position_max=0 gear_scale=1 continuous_joint=false">
     <joint name="${name}">
       <command_interface name="position">
