Commit message: Change chassis to base_link, add prefix to remaining files

File: irc_ros_description/urdf/cpr_platform_medium.xacro (robot description, xacro)
@@ -5,5 +5,5 @@
   <xacro:property name="base_height" value="0.05"/>
   <xacro:property name="wheel_radius" value="0.07308"/>
-  <link name="chassis">
+  <link name="$(arg prefix)base_link">
     <visual>
       <geometry>
@@ -23,7 +23,7 @@
     </inertial>
   </link>
-  <joint name="joint_wheel_1" type="continuous">
-    <parent link="chassis"/>
-    <child link="wheel_1"/>
+  <joint name="$(arg prefix)joint_wheel_1" type="continuous">
+    <parent link="$(arg prefix)base_link"/>
+    <child link="$(arg prefix)wheel_1"/>
     <origin rpy="0.0 0.0 0.0" xyz="0.0 0.25 -0.011"/>
     <!-- <origin rpy="0.0 0.0 0.0" xyz="0.0 0.236425 0.0"/> -->
@@ -31,5 +31,5 @@
     <!-- <limit effort="330.0" lower="-3.12414" upper="3.12414" velocity="2.16"/> -->
   </joint>
-  <link name="wheel_1">
+  <link name="$(arg prefix)wheel_1">
     <visual>
       <geometry>
@@ -47,7 +47,7 @@
     </inertial>
   </link>
-  <joint name="joint_wheel_2" type="continuous">
-    <parent link="chassis"/>
-    <child link="wheel_2"/>
+  <joint name="$(arg prefix)joint_wheel_2" type="continuous">
+    <parent link="$(arg prefix)base_link"/>
+    <child link="$(arg prefix)wheel_2"/>
     <origin rpy="0.0 0.0 0.0" xyz="0.0 -0.25 -0.011"/>
     <!-- <origin rpy="0.0 0.0 0.0" xyz="0.0 -0.236425 0.0"/> -->
@@ -71,18 +71,17 @@
     </inertial>
   </link>
-  <joint name="joint_laser_front" type="fixed">
-    <parent link="chassis"/>
-    <child link="laser_front"/>
+  <joint name="$(arg prefix)joint_laser_front" type="fixed">
+    <parent link="$(arg prefix)base_link"/>
+    <child link="$(arg prefix)laser_front"/>
     <origin rpy="0.0 0.0 0.0" xyz="0.0 0 0"/>
   </joint>
-  <link name="laser_front">
+  <link name="$(arg prefix)laser_front">
   </link>
-  <joint name="joint_lidar_back" type="fixed">
-    <parent link="chassis"/>
+  <joint name="$(arg prefix)joint_lidar_back" type="fixed">
+    <parent link="base_link"/>
     <child link="laser_back"/>
     <origin rpy="0.0 0.0 ${pi}" xyz="-0.54 0 0"/>
-    <!-- <origin rpy="0.0 0.0 ${pi}" xyz="-0.505 0 0"/> -->
   </joint>
-  <link name="laser_back">
+  <link name="$(arg prefix)laser_back">
   </link>
 </robot>

File: irc_ros_description/urdf/gripper_ext_dio_gripper.xacro (robot description, xacro)
@@ -2,5 +2,5 @@
 <robot xmlns:xacro="http://www.ros.org/wiki/xacro"
     name="gripper_ext_dio_gripper">
-  <link name="gripper_mount">
+  <link name="$(arg prefix)gripper_mount">
     <visual>
       <geometry>
@@ -20,10 +20,10 @@
     </inertial>
   </link>
-  <joint name="gripper_mount_joint" type="fixed">
-    <parent link="gripper_mount" />
-    <child link="gripper_base" />
+  <joint name="$(arg prefix)gripper_mount_joint" type="fixed">
+    <parent link="$(arg prefix)gripper_mount" />
+    <child link="$(arg prefix)gripper_base" />
     <origin xyz="0.01 0.0 0.0" rpy="0.0 0.0 0.0" />
   </joint>
-  <link name="gripper_base">
+  <link name="$(arg prefix)gripper_base">
     <visual>
       <geometry>
@@ -43,11 +43,11 @@
     </inertial>
   </link>
-  <joint name="joint99" type="fixed">
-    <parent link="gripper_base"/>
-    <child link="tcp"/>
+  <joint name="$(arg prefix)joint99" type="fixed">
+    <parent link="$(arg prefix)gripper_base"/>
+    <child link="$(arg prefix)tcp"/>
     <origin rpy="0.0 0.0 0.0" xyz="0.07341 0.0 0.0"/>
     <axis xyz="0 0 0"/>
   </joint>
-  <link name="tcp">
+  <link name="$(arg prefix)tcp">
     <inertial>
       <mass value="0.1"/>

File: irc_ros_description/urdf/gripper_none.urdf.xacro (robot description, xacro)
@@ -3,4 +3,4 @@
 <!-- Only requires the following line for xacro support and the definition of gripper_link -->
 <robot xmlns:xacro="http://www.ros.org/wiki/xacro">
-    <link name="gripper_mount" />
+    <link name="$(arg prefix)gripper_mount" />
 </robot>

File: irc_ros_description/urdf/gripper_schmalz_ecbpmi.urdf.xacro (robot description, xacro)
@@ -2,5 +2,5 @@
 <robot xmlns:xacro="http://www.ros.org/wiki/xacro"
     name="gripper_schmalz_ecbpmi">
-  <link name="gripper_mount">
+  <link name="$(arg prefix)gripper_mount">
     <visual>
       <geometry>
@@ -20,10 +20,10 @@
     </inertial>
   </link>
-  <joint name="gripper_mount_joint" type="fixed">
-    <parent link="gripper_mount" />
-    <child link="gripper_base" />
+  <joint name="$(arg prefix)gripper_mount_joint" type="fixed">
+    <parent link="$(arg prefix)gripper_mount" />
+    <child link="$(arg prefix)gripper_base" />
     <origin xyz="0.01 0.0 0.0" rpy="0.0 0.0 0.0" />
   </joint>
-  <link name="gripper_base">
+  <link name="$(arg prefix)gripper_base">
     <visual>
       <geometry>
@@ -43,11 +43,11 @@
     </inertial>
   </link>
-  <joint name="joint99" type="fixed">
-    <parent link="gripper_base"/>
-    <child link="tcp"/>
+  <joint name="$(arg prefix)joint99" type="fixed">
+    <parent link="$(arg prefix)gripper_base"/>
+    <child link="$(arg prefix)tcp"/>
     <origin rpy="0.0 0.0 0.0" xyz="0.07341 0.0 0.0"/>
     <axis xyz="0 0 0"/>
   </joint>
-  <link name="tcp">
+  <link name="$(arg prefix)tcp">
     <inertial>
       <mass value="0.1"/>

File: irc_ros_description/urdf/igus_rebel_4dof.urdf.xacro (robot description, xacro)
@@ -24,11 +24,11 @@
   <joint name="world_joint" type="fixed">
     <parent link="world" />
-    <child link = "base_link" />
+    <child link = "$(arg prefix)base_link" />
     <origin xyz="0.0 0.0 0.0" rpy="0.0 0.0 0.0" />
   </joint>
   <!-- Grippers -->
-  <joint name="hand_to_gripper" type="fixed">
-    <parent link="hand" />
-    <child link = "gripper_mount" />
+  <joint name="$(arg prefix)hand_to_gripper" type="fixed">
+    <parent link="$(arg prefix)hand" />
+    <child link = "$(arg prefix)gripper_mount" />
     <origin xyz="0.0 0.0 0.0" rpy="0.0 ${-pi/2} 0.0" />
   </joint>

File: irc_ros_description/urdf/igus_rebel_4dof_00.xacro (robot description, xacro)
@@ -2,5 +2,5 @@
 <robot xmlns:xacro="http://www.ros.org/wiki/xacro"
        name="igus_rebel_4dof" >
-  <link name="base_link">
+  <link name="$(arg prefix)base_link">
     <visual>
       <geometry>
@@ -18,12 +18,12 @@
     </inertial>
   </link>
-  <joint name="joint1" type="revolute">
-    <parent link="base_link"/>
-    <child link="link_1"/>
+  <joint name="$(arg prefix)joint1" type="revolute">
+    <parent link="$(arg prefix)base_link"/>
+    <child link="$(arg prefix)link_1"/>
     <origin rpy="0.0 0.0 0.0" xyz="0.0 0.0 0.100"/>
     <axis xyz="0 0 -1"/>
     <limit effort="330.0" lower="${-pi*179/180}" upper="${pi*179/180}" velocity="2.16"/>
   </joint>
-  <link name="link_1">
+  <link name="$(arg prefix)link_1">
     <visual>
       <geometry>
@@ -43,12 +43,12 @@
     </inertial>
   </link>
-  <joint name="joint2" type="revolute">
-    <parent link="link_1"/>
-    <child link="link_2"/>
+  <joint name="$(arg prefix)joint2" type="revolute">
+    <parent link="$(arg prefix)link_1"/>
+    <child link="$(arg prefix)link_2"/>
     <origin rpy="0.0 ${pi/6} 0.0" xyz="0.0 0 0.149"/>
     <axis xyz="0 1 0"/>
     <limit effort="330.0" lower="${-pi*2/3}" upper="${pi*2/3}" velocity="2.16"/>
   </joint>
-  <link name="link_2">
+  <link name="$(arg prefix)link_2">
     <visual>
       <geometry>
@@ -68,12 +68,12 @@
     </inertial>
   </link>
-  <joint name="joint3" type="revolute">
-    <parent link="link_2"/>
-    <child link="link_3"/>
+  <joint name="$(arg prefix)joint3" type="revolute">
+    <parent link="$(arg prefix)link_2"/>
+    <child link="$(arg prefix)link_3"/>
     <origin rpy="0.0 ${pi/6} 0.0" xyz="0.0 0.0 0.2384"/>
     <axis xyz="0 1 0"/>
     <limit effort="330.0" lower="${-pi*2/3}" upper="${pi*2/3}" velocity="2.16"/>
   </joint>
-  <link name="link_3">
+  <link name="$(arg prefix)link_3">
     <visual>
       <geometry>
@@ -94,7 +94,7 @@
   </link>
   <xacro:if value="$(arg continuous_last_joint)">
-    <joint name="joint4" type="continuous">
-      <parent link="link_3"/>
-      <child link="link_4"/>
+    <joint name="$(arg prefix)joint4" type="continuous">
+      <parent link="$(arg prefix)link_3"/>
+      <child link="$(arg prefix)link_4"/>
       <origin rpy="0.0 0.0 0.0" xyz="0.0 0.0 0.2423"/>
       <axis xyz="0 -1 0"/>
@@ -103,7 +103,7 @@
   </xacro:if>
   <xacro:unless value="$(arg continuous_last_joint)">
-    <joint name="joint4" type="revolute">
-      <parent link="link_3"/>
-      <child link="link_4"/>
+    <joint name="$(arg prefix)joint4" type="revolute">
+      <parent link="$(arg prefix)link_3"/>
+      <child link="$(arg prefix)link_4"/>
       <origin rpy="0.0 0.0 0.0" xyz="0.0 0.0 0.2423"/>
       <axis xyz="0 -1 0"/>
@@ -111,5 +111,5 @@
     </joint>
   </xacro:unless>
-  <link name="link_4">
+  <link name="$(arg prefix)link_4">
     <visual>
       <geometry>
@@ -129,11 +129,11 @@
     </inertial>
   </link>
-  <joint name="joint5" type="fixed">
-    <parent link="link_4"/>
-    <child link="hand"/>
+  <joint name="$(arg prefix)joint5" type="fixed">
+    <parent link="$(arg prefix)link_4"/>
+    <child link="$(arg prefix)hand"/>
     <origin rpy="0.0 0.0 0.0" xyz="0.0 0.0 0.062"/>
     <axis xyz="0 -1 0"/>
   </joint>
-  <link name="hand">
+  <link name="$(arg prefix)hand">
     <inertial>
       <mass value="0.1"/>
@@ -141,10 +141,10 @@
     </inertial>
   </link>
-  <gpio name="dio_base">
+  <gpio name="$(arg prefix)dio_base">
     <param name="can_id">0x70</param>
     <command_interface name="digital_output" size="7" data_type="bool" />
     <state_interface name="digital_input" size="7" data_type="bool" />
   </gpio>
-  <gpio name="dio_arm">
+  <gpio name="$(arg prefix)dio_arm">
     <param name="can_id">0x80</param>
     <command_interface name="digital_output" size="2" data_type="bool" />

File: irc_ros_description/urdf/igus_rebel_6dof.urdf.xacro (robot description, xacro)
@@ -25,12 +25,12 @@
     <joint name="world_joint" type="fixed">
       <parent link="world" />
-      <child link = "base_link" />
+      <child link = "$(arg prefix)base_link" />
       <origin xyz="0.0 0.0 0.0" rpy="0.0 0.0 0.0" />
     </joint>
   </xacro:if>
   <!-- Grippers -->
-  <joint name="hand_to_gripper" type="fixed">
-    <parent link="hand" />
-    <child link = "gripper_mount" />
+  <joint name="$(arg prefix)hand_to_gripper" type="fixed">
+    <parent link="$(arg prefix)hand" />
+    <child link = "$(arg prefix)gripper_mount" />
     <origin xyz="0.0 0.0 0.0" rpy="0.0 ${-pi/2} 0.0" />
   </joint>

File: irc_ros_description/urdf/igus_rebel_6dof_00.xacro (robot description, xacro)
@@ -2,5 +2,5 @@
 <robot xmlns:xacro="http://www.ros.org/wiki/xacro"
        name="igus_rebel_6dof" >
-  <link name="base_link">
+  <link name="$(arg prefix)base_link">
     <visual>
       <geometry>
@@ -18,12 +18,12 @@
     </inertial>
   </link>
-  <joint name="joint1" type="revolute">
-    <parent link="base_link"/>
-    <child link="link_1"/>
+  <joint name="$(arg prefix)joint1" type="revolute">
+    <parent link="$(arg prefix)base_link"/>
+    <child link="$(arg prefix)link_1"/>
     <origin rpy="0.0 0.0 0.0" xyz="0.0 0 0.100"/>
     <axis xyz="0 0 -1"/>
     <limit effort="330.0" lower="${-pi*179/180}" upper="${pi*179/180}" velocity="2.16"/>
   </joint>
-  <link name="link_1">
+  <link name="$(arg prefix)link_1">
     <visual>
       <geometry>
@@ -43,12 +43,12 @@
     </inertial>
   </link>
-  <joint name="joint2" type="revolute">
-    <parent link="link_1"/>
-    <child link="link_2"/>
+  <joint name="$(arg prefix)joint2" type="revolute">
+    <parent link="$(arg prefix)link_1"/>
+    <child link="$(arg prefix)link_2"/>
     <origin rpy="0.0 ${pi/6} 0.0" xyz="0.0 0 0.149"/>
     <axis xyz="0 1 0"/>
     <limit effort="330.0" lower="${-pi*2/3}" upper="${pi*2/3}" velocity="2.16"/>
   </joint>
-  <link name="link_2">
+  <link name="$(arg prefix)link_2">
     <visual>
       <geometry>
@@ -68,12 +68,12 @@
     </inertial>
   </link>
-  <joint name="joint3" type="revolute">
-    <parent link="link_2"/>
-    <child link="link_5"/>
+  <joint name="$(arg prefix)joint3" type="revolute">
+    <parent link="$(arg prefix)link_2"/>
+    <child link="$(arg prefix)link_5"/>
     <origin rpy="0.0 ${pi/6} 0.0" xyz="0.0 0.0 0.2384"/>
     <axis xyz="0 1 0"/>
     <limit effort="330.0" lower="${-pi*2/3}" upper="${pi*2/3}" velocity="2.16"/>
   </joint>
-  <link name="link_5">
+  <link name="$(arg prefix)link_5">
     <visual>
       <geometry>
@@ -93,7 +93,7 @@
     </inertial>
   </link>
-  <joint name="joint4" type="revolute">
-    <parent link="link_5"/>
-    <child link="link_6"/>
+  <joint name="$(arg prefix)joint4" type="revolute">
+    <parent link="$(arg prefix)link_5"/>
+    <child link="$(arg prefix)link_6"/>
     <!-- FIXME The 0.03m offset are most likely caused by the mesh file -->
     <origin rpy="0.0 0.0 0.0" xyz="0.0 0 ${0.149 - 0.03}"/>
@@ -101,5 +101,5 @@
     <limit effort="330.0" lower="${-pi*179/180}" upper="${pi*179/180}" velocity="2.16"/>
   </joint>
-  <link name="link_6">
+  <link name="$(arg prefix)link_6">
     <visual>
       <geometry>
@@ -119,7 +119,7 @@
     </inertial>
   </link>
-  <joint name="joint5" type="revolute">
-    <parent link="link_6"/>
-    <child link="link_7"/>
+  <joint name="$(arg prefix)joint5" type="revolute">
+    <parent link="$(arg prefix)link_6"/>
+    <child link="$(arg prefix)link_7"/>
     <!-- FIXME The 0.03m offset are most likely caused by the mesh file -->
     <origin rpy="0.0 0.0 0.0" xyz="0.0 0 ${0.14 + 0.03}"/>
@@ -127,5 +127,5 @@
     <limit effort="330.0" lower="${-pi*19/36}" upper="${pi*19/36}" velocity="2.16"/>
   </joint>
-  <link name="link_7">
+  <link name="$(arg prefix)link_7">
     <visual>
       <geometry>
@@ -146,7 +146,7 @@
   </link>
   <xacro:if value="$(arg continuous_last_joint)">
-  <joint name="joint6" type="continuous">
-      <parent link="link_7"/>
-      <child link="link_8"/>
+  <joint name="$(arg prefix)joint6" type="continuous">
+      <parent link="$(arg prefix)link_7"/>
+      <child link="$(arg prefix)link_8"/>
       <origin rpy="0.0 0.0 0.0" xyz="0.0 0 0.1208"/>
       <axis xyz="0 0 1"/>
@@ -155,7 +155,7 @@
   </xacro:if>
   <xacro:unless value="$(arg continuous_last_joint)">
-    <joint name="joint6" type="revolute">
-      <parent link="link_7"/>
-      <child link="link_8"/>
+    <joint name="$(arg prefix)joint6" type="revolute">
+      <parent link="$(arg prefix)link_7"/>
+      <child link="$(arg prefix)link_8"/>
       <origin rpy="0.0 0.0 0.0" xyz="0.0 0 0.1208"/>
       <axis xyz="0 0 1"/>
@@ -163,5 +163,5 @@
     </joint>
   </xacro:unless>
-  <link name="link_8">
+  <link name="$(arg prefix)link_8">
     <visual>
       <geometry>
@@ -181,12 +181,12 @@
     </inertial>
   </link>
-  <joint name="joint7" type="fixed">
-    <parent link="link_8"/>
-    <child link="hand"/>
+  <joint name="$(arg prefix)joint7" type="fixed">
+    <parent link="$(arg prefix)link_8"/>
+    <child link="$(arg prefix)hand"/>
     <origin rpy="0.0 0.0 0.0" xyz="0.0 0 0.0012"/>
     <axis xyz="0 0 1"/>
     <limit effort="330.0" lower="-3.12414" upper="3.12414" velocity="2.16"/>
   </joint>
-  <link name="hand">
+  <link name="$(arg prefix)hand">
     <inertial>
       <mass value="0.1"/>

File: irc_ros_description/urdf/igus_rebel_6dof_pre.xacro (robot description, xacro)
@@ -2,5 +2,5 @@
 <robot xmlns:xacro="http://www.ros.org/wiki/xacro"
        name="igus_rebel_6dof" >
-  <link name="base_link">
+  <link name="$(arg prefix)base_link">
     <visual>
       <geometry>
@@ -18,12 +18,12 @@
     </inertial>
   </link>
-  <joint name="joint1" type="revolute">
-    <parent link="base_link"/>
-    <child link="link_1"/>
+  <joint name="$(arg prefix)joint1" type="revolute">
+    <parent link="$(arg prefix)base_link"/>
+    <child link="$(arg prefix)link_1"/>
     <origin rpy="0.0 0.0 0.0" xyz="0.0 0 0.144"/>
     <axis xyz="0 0 -1"/>
     <limit effort="330.0" lower="${-pi*179/180}" upper="${pi*179/180}" velocity="2.16"/>
   </joint>
-  <link name="link_1">
+  <link name="$(arg prefix)link_1">
     <visual>
       <geometry>
@@ -43,12 +43,12 @@
     </inertial>
   </link>
-  <joint name="joint2" type="revolute">
-    <parent link="link_1"/>
-    <child link="link_2"/>
+  <joint name="$(arg prefix)joint2" type="$(arg prefix)revolute">
+    <parent link="$(arg prefix)link_1"/>
+    <child link="$(arg prefix)link_2"/>
     <origin rpy="0.0 0.0 0.0" xyz="0.0 0 0.130"/>
     <axis xyz="0 1 0"/>
     <limit effort="330.0" lower="${-pi*2/3 + pi/6}" upper="${pi*2/3 + pi/6}" velocity="2.16"/>
   </joint>
-  <link name="link_2">
+  <link name="$(arg prefix)link_2">
     <visual>
       <geometry>
@@ -68,12 +68,12 @@
     </inertial>
   </link>
-  <joint name="joint3" type="revolute">
-    <parent link="link_2"/>
-    <child link="link_5"/>
+  <joint name="$(arg prefix)joint3" type="revolute">
+    <parent link="$(arg prefix)link_2"/>
+    <child link="$(arg prefix)link_5"/>
     <origin rpy="0.0 0.0 0.0" xyz="0.0 0.0 0.2384"/>
     <axis xyz="0 1 0"/>
     <limit effort="330.0" lower="${-pi*2/3 + pi/6}" upper="${pi*2/3 + pi/6}" velocity="2.16"/>
   </joint>
-  <link name="link_5">
+  <link name="$(arg prefix)link_5">
     <visual>
       <geometry>
@@ -93,7 +93,7 @@
     </inertial>
   </link>
-  <joint name="joint4" type="revolute">
-    <parent link="link_5"/>
-    <child link="link_6"/>
+  <joint name="$(arg prefix)joint4" type="revolute">
+    <parent link="$(arg prefix)link_5"/>
+    <child link="$(arg prefix)link_6"/>
     <!-- FIXME The 0.03m offset are most likely caused by the mesh file -->
     <origin rpy="0.0 0.0 0.0" xyz="0.0 0 ${0.149 - 0.03}"/>
@@ -101,5 +101,5 @@
     <limit effort="330.0" lower="${-pi*179/180}" upper="${pi*179/180}" velocity="2.16"/>
   </joint>
-  <link name="link_6">
+  <link name="$(arg prefix)link_6">
     <visual>
       <geometry>
@@ -119,7 +119,7 @@
     </inertial>
   </link>
-  <joint name="joint5" type="revolute">
-    <parent link="link_6"/>
-    <child link="link_7"/>
+  <joint name="$(arg prefix)joint5" type="revolute">
+    <parent link="$(arg prefix)link_6"/>
+    <child link="$(arg prefix)link_7"/>
     <!-- FIXME The 0.03m offset are most likely caused by the mesh file -->
     <origin rpy="0.0 0.0 0.0" xyz="0.0 0 ${0.14 + 0.03}"/>
@@ -127,5 +127,5 @@
     <limit effort="330.0" lower="${-pi*19/36}" upper="${pi*19/36}" velocity="2.16"/>
   </joint>
-  <link name="link_7">
+  <link name="$(arg prefix)link_7">
     <visual>
       <geometry>
@@ -146,7 +146,7 @@
   </link>
   <xacro:if value="$(arg continuous_last_joint)">
-     <joint name="joint6" type="continuous">
-      <parent link="link_7"/>
-      <child link="link_8"/>
+     <joint name="$(arg prefix)joint6" type="continuous">
+      <parent link="$(arg prefix)link_7"/>
+      <child link="$(arg prefix)link_8"/>
       <origin rpy="0.0 0.0 0.0" xyz="0.0 0 0.1208"/>
       <axis xyz="0 0 1"/>
@@ -155,7 +155,7 @@
   </xacro:if>
   <xacro:unless value="$(arg continuous_last_joint)">
-    <joint name="joint6" type="revolute">
-      <parent link="link_7"/>
-      <child link="link_8"/>
+    <joint name="$(arg prefix)joint6" type="revolute">
+      <parent link="$(arg prefix)link_7"/>
+      <child link="$(arg prefix)link_8"/>
       <origin rpy="0.0 0.0 0.0" xyz="0.0 0 0.1208"/>
       <axis xyz="0 0 1"/>
@@ -181,12 +181,12 @@
     </inertial>
   </link>
-  <joint name="joint7" type="fixed">
-    <parent link="link_8"/>
-    <child link="hand"/>
+  <joint name="$(arg prefix)joint7" type="fixed">
+    <parent link="$(arg prefix)link_8"/>
+    <child link="$(arg prefix)hand"/>
     <origin rpy="0.0 0.0 0.0" xyz="0.0 0 0.0012"/>
     <axis xyz="0 0 1"/>
     <limit effort="330.0" lower="-3.12414" upper="3.12414" velocity="2.16"/>
   </joint>
-  <link name="hand">
+  <link name="$(arg prefix)hand">
     <inertial>
       <mass value="0.1"/>

File: irc_ros_description/urdf/igus_robolink_rl_dp_5.urdf.xacro (robot description, xacro)
@@ -21,12 +21,12 @@
   <joint name="world_joint" type="fixed">
     <parent link="world" />
-    <child link = "base_link" />
+    <child link = "$(arg prefix)base_link" />
     <origin xyz="0.0 0.0 0.0" rpy="0.0 0.0 0.0" />
   </joint>
   <!-- Grippers -->
   <xacro:if value="$(arg use_gripper)">
-    <joint name="hand_to_gripper" type="fixed">
-      <parent link="hand" />
-      <child link = "gripper_mount" />
+    <joint name="$(arg prefix)hand_to_gripper" type="fixed">
+      <parent link="$(arg prefix)hand" />
+      <child link = "$(arg prefix)gripper_mount" />
       <origin xyz="0.0 0.0 0.0" rpy="0.0 ${-pi/2} 0.0" />
     </joint>
