Commit message: Change chassis to base_link, add prefix to remaining files

File: irc_ros_description/urdf/igus_robolink_rl_dp_5.xacro (robot description, xacro)
@@ -2,5 +2,5 @@
 <robot xmlns:xacro="http://www.ros.org/wiki/xacro"
        name="igus_robolink_rl_dp_5" >
-  <link name="base_link">
+  <link name="$(arg prefix)base_link">
     <visual>
       <geometry>
@@ -18,12 +18,12 @@
     </inertial>
   </link>
-  <joint name="joint1" type="revolute">
-    <parent link="base_link"/>
-    <child link="link_1"/>
+  <joint name="$(arg prefix)joint1" type="revolute">
+    <parent link="$(arg prefix)base_link"/>
+    <child link="$(arg prefix)link_1"/>
     <origin rpy="0.0 0.0 0.0" xyz="0.0 0 0.0095"/>
     <axis xyz="0 0 -1"/>
     <limit effort="330.0" lower="${-pi*7/9}" upper="${pi*7/9}" velocity="2.16"/>
   </joint>
-  <link name="link_1">
+  <link name="$(arg prefix)link_1">
     <visual>
       <geometry>
@@ -43,12 +43,12 @@
     </inertial>
   </link>
-  <joint name="joint2" type="revolute">
-    <parent link="link_1"/>
-    <child link="link_2"/>
+  <joint name="$(arg prefix)joint2" type="revolute">
+    <parent link="$(arg prefix)link_1"/>
+    <child link="$(arg prefix)link_2"/>
     <origin rpy="0.0 0.0 0.0" xyz="0.0 0 0.145"/>
     <axis xyz="0 1 0"/>
     <limit effort="330.0" lower="${-pi*5/18}" upper="${pi/2}" velocity="2.16"/>
   </joint>
-  <link name="link_2">
+  <link name="$(arg prefix)link_2">
     <visual>
       <geometry>
@@ -68,12 +68,12 @@
     </inertial>
   </link>
-  <joint name="joint3" type="revolute">
-    <parent link="link_2"/>
-    <child link="link_5"/>
+  <joint name="$(arg prefix)joint3" type="revolute">
+    <parent link="$(arg prefix)link_2"/>
+    <child link="$(arg prefix)link_5"/>
     <origin rpy="0.0 1.57 0.0" xyz="0.0 0.0 0.350"/>
     <axis xyz="0 1 0"/>
     <limit effort="330.0" lower="${-pi*41/36}" upper="${pi*5/36}" velocity="2.16"/>
   </joint>
-  <link name="link_5">
+  <link name="$(arg prefix)link_5">
     <visual>
       <geometry>
@@ -93,12 +93,12 @@
     </inertial>
   </link>
-  <joint name="joint4" type="revolute">
-    <parent link="link_5"/>
-    <child link="link_6"/>
+  <joint name="$(arg prefix)joint4" type="revolute">
+    <parent link="$(arg prefix)link_5"/>
+    <child link="$(arg prefix)link_6"/>
     <origin rpy="0.0 0.0 0.0" xyz="0.0 0 0.270"/>
     <axis xyz="0 1 0"/>
     <limit effort="330.0" lower="${-pi*5/9}" upper="${pi*5/9}" velocity="2.16"/>
   </joint>
-  <link name="link_6">
+  <link name="$(arg prefix)link_6">
     <visual>
       <geometry>
@@ -119,7 +119,7 @@
   </link>
   <xacro:if value="$(arg continuous_last_joint)">
-    <joint name="joint5" type="continuous">
-      <parent link="link_6"/>
-      <child link="link_7"/>
+    <joint name="$(arg prefix)joint5" type="continuous">
+      <parent link="$(arg prefix)link_6"/>
+      <child link="$(arg prefix)link_7"/>
       <origin rpy="0.0 0.0 0.0" xyz="0.0 0 0.1785"/>
       <axis xyz="0 0 1"/>
@@ -128,7 +128,7 @@
   </xacro:if>
   <xacro:unless value="$(arg continuous_last_joint)">
-    <joint name="joint5" type="revolute">
-      <parent link="link_6"/>
-      <child link="link_7"/>
+    <joint name="$(arg prefix)joint5" type="revolute">
+      <parent link="$(arg prefix)link_6"/>
+      <child link="$(arg prefix)link_7"/>
       <origin rpy="0.0 0.0 0.0" xyz="0.0 0 0.1785"/>
       <axis xyz="0 0 1"/>
@@ -136,5 +136,5 @@
     </joint>
   </xacro:unless>
-  <link name="link_7">
+  <link name="$(arg prefix)link_7">
     <visual>
       <geometry>
@@ -154,12 +154,12 @@
     </inertial>
   </link>
-  <joint name="joint6" type="fixed">
-    <parent link="link_7"/>
-    <child link="hand"/>
+  <joint name="$(arg prefix)joint6" type="fixed">
+    <parent link="$(arg prefix)link_7"/>
+    <child link="$(arg prefix)hand"/>
     <origin rpy="0.0 0.0 0.0" xyz="0.0 0 0.0115"/>
     <axis xyz="0 0 1"/>
     <limit effort="330.0" lower="-1.65806" upper="1.65806" velocity="2.16"/>
   </joint>
-  <link name="hand">
+  <link name="$(arg prefix)hand">
     <inertial>
       <mass value="0.1"/>

File: irc_ros_description/urdf/rebel_on_platform.urdf.xacro (robot description, xacro)
@@ -2,9 +2,9 @@
 <robot xmlns:xacro="http://www.ros.org/wiki/xacro"
        name="rebel_on_platform" >
-  <xacro:include filename="$(find irc_ros_description)/urdf/igus_rebel_6dof.urdf.xacro"/>
-  <xacro:include filename="$(find irc_ros_description)/urdf/cpr_platform_medium.urdf.xacro"/>
+  <xacro:include filename="$(find irc_ros_description)/urdf/igus_rebel_6dof.urdf.xacro" prefix="rebel_1_" />
+  <xacro:include filename="$(find irc_ros_description)/urdf/cpr_platform_medium.urdf.xacro" prefix=""/>
   <joint name="platform_to_rebel" type="fixed">
-    <parent link="chassis" />
-    <child link = "base_link" />
+    <parent link="base_link" />
+    <child link="rebel_1_base_link" />
     <origin xyz="0.0 0.0 ${0.7-0.1}" rpy="0.0 0.0 ${-pi/6}" />
   </joint>
