Commit message: Change remaining robot urdfs, add missing xacro header

File: irc_ros_description/urdf/igus_rebel_4dof.urdf.xacro (robot description, xacro)
@@ -6,4 +6,10 @@
   <!-- Gripper selection -->
   <xacro:arg name="gripper" default="schmalz_ecbpmi" />
+  <!-- Enable continuous rotation on the last join. While the last axis can turn continuously,
+  it is limited here in case a tool with wiring is mounted. If you are certain that no wiring
+  issues can arise you may enable this -->
+  <xacro:arg name="continuous_last_joint" default="false" />
+  <!-- TODO -->
+  <xacro:arg name="root_link" default="false" />
   <xacro:include filename="$(find irc_ros_description)/urdf/igus_rebel_4dof_$(arg rebel_version).xacro" />
   <xacro:include filename="$(find irc_ros_description)/urdf/igus_rebel_4dof_$(arg rebel_version).ros2_control.xacro" />

File: irc_ros_description/urdf/igus_rebel_4dof_00.ros2_control.xacro (robot description, xacro)
@@ -58,6 +58,8 @@
   <joint name="joint4">
     <command_interface name="position">
-      <param name="min">${-pi*19/36}</param>
-      <param name="max">${pi*19/36}</param>
+      <xacro:unless value="$(arg continuous_last_joint)">
+        <param name="min">${-pi*19/36}</param>
+        <param name="max">${pi*19/36}</param>
+      </xacro:unless>
     </command_interface>
     <command_interface name="velocity">

File: irc_ros_description/urdf/igus_rebel_4dof_00.xacro (robot description, xacro)
@@ -1,4 +1,5 @@
 <?xml version="1.0" ?>
-<robot name="igus_rebel_4dof">
+<robot xmlns:xacro="http://wiki.ros.org/xacro"
+       name="igus_rebel_4dof" >
   <link name="base_link">
     <visual>
@@ -92,11 +93,22 @@
     </inertial>
   </link>
-  <joint name="joint4" type="revolute">
-    <parent link="link_3"/>
-    <child link="link_4"/>
-    <origin rpy="0.0 0.0 0.0" xyz="0.0 0.0 0.2423"/>
-    <axis xyz="0 -1 0"/>
-    <limit effort="330.0" lower="${-pi*179/180}" upper="${pi*179/180}" velocity="2.16"/>
-  </joint>
+  <xacro:if value="$(arg continuous_last_joint)">
+    <joint name="joint4" type="continuous">
+      <parent link="link_3"/>
+      <child link="link_4"/>
+      <origin rpy="0.0 0.0 0.0" xyz="0.0 0.0 0.2423"/>
+      <axis xyz="0 -1 0"/>
+      <limit effort="330.0" velocity="2.16"/>
+    </joint>
+  </xacro:if>
+  <xacro:unless value="$(arg continuous_last_joint)">
+    <joint name="joint4" type="revolute">
+      <parent link="link_3"/>
+      <child link="link_4"/>
+      <origin rpy="0.0 0.0 0.0" xyz="0.0 0.0 0.2423"/>
+      <axis xyz="0 -1 0"/>
+      <limit effort="330.0" lower="${-pi*179/180}" upper="${pi*179/180}" velocity="2.16"/>
+    </joint>
+  </xacro:unless>
   <link name="link_4">
     <visual>

File: irc_ros_description/urdf/igus_rebel_4dof_01.ros2_control.xacro (robot description, xacro)
@@ -58,6 +58,8 @@
   <joint name="joint4">
     <command_interface name="position">
-      <param name="min">${-pi*19/36}</param>
-      <param name="max">${pi*19/36}</param>
+      <xacro:unless value="$(arg continuous_last_joint)">
+        <param name="min">${-pi*19/36}</param>
+        <param name="max">${pi*19/36}</param>
+      </xacro:unless>
     </command_interface>
     <command_interface name="velocity">

File: irc_ros_description/urdf/igus_rebel_6dof.urdf.xacro (robot description, xacro)
@@ -6,8 +6,8 @@
   <!-- Gripper selection -->
   <xacro:arg name="gripper" default="ext_dio_gripper" />
-  <!-- Enable continuous rotation on the last joint -->
-  <!-- While the last axis can turn continuously, it is limited here in case a tool with wiring is mounted.
-  If you are certain that no wiring issues can arise you may change this do a continuous joint -->
-  <xacro:arg name="continuous_last_joint" default="true" />
+  <!-- Enable continuous rotation on the last join. While the last axis can turn continuously,
+  it is limited here in case a tool with wiring is mounted. If you are certain that no wiring
+  issues can arise you may enable this -->
+  <xacro:arg name="continuous_last_joint" default="false" />
   <!-- TODO -->
   <xacro:arg name="root_link" default="false" />

File: irc_ros_description/urdf/igus_rebel_6dof_00.xacro (robot description, xacro)
@@ -1,4 +1,5 @@
 <?xml version="1.0" ?>
-<robot name="igus_rebel_6dof">
+<robot xmlns:xacro="http://wiki.ros.org/xacro"
+       name="igus_rebel_6dof" >
   <link name="base_link">
     <visual>

File: irc_ros_description/urdf/igus_rebel_6dof_01.ros2_control.xacro (robot description, xacro)
@@ -1,4 +1,5 @@
 <?xml version="1.0" ?>
-<robot xmlns:xacro="http://www.ros.org/wiki/xacro">
+<robot xmlns:xacro="http://wiki.ros.org/xacro"
+       name="igus_rebel_6dof" >
   <ros2_control name="Rebel" type="system">
     <hardware>

File: irc_ros_description/urdf/igus_rebel_6dof_pre.ros2_control.xacro (robot description, xacro)
@@ -82,8 +82,8 @@
     <joint name="joint6">
       <command_interface name="position">
-        <!-- While the last axis can turn continuously, it is limited here in case a tool with wiring is mounted.
-        If you are certain that no wiring issues can arise you may change this do a continuous joint -->
-        <param name="min">${-pi*179/180}</param>
-        <param name="max">${pi*179/180}</param>
+        <xacro:unless value="$(arg continuous_last_joint)">
+          <param name="min">${-pi*179/180}</param>
+          <param name="max">${pi*179/180}</param>
+        </xacro:unless>
       </command_interface>
       <command_interface name="velocity">

File: irc_ros_description/urdf/igus_rebel_6dof_pre.xacro (robot description, xacro)
@@ -1,4 +1,5 @@
 <?xml version="1.0" ?>
-<robot name="igus_rebel_6dof">
+<robot xmlns:xacro="http://wiki.ros.org/xacro"
+       name="igus_rebel_6dof" >
   <link name="base_link">
     <visual>
@@ -144,11 +145,22 @@
     </inertial>
   </link>
-  <joint name="joint6" type="revolute">
-    <parent link="link_7"/>
-    <child link="link_8"/>
-    <origin rpy="0.0 0.0 0.0" xyz="0.0 0 0.1208"/>
-    <axis xyz="0 0 1"/>
-    <limit effort="330.0" lower="${-pi*179/180}" upper="${pi*179/180}" velocity="2.16"/>
-  </joint>
+  <xacro:if value="$(arg continuous_last_joint)">
+     <joint name="joint6" type="continuous">
+      <parent link="link_7"/>
+      <child link="link_8"/>
+      <origin rpy="0.0 0.0 0.0" xyz="0.0 0 0.1208"/>
+      <axis xyz="0 0 1"/>
+      <limit effort="330.0" velocity="2.16"/>
+    </joint>
+  </xacro:if>
+  <xacro:unless value="$(arg continuous_last_joint)">
+    <joint name="joint6" type="revolute">
+      <parent link="link_7"/>
+      <child link="link_8"/>
+      <origin rpy="0.0 0.0 0.0" xyz="0.0 0 0.1208"/>
+      <axis xyz="0 0 1"/>
+      <limit effort="330.0" lower="${-pi*179/180}" upper="${pi*179/180}" velocity="2.16"/>
+    </joint>
+  </xacro:unless>
   <link name="link_8">
     <visual>

File: irc_ros_description/urdf/igus_robolink_rl_dp_5.urdf.xacro (robot description, xacro)
@@ -5,6 +5,8 @@
   <xacro:arg name="use_gripper" default="false" />
   <xacro:arg name="gripper" default="schmalz_ecbpmi" />
-  <!-- Enable continuous rotation on the last joint -->
-  <xacro:arg name="continuous_last_joint" default="true" />
+  <!-- Enable continuous rotation on the last join. While the last axis can turn continuously,
+  it is limited here in case a tool with wiring is mounted. If you are certain that no wiring
+  issues can arise you may enable this -->
+  <xacro:arg name="continuous_last_joint" default="false" />
   <xacro:include filename="$(find irc_ros_description)/urdf/igus_robolink_rl_dp_5.xacro" />
   <xacro:include filename="$(find irc_ros_description)/urdf/igus_robolink_rl_dp_5.ros2_control.xacro" />

Commit message: Adapt gripper selection

File: irc_ros_description/urdf/igus_rebel_4dof.urdf.xacro (robot description, xacro)
@@ -29,9 +29,5 @@
   </joint>
   <!-- Grippers -->
-  <xacro:include filename="$(find irc_ros_description)/urdf/grippers/$(arg gripper).urdf.xacro" />
-  <joint name="$(arg prefix)flange_to_gripper" type="fixed">
-    <parent link="$(arg prefix)flange" />
-    <child link = "$(arg prefix)gripper_mount" />
-    <origin xyz="0.0 0.0 0.0" rpy="0.0 ${-pi/2} 0.0" />
-  </joint>
+  <xacro:include filename="$(find irc_ros_description)/urdf/grippers/grippers.macro.xacro" />
+  <xacro:gripper prefix="$(arg prefix)" gripper_type="$(arg gripper)" parent_link="$(arg prefix)flange" />
 </robot>

File: irc_ros_description/urdf/igus_rebel_6dof.urdf.xacro (robot description, xacro)
@@ -16,5 +16,5 @@
   <!-- Gripper selection -->
   <xacro:arg name="gripper" default="none" />
-  <!-- Include and call relevant macro -->
+  <!-- Include and call rebel macro -->
   <xacro:include filename="$(find irc_ros_description)/urdf/robots/igus_rebel_6dof.macro.xacro" />
   <xacro:igus_rebel_6dof prefix="$(arg prefix)" continuous_last_joint="$(arg continuous_last_joint)" rebel_version="'$(arg rebel_version)'" controller_type="$(arg controller_type)" />
@@ -27,9 +27,5 @@
   </joint>
   <!-- Grippers -->
-  <xacro:include filename="$(find irc_ros_description)/urdf/grippers/$(arg gripper).urdf.xacro" />
-  <joint name="$(arg prefix)flange_to_gripper" type="fixed">
-    <parent link="$(arg prefix)flange" />
-    <child link = "$(arg prefix)gripper_mount" />
-    <origin xyz="0.0 0.0 0.0" rpy="0.0 ${-pi/2} 0.0" />
-  </joint>
+  <xacro:include filename="$(find irc_ros_description)/urdf/grippers/grippers.macro.xacro" />
+  <xacro:gripper prefix="$(arg prefix)" gripper_type="$(arg gripper)" parent_link="$(arg prefix)flange" />
 </robot>

File: irc_ros_description/urdf/igus_robolink_rl_dp_5.urdf.xacro (robot description, xacro)
@@ -25,9 +25,5 @@
   </joint>
   <!-- Grippers -->
-  <xacro:include filename="$(find irc_ros_description)/urdf/grippers/$(arg gripper).urdf.xacro" />
-  <joint name="$(arg prefix)flange_to_gripper" type="fixed">
-    <parent link="$(arg prefix)flange" />
-    <child link = "$(arg prefix)gripper_mount" />
-    <origin xyz="0.0 0.0 0.0" rpy="0.0 ${-pi/2} 0.0" />
-  </joint>
+  <xacro:include filename="$(find irc_ros_description)/urdf/grippers/grippers.macro.xacro" />
+  <xacro:gripper prefix="$(arg prefix)" gripper_type="$(arg gripper)" parent_link="$(arg prefix)flange" />
 </robot>
