Commit message: Reordered urdfs, divided urdfs into macros

File: irc_ros_description/urdf/cpr_platform_medium.urdf.xacro (robot description, xacro)
@@ -8,6 +8,5 @@
   <xacro:arg name="use_cri" default="false"/>
   <xacro:arg name="prefix" default="" />
-  <xacro:include filename="$(find irc_ros_description)/urdf/din_rail_module.ros2_control.xacro" />
-  <xacro:include filename="$(find irc_ros_description)/urdf/cpr_platform_medium.xacro" />
-  <xacro:include filename="$(find irc_ros_description)/urdf/cpr_platform_medium.ros2_control.xacro" />
+  <xacro:include filename="$(find irc_ros_description)/urdf/platforms/cpr_platform_medium.macro.xacro" />
+  <xacro:cpr_platform_medium prefix="${prefix}" />
 </robot>

File: irc_ros_description/urdf/grippers/ext_dio_gripper.ros2_control.xacro (robot description, xacro)
@@ -3,9 +3,9 @@
 <ros2_control name="gripper_ext_dio_gripper" type="system">
   <hardware>
-    <!-- Only works via CAN -->
+    <!-- This gripper only works via CAN -->
     <plugin>irc_hardware/IrcRosCan</plugin>
     <param name="can_socket">can0</param>
   </hardware>
-  <gpio name="$(arg prefix)dio_ext">
+  <gpio name="${prefix}dio_ext">
     <param name="can_id">0x90</param>
     <command_interface name="digital_output" size="7" data_type="bool" />

File: irc_ros_description/urdf/grippers/ext_dio_gripper.urdf.xacro (robot description, xacro)
@@ -1,5 +1,5 @@
 <?xml version="1.0"?>
 <robot xmlns:xacro="http://www.ros.org/wiki/xacro"
-       name="cpr_platform_medium" >
+       name="gripper_ext_dio_gripper" >
   <xacro:include filename="$(find irc_ros_description)/urdf/gripper_ext_dio_gripper.xacro" />
   <xacro:include filename="$(find irc_ros_description)/urdf/gripper_ext_dio_gripper.ros2_control.xacro" />

File: irc_ros_description/urdf/grippers/none.urdf.xacro (robot description, xacro)
@@ -1,2 +1,3 @@
+<?xml version="1.0"?>
 <!-- Nearly empty file to enable including no gripper via -->
 <!-- <xacro:include filename="$(find irc_ros_description)/urdf/gripper_$(arg gripper).urdf.xacro" /> -->

File: irc_ros_description/urdf/grippers/schmalz_ecbpmi.urdf.xacro (robot description, xacro)
@@ -1,5 +1,5 @@
 <?xml version="1.0"?>
 <robot xmlns:xacro="http://www.ros.org/wiki/xacro"
-    name="gripper_ext_dio_gripper">
+       name="gripper_schmalz_ecbpmi">
   <link name="$(arg prefix)gripper_mount">
     <visual>

File: irc_ros_description/urdf/igus_rebel_4dof.urdf.xacro (robot description, xacro)
@@ -2,5 +2,5 @@
 <robot xmlns:xacro="http://www.ros.org/wiki/xacro"
        name="igus_rebel_4dof" >
-  <!-- Controller settings -->
+  <!-- Controller settings, only enable a single one in the launch file -->
   <xacro:arg name="use_mock_hardware" default="false"/>
   <xacro:arg name="use_gazebo" default="false"/>
@@ -8,8 +8,8 @@
   <xacro:arg name="use_cri" default="false"/>
   <xacro:include filename="$(find irc_ros_description)/urdf/rebel_joint.ros2_control.xacro" />
-  <!-- (Internal) hardware selection  -->
+  <!-- Rebel version selection  -->
   <xacro:arg name="rebel_version" default="01" />
   <!-- Gripper selection -->
-  <xacro:arg name="gripper" default="schmalz_ecbpmi" />
+  <xacro:arg name="gripper" default="none" />
   <!-- Enable continuous rotation on the last join. While the last axis can turn continuously,
   it is limited here in case a tool with wiring is mounted. If you are certain that no wiring

File: irc_ros_description/urdf/igus_rebel_6dof.urdf.xacro (robot description, xacro)
@@ -2,37 +2,37 @@
 <robot xmlns:xacro="http://www.ros.org/wiki/xacro"
        name="igus_rebel_6dof" >
-  <!-- Controller settings -->
+  <!-- Controller settings, only enable a single one in the launch file -->
   <xacro:arg name="use_mock_hardware" default="false"/>
   <xacro:arg name="use_gazebo" default="false"/>
   <xacro:arg name="use_cprcanv2" default="false"/>
   <xacro:arg name="use_cri" default="false"/>
-  <xacro:include filename="$(find irc_ros_description)/urdf/rebel_joint.ros2_control.xacro" />
-  <!-- (Internal) hardware selection  -->
-  <xacro:arg name="rebel_version" default="00" />
-  <!-- Gripper selection -->
-  <xacro:arg name="gripper" default="none" />
+  <!-- Rebel version selection  -->
+  <xacro:arg name="rebel_version" default="01" />
   <!-- Enable continuous rotation on the last join. While the last axis can turn continuously,
   it is limited here in case a tool with wiring is mounted. If you are certain that no wiring
   issues can arise you may enable this -->
   <xacro:arg name="continuous_last_joint" default="false" />
-  <!-- TODO -->
-  <xacro:arg name="root_link" default="false" />
+  <!-- Prefix used for all joints and links, required for multi-robot setups!
+  Only change this over the launch file parameters, so the rest of the stack
+  knows what joint names to look for. -->
   <xacro:arg name="prefix" default="" />
-  <xacro:include filename="$(find irc_ros_description)/urdf/igus_rebel_6dof_$(arg rebel_version).xacro" />
-  <xacro:include filename="$(find irc_ros_description)/urdf/igus_rebel_6dof_$(arg rebel_version).ros2_control.xacro" />
-  <xacro:if value="$(arg root_link)">
-    <link name="world" />
-    <joint name="world_joint" type="fixed">
-      <parent link="world" />
-      <child link = "$(arg prefix)base_link" />
-      <origin xyz="0.0 0.0 0.0" rpy="0.0 0.0 0.0" />
-    </joint>
-  </xacro:if>
+  <!-- Gripper selection -->
+  <xacro:arg name="gripper" default="none" />
+  <!-- Include and call relevant macro -->
+  <xacro:include filename="$(find irc_ros_description)/urdf/robots/igus_rebel_6dof.macro.xacro" />
+  <xacro:igus_rebel_6dof prefix="$(arg prefix)" continuous_last_joint="$(arg continuous_last_joint)" rebel_version="'$(arg rebel_version)'" />
+  <!-- Add world link -->
+  <link name="world" />
+  <joint name="world_to_$(arg prefix)base" type="fixed">
+    <parent link="world" />
+    <child link = "$(arg prefix)base_link" />
+    <origin xyz="0.0 0.0 0.0" rpy="0.0 0.0 0.0" />
+  </joint>
   <!-- Grippers -->
-  <joint name="$(arg prefix)hand_to_gripper" type="fixed">
-    <parent link="$(arg prefix)hand" />
+  <xacro:include filename="$(find irc_ros_description)/urdf/grippers/$(arg gripper).urdf.xacro" />
+  <joint name="$(arg prefix)flange_to_gripper" type="fixed">
+    <parent link="$(arg prefix)flange" />
     <child link = "$(arg prefix)gripper_mount" />
     <origin xyz="0.0 0.0 0.0" rpy="0.0 ${-pi/2} 0.0" />
   </joint>
-  <xacro:include filename="$(find irc_ros_description)/urdf/gripper_$(arg gripper).urdf.xacro" />
 </robot>

File: irc_ros_description/urdf/igus_robolink_rl_dp_5.urdf.xacro (robot description, xacro)
@@ -7,17 +7,20 @@
   <xacro:arg name="use_cprcanv2" default="false"/>
   <xacro:arg name="use_cri" default="false"/>
-  <xacro:include filename="$(find irc_ros_description)/urdf/din_rail_module.ros2_control.xacro" />
-  <!-- Gripper selection -->
-  <xacro:arg name="use_gripper" default="false" />
-  <xacro:arg name="gripper" default="schmalz_ecbpmi" />
   <!-- Enable continuous rotation on the last join. While the last axis can turn continuously,
   it is limited here in case a tool with wiring is mounted. If you are certain that no wiring
   issues can arise you may enable this -->
   <xacro:arg name="continuous_last_joint" default="false" />
+  <!-- Prefix used for all joints and links, required for multi-robot setups!
+  Only change this over the launch file parameters, so the rest of the stack
+  knows what joint names to look for. -->
   <xacro:arg name="prefix" default="" />
-  <xacro:include filename="$(find irc_ros_description)/urdf/igus_robolink_rl_dp_5.xacro" />
-  <xacro:include filename="$(find irc_ros_description)/urdf/igus_robolink_rl_dp_5.ros2_control.xacro" />
+  <!-- Gripper selection -->
+  <xacro:arg name="gripper" default="none" />
+  <!-- Include and call relevant macro -->
+  <xacro:include filename="$(find irc_ros_description)/urdf/robots/igus_robolink_rl_dp_5.macro.xacro" />
+  <xacro:igus_robolink_rl_dp_5 prefix="$(arg prefix)" continuous_last_joint="$(arg continuous_last_joint)" />
+  <!-- Add world link -->
   <link name="world" />
-  <joint name="world_joint" type="fixed">
+  <joint name="world_to_$(arg prefix)base" type="fixed">
     <parent link="world" />
     <child link = "$(arg prefix)base_link" />
@@ -25,11 +28,9 @@
   </joint>
   <!-- Grippers -->
-  <xacro:if value="$(arg use_gripper)">
-    <joint name="$(arg prefix)hand_to_gripper" type="fixed">
-      <parent link="$(arg prefix)hand" />
-      <child link = "$(arg prefix)gripper_mount" />
-      <origin xyz="0.0 0.0 0.0" rpy="0.0 ${-pi/2} 0.0" />
-    </joint>
-    <xacro:include filename="$(find irc_ros_description)/urdf/gripper_$(arg gripper).urdf.xacro" />
-  </xacro:if>
+  <xacro:include filename="$(find irc_ros_description)/urdf/grippers/$(arg gripper).urdf.xacro" />
+  <joint name="$(arg prefix)flange_to_gripper" type="fixed">
+    <parent link="$(arg prefix)flange" />
+    <child link = "$(arg prefix)gripper_mount" />
+    <origin xyz="0.0 0.0 0.0" rpy="0.0 ${-pi/2} 0.0" />
+  </joint>
 </robot>

File: irc_ros_description/urdf/modules/din_rail.ros2_control.xacro (robot description, xacro)
@@ -19,5 +19,5 @@
       <param name="gear_scale">${gear_scale}</param>
       <param name="controller_type">open_loop</param>
-      <param name="referencing_required">"${referencing_required}"</param>
+      <param name="referencing_required">${referencing_required}</param>
       <param name="referencing_priority">${referencing_priority}</param>
     </joint>

File: irc_ros_description/urdf/rebel_on_platform.urdf.xacro (robot description, xacro)
@@ -2,6 +2,13 @@
 <robot xmlns:xacro="http://www.ros.org/wiki/xacro"
        name="rebel_on_platform" >
-  <xacro:include filename="$(find irc_ros_description)/urdf/igus_rebel_6dof.urdf.xacro" prefix="rebel_1_" />
-  <xacro:include filename="$(find irc_ros_description)/urdf/cpr_platform_medium.urdf.xacro" prefix=""/>
+  <!-- Controller settings -->
+  <xacro:arg name="use_mock_hardware" default="false"/>
+  <xacro:arg name="use_gazebo" default="false"/>
+  <xacro:arg name="use_cprcanv2" default="false"/>
+  <xacro:arg name="use_cri" default="false"/>
+  <xacro:include filename="$(find irc_ros_description)/urdf/robots/igus_rebel_6dof.macro.xacro"/>
+  <xacro:include filename="$(find irc_ros_description)/urdf/platforms/cpr_platform_medium.macro.xacro"/>
+  <xacro:igus_rebel_6dof prefix="rebel_1_" rebel_version="01" />
+  <xacro:cpr_platform_medium prefix="" />
   <joint name="platform_to_rebel" type="fixed">
     <parent link="base_link" />

File: irc_ros_description/urdf/robots/igus_rebel_4dof_01.description.xacro (robot description, xacro)
@@ -1,4 +1,5 @@
 <?xml version="1.0" ?>
-<robot xmlns:xacro="http://www.ros.org/wiki/xacro">
+<robot xmlns:xacro="http://www.ros.org/wiki/xacro"
+       name="igus_rebel_4dof" >
 <xacro:include filename="$(find irc_ros_description)/urdf/igus_rebel_6dof_00.xacro" />
 </robot>
