Commit message: Fix errors caused by new macros

File: irc_ros_description/urdf/cpr_platform_medium.urdf.xacro (robot description, xacro)
@@ -3,10 +3,7 @@
        name="cpr_platform_medium" >
   <!-- Controller settings -->
-  <xacro:arg name="use_mock_hardware" default="false"/>
-  <xacro:arg name="use_gazebo" default="false"/>
-  <xacro:arg name="use_cprcanv2" default="false"/>
-  <xacro:arg name="use_cri" default="false"/>
+  <xacro:arg name="controller_type" default="mock_hardware"/>
   <xacro:arg name="prefix" default="" />
   <xacro:include filename="$(find irc_ros_description)/urdf/platforms/cpr_platform_medium.macro.xacro" />
-  <xacro:cpr_platform_medium prefix="$(arg prefix)" />
+  <xacro:cpr_platform_medium prefix="$(arg prefix)" controller_type="$(arg controller_type)" />
 </robot>

File: irc_ros_description/urdf/igus_rebel_4dof.urdf.xacro (robot description, xacro)
@@ -3,9 +3,5 @@
        name="igus_rebel_4dof" >
   <!-- Controller settings, only enable a single one in the launch file -->
-  <xacro:arg name="use_mock_hardware" default="false"/>
-  <xacro:arg name="use_gazebo" default="false"/>
-  <xacro:arg name="use_cprcanv2" default="false"/>
-  <xacro:arg name="use_cri" default="false"/>
-  <xacro:include filename="$(find irc_ros_description)/urdf/rebel_joint.ros2_control.xacro" />
+  <xacro:arg name="controller_type" default="mock_hardware"/>
   <!-- Rebel version selection  -->
   <xacro:arg name="rebel_version" default="01" />
@@ -16,11 +12,16 @@
   issues can arise you may enable this -->
   <xacro:arg name="continuous_last_joint" default="false" />
-  <!-- TODO -->
-  <xacro:arg name="root_link" default="false" />
+  <!-- Prefix used for all joints and links, required for multi-robot setups!
+  Only change this over the launch file parameters, so the rest of the stack
+  knows what joint names to look for. -->
   <xacro:arg name="prefix" default="" />
-  <xacro:include filename="$(find irc_ros_description)/urdf/igus_rebel_4dof_$(arg rebel_version).xacro" />
-  <xacro:include filename="$(find irc_ros_description)/urdf/igus_rebel_4dof_$(arg rebel_version).ros2_control.xacro" />
+  <!-- Gripper selection -->
+  <xacro:arg name="gripper" default="none" />
+  <!-- Include and call relevant macro -->
+  <xacro:include filename="$(find irc_ros_description)/urdf/robots/igus_rebel_4dof.macro.xacro" />
+  <xacro:igus_rebel_4dof prefix="$(arg prefix)" continuous_last_joint="$(arg continuous_last_joint)" rebel_version="'$(arg rebel_version)'" controller_type="$(arg controller_type)" />
+  <!-- Add world link -->
   <link name="world" />
-  <joint name="world_joint" type="fixed">
+  <joint name="world_to_$(arg prefix)base" type="fixed">
     <parent link="world" />
     <child link = "$(arg prefix)base_link" />
@@ -28,9 +29,9 @@
   </joint>
   <!-- Grippers -->
-  <joint name="$(arg prefix)hand_to_gripper" type="fixed">
-    <parent link="$(arg prefix)hand" />
+  <xacro:include filename="$(find irc_ros_description)/urdf/grippers/$(arg gripper).urdf.xacro" />
+  <joint name="$(arg prefix)flange_to_gripper" type="fixed">
+    <parent link="$(arg prefix)flange" />
     <child link = "$(arg prefix)gripper_mount" />
     <origin xyz="0.0 0.0 0.0" rpy="0.0 ${-pi/2} 0.0" />
   </joint>
-  <xacro:include filename="$(find irc_ros_description)/urdf/gripper_$(arg gripper).urdf.xacro" />
 </robot>

File: irc_ros_description/urdf/igus_rebel_6dof.urdf.xacro (robot description, xacro)
@@ -3,8 +3,5 @@
        name="igus_rebel_6dof" >
   <!-- Controller settings, only enable a single one in the launch file -->
-  <xacro:arg name="use_mock_hardware" default="false"/>
-  <xacro:arg name="use_gazebo" default="false"/>
-  <xacro:arg name="use_cprcanv2" default="false"/>
-  <xacro:arg name="use_cri" default="false"/>
+  <xacro:arg name="controller_type" default="mock_hardware"/>
   <!-- Rebel version selection  -->
   <xacro:arg name="rebel_version" default="01" />
@@ -21,5 +18,5 @@
   <!-- Include and call relevant macro -->
   <xacro:include filename="$(find irc_ros_description)/urdf/robots/igus_rebel_6dof.macro.xacro" />
-  <xacro:igus_rebel_6dof prefix="$(arg prefix)" continuous_last_joint="$(arg continuous_last_joint)" rebel_version="'$(arg rebel_version)'" />
+  <xacro:igus_rebel_6dof prefix="$(arg prefix)" continuous_last_joint="$(arg continuous_last_joint)" rebel_version="'$(arg rebel_version)'" controller_type="$(arg controller_type)" />
   <!-- Add world link -->
   <link name="world" />

File: irc_ros_description/urdf/igus_robolink_rl_dp_5.urdf.xacro (robot description, xacro)
@@ -3,8 +3,5 @@
        name="igus_robolink_rl_dp_5" >
   <!-- Controller settings -->
-  <xacro:arg name="use_mock_hardware" default="false"/>
-  <xacro:arg name="use_gazebo" default="false"/>
-  <xacro:arg name="use_cprcanv2" default="false"/>
-  <xacro:arg name="use_cri" default="false"/>
+  <xacro:arg name="controller_type" default="mock_hardware"/>
   <!-- Enable continuous rotation on the last join. While the last axis can turn continuously,
   it is limited here in case a tool with wiring is mounted. If you are certain that no wiring
@@ -19,5 +16,5 @@
   <!-- Include and call relevant macro -->
   <xacro:include filename="$(find irc_ros_description)/urdf/robots/igus_robolink_rl_dp_5.macro.xacro" />
-  <xacro:igus_robolink_rl_dp_5 prefix="$(arg prefix)" continuous_last_joint="$(arg continuous_last_joint)" />
+  <xacro:igus_robolink_rl_dp_5 prefix="$(arg prefix)" continuous_last_joint="$(arg continuous_last_joint)" controller_type="$(arg controller_type)"/>
   <!-- Add world link -->
   <link name="world" />

File: irc_ros_description/urdf/platforms/cpr_platform_medium.macro.xacro (robot description, xacro)
@@ -5,8 +5,8 @@
   <xacro:include filename="$(find irc_ros_description)/urdf/platforms/cpr_platform_medium.description.xacro" />
   <xacro:include filename="$(find irc_ros_description)/urdf/platforms/cpr_platform_medium.ros2_control.xacro" />
-  <xacro:macro name="cpr_platform_medium" params="prefix">
+  <xacro:macro name="cpr_platform_medium" params="prefix controller_type">
     <!-- Call macros once -->
     <xacro:cpr_platform_medium_description prefix="${prefix}"/>
-    <xacro:cpr_platform_medium_ros2_control prefix="${prefix}" />
+    <xacro:cpr_platform_medium_ros2_control prefix="${prefix}" controller_type="${controller_type}"/>
   </xacro:macro>
 </robot>

File: irc_ros_description/urdf/platforms/cpr_platform_medium.ros2_control.xacro (robot description, xacro)
@@ -1,19 +1,19 @@
 <?xml version="1.0" ?>
 <robot xmlns:xacro="http://www.ros.org/wiki/xacro">
-  <xacro:macro name="cpr_platform_medium_ros2_control" params="prefix">
+  <xacro:macro name="cpr_platform_medium_ros2_control" params="prefix controller_type">
     <ros2_control name="cpr_platform_medium" type="system">
       <hardware>
-        <xacro:if value="$(arg use_mock_hardware)">
+        <xacro:if value="${controller_type == 'mock_hardware'}">
           <plugin>mock_components/GenericSystem</plugin>
         </xacro:if>
-        <xacro:if value="$(arg use_gazebo)">
+        <xacro:if value="${controller_type == 'gazebo'}">
             <plugin>gazebo_ros2_control/GazeboSystem</plugin>
         </xacro:if>
-        <xacro:unless value="$(arg use_mock_hardware)">
-          <xacro:if value="$(arg use_cprcanv2)">
+        <xacro:unless value="${controller_type == 'mock_hardware'}">
+          <xacro:if value="${controller_type == 'cprcanv2'}">
             <plugin>irc_hardware/IrcRosCan</plugin>
             <param name="can_socket">can0</param>
           </xacro:if>
-          <xacro:if value="$(arg use_cri)">
+          <xacro:if value="${controller_type == 'cri'}">
             <plugin>irc_hardware/IrcRosCri</plugin>
             <param name="ip">192.168.3.11</param>

File: irc_ros_description/urdf/rebel_on_platform.urdf.xacro (robot description, xacro)
@@ -3,12 +3,13 @@
        name="rebel_on_platform" >
   <!-- Controller settings -->
-  <xacro:arg name="use_mock_hardware" default="false"/>
-  <xacro:arg name="use_gazebo" default="false"/>
-  <xacro:arg name="use_cprcanv2" default="false"/>
-  <xacro:arg name="use_cri" default="false"/>
+  <xacro:arg name="controller_type" default="mock_hardware"/>
+  <!-- Enable continuous rotation on the last join. While the last axis can turn continuously,
+  it is limited here in case a tool with wiring is mounted. If you are certain that no wiring
+  issues can arise you may enable this -->
+  <xacro:arg name="continuous_last_joint" default="false" />
   <xacro:include filename="$(find irc_ros_description)/urdf/robots/igus_rebel_6dof.macro.xacro"/>
   <xacro:include filename="$(find irc_ros_description)/urdf/platforms/cpr_platform_medium.macro.xacro"/>
-  <xacro:igus_rebel_6dof prefix="rebel_1_" rebel_version="01" />
-  <xacro:cpr_platform_medium prefix="" />
+  <xacro:cpr_platform_medium prefix="" controller_type="$(arg controller_type)" />
+  <xacro:igus_rebel_6dof prefix="rebel_1_" continuous_last_joint="$(arg continuous_last_joint)" rebel_version="'00'"  controller_type="$(arg controller_type)" />
   <joint name="platform_to_rebel" type="fixed">
     <parent link="base_link" />

File: irc_ros_description/urdf/robots/igus_rebel_4dof.macro.xacro (robot description, xacro)
@@ -2,11 +2,19 @@
 <robot xmlns:xacro="http://www.ros.org/wiki/xacro"
        name="igus_rebel_4dof" >
-  <xacro:macro name="igus_rebel_4dof" params="prefix continuous_last_joint=false rebel_version=01">
-    <!-- Include relevant macros -->
-    <xacro:include filename="$(find irc_ros_description)/urdf/robots/igus_rebel_4dof_${rebel_version}.description.xacro" />
-    <xacro:include filename="$(find irc_ros_description)/urdf/robots/igus_rebel_4dof_${rebel_version}.ros2_control.xacro" />
+  <!-- Include all igus_rebel_4dof macros -->
+  <xacro:include filename="$(find irc_ros_description)/urdf/robots/igus_rebel_4dof_00.description.xacro" />
+  <xacro:include filename="$(find irc_ros_description)/urdf/robots/igus_rebel_4dof_00.ros2_control.xacro" />
+  <xacro:include filename="$(find irc_ros_description)/urdf/robots/igus_rebel_4dof_01.description.xacro" />
+  <xacro:include filename="$(find irc_ros_description)/urdf/robots/igus_rebel_4dof_01.ros2_control.xacro" />
+  <xacro:macro name="igus_rebel_4dof" params="prefix controller_type continuous_last_joint=false rebel_version">
     <!-- Call macros once -->
-    <xacro:igus_rebel_4dof prefix="${prefix}" continuous_last_joint="${continuous_last_joint}" />
-    <xacro:igus_rebel_4dof prefix="${prefix}" continuous_last_joint="${continuous_last_joint}" />
+    <xacro:if value="${rebel_version == '00'}">
+      <xacro:igus_rebel_4dof_00_description prefix="${prefix}" continuous_last_joint="${continuous_last_joint}" />
+      <xacro:igus_rebel_4dof_00_ros2_control prefix="${prefix}" controller_type="${controller_type}" continuous_last_joint="${continuous_last_joint}" />
+    </xacro:if>
+    <xacro:if value="${rebel_version == '01'}">
+      <xacro:igus_rebel_4dof_00_description prefix="${prefix}" continuous_last_joint="${continuous_last_joint}" />
+      <xacro:igus_rebel_4dof_01_ros2_control prefix="${prefix}" controller_type="${controller_type}" continuous_last_joint="${continuous_last_joint}" />
+    </xacro:if>
   </xacro:macro>
 </robot>

File: irc_ros_description/urdf/robots/igus_rebel_4dof_00.description.xacro (robot description, xacro)
@@ -94,5 +94,5 @@
       </inertial>
     </link>
-    <xacro:if value="$(arg continuous_last_joint)">
+    <xacro:if value="${continuous_last_joint}">
       <joint name="${prefix}joint4" type="continuous">
         <parent link="${prefix}link_3"/>
@@ -103,5 +103,5 @@
       </joint>
     </xacro:if>
-    <xacro:unless value="$(arg continuous_last_joint)">
+    <xacro:unless value="${continuous_last_joint}">
       <joint name="${prefix}joint4" type="revolute">
         <parent link="${prefix}link_3"/>
@@ -132,9 +132,9 @@
     <joint name="${prefix}joint5" type="fixed">
       <parent link="${prefix}link_4"/>
-      <child link="${prefix}hand"/>
+      <child link="${prefix}flange"/>
       <origin rpy="0.0 0.0 0.0" xyz="0.0 0.0 0.062"/>
       <axis xyz="0 -1 0"/>
     </joint>
-    <link name="${prefix}hand">
+    <link name="${prefix}flange">
       <inertial>
         <mass value="0.1"/>

File: irc_ros_description/urdf/robots/igus_rebel_4dof_00.ros2_control.xacro (robot description, xacro)
@@ -1,19 +1,19 @@
 <?xml version="1.0" ?>
 <robot xmlns:xacro="http://www.ros.org/wiki/xacro">
-  <xacro:macro name="igus_rebel_4dof_00_ros2_control" params="prefix continuous_last_joint">
+  <xacro:macro name="igus_rebel_4dof_00_ros2_control" params="prefix controller_type continuous_last_joint">
     <ros2_control name="igus_rebel_4dof" type="system">
       <hardware>
-        <xacro:if value="$(arg use_mock_hardware)">
+        <xacro:if value="${controller_type == 'mock_hardware'}">
           <plugin>mock_components/GenericSystem</plugin>
         </xacro:if>
-        <xacro:if value="$(arg use_gazebo)">
+        <xacro:if value="${controller_type == 'gazebo'}">
             <plugin>gazebo_ros2_control/GazeboSystem</plugin>
         </xacro:if>
-        <xacro:unless value="$(arg use_mock_hardware)">
-          <xacro:if value="$(arg use_cprcanv2)">
+        <xacro:unless value="${controller_type == 'mock_hardware'}">
+          <xacro:if value="${controller_type == 'cprcanv2'}">
             <plugin>irc_hardware/IrcRosCan</plugin>
             <param name="can_socket">can0</param>
           </xacro:if>
-          <xacro:if value="$(arg use_cri)">
+          <xacro:if value="${controller_type == 'cri'}">
             <plugin>irc_hardware/IrcRosCri</plugin>
             <param name="ip">192.168.3.11</param>
@@ -27,5 +27,5 @@
       <xacro:rebel_joint name="${prefix}joint2" can_id="0x20" position_min="${-pi*2/3}" position_max="${pi*2/3}" gear_scale="1031.11" />
       <xacro:rebel_joint name="${prefix}joint3" can_id="0x30" position_min="${-pi*2/3}" position_max="${pi*2/3}" gear_scale="1031.11" />
-      <xacro:rebel_joint name="${prefix}joint4" can_id="0x40" position_min="${-pi*19/36}" position_max="${pi*19/36}" gear_scale="1031.11" continuous_last_joint="$(arg continuous_last_joint)" />
+      <xacro:rebel_joint name="${prefix}joint4" can_id="0x40" position_min="${-pi*19/36}" position_max="${pi*19/36}" gear_scale="1031.11" continuous_joint="${continuous_last_joint}" />
       <gpio name="${prefix}dio_base">
         <param name="can_id">0x70</param>

File: irc_ros_description/urdf/robots/igus_rebel_4dof_01.description.xacro (robot description, xacro)
@@ -2,4 +2,4 @@
 <robot xmlns:xacro="http://www.ros.org/wiki/xacro"
        name="igus_rebel_4dof" >
-<xacro:include filename="$(find irc_ros_description)/urdf/igus_rebel_6dof_00.xacro" />
+<xacro:include filename="$(find irc_ros_description)/urdf/robots/igus_rebel_4dof_00.description.xacro" />
 </robot>

File: irc_ros_description/urdf/robots/igus_rebel_4dof_01.ros2_control.xacro (robot description, xacro)
@@ -1,19 +1,19 @@
 <?xml version="1.0" ?>
 <robot xmlns:xacro="http://www.ros.org/wiki/xacro">
-  <xacro:macro name="igus_rebel_4dof_01_ros2_control" params="prefix continuous_last_joint">
+  <xacro:macro name="igus_rebel_4dof_01_ros2_control" params="prefix controller_type continuous_last_joint">
     <ros2_control name="igus_rebel_4dof" type="system">
       <hardware>
-        <xacro:if value="$(arg use_mock_hardware)">
+        <xacro:if value="${controller_type == 'mock_hardware'}">
           <plugin>mock_components/GenericSystem</plugin>
         </xacro:if>
-        <xacro:if value="$(arg use_gazebo)">
+        <xacro:if value="${controller_type == 'gazebo'}">
             <plugin>gazebo_ros2_control/GazeboSystem</plugin>
         </xacro:if>
-        <xacro:unless value="$(arg use_mock_hardware)">
-          <xacro:if value="$(arg use_cprcanv2)">
+        <xacro:unless value="${controller_type == 'mock_hardware'}">
+          <xacro:if value="${controller_type == 'cprcanv2'}">
             <plugin>irc_hardware/IrcRosCan</plugin>
             <param name="can_socket">can0</param>
           </xacro:if>
-          <xacro:if value="$(arg use_cri)">
+          <xacro:if value="${controller_type == 'cri'}">
             <plugin>irc_hardware/IrcRosCri</plugin>
             <param name="ip">192.168.3.11</param>
@@ -26,5 +26,5 @@
       <xacro:rebel_joint name="${prefix}joint2" can_id="0x20" position_min="${-pi*2/3}" position_max="${pi*2/3}" gear_scale="1443.55" />
       <xacro:rebel_joint name="${prefix}joint3" can_id="0x30" position_min="${-pi*2/3}" position_max="${pi*2/3}" gear_scale="1443.55" />
-      <xacro:rebel_joint name="${prefix}joint4" can_id="0x40" position_min="${-pi*19/36}" position_max="${pi*19/36}" gear_scale="1031.11" continuous_joint="$(arg continuous_last_joint)" />
+      <xacro:rebel_joint name="${prefix}joint4" can_id="0x40" position_min="${-pi*19/36}" position_max="${pi*19/36}" gear_scale="1031.11" continuous_joint="${continuous_last_joint}" />
       <gpio name="${prefix}dio_base">
         <param name="can_id">0x70</param>

File: irc_ros_description/urdf/robots/igus_rebel_6dof.macro.xacro (robot description, xacro)
@@ -9,17 +9,17 @@
   <xacro:include filename="$(find irc_ros_description)/urdf/robots/igus_rebel_6dof_01.description.xacro" />
   <xacro:include filename="$(find irc_ros_description)/urdf/robots/igus_rebel_6dof_01.ros2_control.xacro" />
-  <xacro:macro name="igus_rebel_6dof" params="prefix continuous_last_joint=false rebel_version">
+  <xacro:macro name="igus_rebel_6dof" params="prefix controller_type continuous_last_joint=false rebel_version">
     <!-- Call macros once -->
     <xacro:if value="${rebel_version == 'pre'}">
       <xacro:igus_rebel_6dof_pre_description prefix="${prefix}" continuous_last_joint="${continuous_last_joint}" />
-      <xacro:igus_rebel_6dof_pre_ros2_control prefix="${prefix}" continuous_last_joint="${continuous_last_joint}" />
+      <xacro:igus_rebel_6dof_pre_ros2_control prefix="${prefix}" controller_type="${controller_type}" continuous_last_joint="${continuous_last_joint}" />
     </xacro:if>
     <xacro:if value="${rebel_version == '00'}">
       <xacro:igus_rebel_6dof_00_description prefix="${prefix}" continuous_last_joint="${continuous_last_joint}" />
-      <xacro:igus_rebel_6dof_00_ros2_control prefix="${prefix}" continuous_last_joint="${continuous_last_joint}" />
+      <xacro:igus_rebel_6dof_00_ros2_control prefix="${prefix}" controller_type="${controller_type}" continuous_last_joint="${continuous_last_joint}" />
     </xacro:if>
     <xacro:if value="${rebel_version == '01'}">
       <xacro:igus_rebel_6dof_00_description prefix="${prefix}" continuous_last_joint="${continuous_last_joint}" />
-      <xacro:igus_rebel_6dof_01_ros2_control prefix="${prefix}" continuous_last_joint="${continuous_last_joint}" />
+      <xacro:igus_rebel_6dof_01_ros2_control prefix="${prefix}" controller_type="${controller_type}" continuous_last_joint="${continuous_last_joint}" />
     </xacro:if>
   </xacro:macro>

File: irc_ros_description/urdf/robots/igus_rebel_6dof_00.description.xacro (robot description, xacro)
@@ -146,5 +146,5 @@
       </inertial>
     </link>
-    <xacro:if value="$(arg continuous_last_joint)">
+    <xacro:if value="${continuous_last_joint}">
     <joint name="${prefix}joint6" type="continuous">
         <parent link="${prefix}link_7"/>
@@ -155,5 +155,5 @@
       </joint>
     </xacro:if>
-    <xacro:unless value="$(arg continuous_last_joint)">
+    <xacro:unless value="${continuous_last_joint}">
       <joint name="${prefix}joint6" type="revolute">
         <parent link="${prefix}link_7"/>

File: irc_ros_description/urdf/robots/igus_rebel_6dof_00.ros2_control.xacro (robot description, xacro)
@@ -1,19 +1,19 @@
 <?xml version="1.0" ?>
 <robot xmlns:xacro="http://www.ros.org/wiki/xacro">
-  <xacro:macro name="igus_rebel_6dof_00_ros2_control" params="prefix continuous_last_joint">
+  <xacro:macro name="igus_rebel_6dof_00_ros2_control" params="prefix controller_type continuous_last_joint">
     <ros2_control name="igus_rebel_6dof" type="system">
       <hardware>
-        <xacro:if value="$(arg use_mock_hardware)">
+        <xacro:if value="${controller_type == 'mock_hardware'}">
           <plugin>mock_components/GenericSystem</plugin>
         </xacro:if>
-        <xacro:if value="$(arg use_gazebo)">
+        <xacro:if value="${controller_type == 'gazebo'}">
             <plugin>gazebo_ros2_control/GazeboSystem</plugin>
         </xacro:if>
-        <xacro:unless value="$(arg use_mock_hardware)">
-          <xacro:if value="$(arg use_cprcanv2)">
+        <xacro:unless value="${controller_type == 'mock_hardware'}">
+          <xacro:if value="${controller_type == 'cprcanv2'}">
             <plugin>irc_hardware/IrcRosCan</plugin>
             <param name="can_socket">can0</param>
           </xacro:if>
-          <xacro:if value="$(arg use_cri)">
+          <xacro:if value="${controller_type == 'cri'}">
             <plugin>irc_hardware/IrcRosCri</plugin>
             <param name="ip">192.168.3.11</param>
@@ -29,5 +29,5 @@
       <xacro:rebel_joint name="${prefix}joint4" can_id="0x40" position_min="${-pi*179/180}" position_max="${pi*179/180}" gear_scale="-1031.11" />
       <xacro:rebel_joint name="${prefix}joint5" can_id="0x50" position_min="${-pi*19/36}" position_max="${pi*19/36}" gear_scale="1031.11" />
-      <xacro:rebel_joint name="${prefix}joint6" can_id="0x60" position_min="${-pi*179/180}" position_max="${pi*179/180}" gear_scale="-1031.11" continuous_joint="$(arg continuous_last_joint)" />
+      <xacro:rebel_joint name="${prefix}joint6" can_id="0x60" position_min="${-pi*179/180}" position_max="${pi*179/180}" gear_scale="-1031.11" continuous_joint="${continuous_last_joint}" />
       <gpio name="${prefix}dio_base">
         <param name="can_id">0x70</param>
