Commit message: Fix errors caused by new macros

File: irc_ros_description/urdf/robots/igus_rebel_6dof_01.ros2_control.xacro (robot description, xacro)
@@ -1,19 +1,19 @@
 <?xml version="1.0" ?>
 <robot xmlns:xacro="http://www.ros.org/wiki/xacro">
-  <xacro:macro name="igus_rebel_6dof_01_ros2_control" params="prefix continuous_last_joint">
+  <xacro:macro name="igus_rebel_6dof_01_ros2_control" params="prefix controller_type continuous_last_joint">
     <ros2_control name="igus_rebel_6dof" type="system">
       <hardware>
-        <xacro:if value="$(arg use_mock_hardware)">
+        <xacro:if value="${controller_type == 'mock_hardware'}">
           <plugin>mock_components/GenericSystem</plugin>
         </xacro:if>
-        <xacro:if value="$(arg use_gazebo)">
+        <xacro:if value="${controller_type == 'gazebo'}">
             <plugin>gazebo_ros2_control/GazeboSystem</plugin>
         </xacro:if>
-        <xacro:unless value="$(arg use_mock_hardware)">
-          <xacro:if value="$(arg use_cprcanv2)">
+        <xacro:unless value="${controller_type == 'mock_hardware'}">
+          <xacro:if value="${controller_type == 'cprcanv2'}">
             <plugin>irc_hardware/IrcRosCan</plugin>
             <param name="can_socket">can0</param>
           </xacro:if>
-          <xacro:if value="$(arg use_cri)">
+          <xacro:if value="${controller_type == 'cri'}">
             <plugin>irc_hardware/IrcRosCri</plugin>
             <param name="ip">192.168.3.11</param>
@@ -29,5 +29,5 @@
       <xacro:rebel_joint name="${prefix}joint4" can_id="0x40" position_min="${-pi*179/180}" position_max="${pi*179/180}" gear_scale="-1443.55" />
       <xacro:rebel_joint name="${prefix}joint5" can_id="0x50" position_min="${-pi*19/36}" position_max="${pi*19/36}" gear_scale="1031.11" />
-      <xacro:rebel_joint name="${prefix}joint6" can_id="0x60" position_min="${-pi*179/180}" position_max="${pi*179/180}" gear_scale="-1031.11" continuous_joint="$(arg continuous_last_joint)" />
+      <xacro:rebel_joint name="${prefix}joint6" can_id="0x60" position_min="${-pi*179/180}" position_max="${pi*179/180}" gear_scale="-1031.11" continuous_joint="${continuous_last_joint}" />
       <gpio name="${prefix}dio_base">
         <param name="can_id">0x70</param>

File: irc_ros_description/urdf/robots/igus_rebel_6dof_pre.description.xacro (robot description, xacro)
@@ -146,5 +146,5 @@
       </inertial>
     </link>
-    <xacro:if value="$(arg continuous_last_joint)">
+    <xacro:if value="${continuous_last_joint}">
       <joint name="${prefix}joint6" type="continuous">
         <parent link="${prefix}link_7"/>
@@ -155,5 +155,5 @@
       </joint>
     </xacro:if>
-    <xacro:unless value="$(arg continuous_last_joint)">
+    <xacro:unless value="${continuous_last_joint}">
       <joint name="${prefix}joint6" type="revolute">
         <parent link="${prefix}link_7"/>

File: irc_ros_description/urdf/robots/igus_rebel_6dof_pre.ros2_control.xacro (robot description, xacro)
@@ -1,19 +1,19 @@
 <?xml version="1.0" ?>
 <robot xmlns:xacro="http://www.ros.org/wiki/xacro">
-  <xacro:macro name="igus_rebel_6dof_pre_ros2_control" params="prefix continuous_last_joint">
+  <xacro:macro name="igus_rebel_6dof_pre_ros2_control" params="prefix controller_type continuous_last_joint">
     <ros2_control name="igus_rebel_6dof" type="system">
       <hardware>
-        <xacro:if value="$(arg use_mock_hardware)">
+        <xacro:if value="${controller_type == 'mock_hardware'}">
           <plugin>mock_components/GenericSystem</plugin>
         </xacro:if>
-        <xacro:if value="$(arg use_gazebo)">
+        <xacro:if value="${controller_type == 'gazebo'}">
             <plugin>gazebo_ros2_control/GazeboSystem</plugin>
         </xacro:if>
-        <xacro:unless value="$(arg use_mock_hardware)">
-          <xacro:if value="$(arg use_cprcanv2)">
+        <xacro:unless value="${controller_type == 'mock_hardware'}">
+          <xacro:if value="${controller_type == 'cprcanv2'}">
             <plugin>irc_hardware/IrcRosCan</plugin>
             <param name="can_socket">can0</param>
           </xacro:if>
-          <xacro:if value="$(arg use_cri)">
+          <xacro:if value="${controller_type == 'cri'}">
             <plugin>irc_hardware/IrcRosCri</plugin>
             <param name="ip">192.168.3.11</param>
@@ -28,5 +28,5 @@
       <xacro:rebel_joint name="${prefix}joint4" can_id="0x40" position_min="${-pi*179/180}" position_max="${pi*179/180}" gear_scale="-1031.11" />
       <xacro:rebel_joint name="${prefix}joint5" can_id="0x50" position_min="${-pi*19/36}" position_max="${pi*19/36}" gear_scale="1031.11" />
-      <xacro:rebel_joint name="${prefix}joint6" can_id="0x60" position_min="${-pi*179/180}" position_max="${pi*179/180}" gear_scale="-1031.11" continuous_joint="$(arg continuous_last_joint)" />
+      <xacro:rebel_joint name="${prefix}joint6" can_id="0x60" position_min="${-pi*179/180}" position_max="${pi*179/180}" gear_scale="-1031.11" continuous_joint="${continuous_last_joint}" />
       <!-- Pre version does not have GPIOs -->
     </ros2_control>

File: irc_ros_description/urdf/robots/igus_robolink_rl_dp_5.description.xacro (robot description, xacro)
@@ -119,5 +119,5 @@
       </inertial>
     </link>
-    <xacro:if value="$(arg continuous_last_joint)">
+    <xacro:if value="${continuous_last_joint}">
       <joint name="${prefix}joint5" type="continuous">
         <parent link="${prefix}link_6"/>
@@ -128,5 +128,5 @@
       </joint>
     </xacro:if>
-    <xacro:unless value="$(arg continuous_last_joint)">
+    <xacro:unless value="${continuous_last_joint}">
       <joint name="${prefix}joint5" type="revolute">
         <parent link="${prefix}link_6"/>

File: irc_ros_description/urdf/robots/igus_robolink_rl_dp_5.macro.xacro (robot description, xacro)
@@ -5,8 +5,8 @@
   <xacro:include filename="$(find irc_ros_description)/urdf/robots/igus_robolink_rl_dp_5.description.xacro" />
   <xacro:include filename="$(find irc_ros_description)/urdf/robots/igus_robolink_rl_dp_5.ros2_control.xacro" />
-  <xacro:macro name="igus_robolink_rl_dp_5" params="prefix continuous_last_joint=false">
+  <xacro:macro name="igus_robolink_rl_dp_5" params="prefix controller_type continuous_last_joint=false">
     <!-- Call macros once -->
     <xacro:igus_robolink_rl_dp_5_description prefix="${prefix}" continuous_last_joint="${continuous_last_joint}" />
-    <xacro:igus_robolink_rl_dp_5_ros2_control prefix="${prefix}" continuous_last_joint="${continuous_last_joint}" />
+    <xacro:igus_robolink_rl_dp_5_ros2_control prefix="${prefix}" controller_type="${controller_type}" continuous_last_joint="${continuous_last_joint}" />
   </xacro:macro>
 </robot>
