Commit message: renamed controller_type to hardware_protocol

File: irc_ros_description/urdf/cpr_platform_medium.urdf.xacro (robot description, xacro)
@@ -3,7 +3,7 @@
        name="cpr_platform_medium" >
   <!-- Controller settings -->
-  <xacro:arg name="controller_type" default="cprcanv2"/>
+  <xacro:arg name="hardware_protocol" default="cprcanv2"/>
   <xacro:arg name="prefix" default="" />
   <xacro:include filename="$(find irc_ros_description)/urdf/platforms/cpr_platform_medium.macro.xacro" />
-  <xacro:cpr_platform_medium prefix="$(arg prefix)" controller_type="$(arg controller_type)" />
+  <xacro:cpr_platform_medium prefix="$(arg prefix)" hardware_protocol="$(arg hardware_protocol)" />
 </robot>

File: irc_ros_description/urdf/igus_rebel_4dof.urdf.xacro (robot description, xacro)
@@ -3,5 +3,5 @@
        name="igus_rebel_4dof" >
   <!-- Controller settings, only enable a single one in the launch file -->
-  <xacro:arg name="controller_type" default="cprcanv2"/>
+  <xacro:arg name="hardware_protocol" default="cprcanv2"/>
   <!-- Rebel version selection  -->
   <xacro:arg name="rebel_version" default="01" />
@@ -20,5 +20,5 @@
   <!-- Include and call relevant macro -->
   <xacro:include filename="$(find irc_ros_description)/urdf/robots/igus_rebel_4dof.macro.xacro" />
-  <xacro:igus_rebel_4dof prefix="$(arg prefix)" continuous_last_joint="$(arg continuous_last_joint)" rebel_version="'$(arg rebel_version)'" controller_type="$(arg controller_type)" />
+  <xacro:igus_rebel_4dof prefix="$(arg prefix)" continuous_last_joint="$(arg continuous_last_joint)" rebel_version="'$(arg rebel_version)'" hardware_protocol="$(arg hardware_protocol)" />
   <!-- Add world link -->
   <link name="world" />

File: irc_ros_description/urdf/igus_rebel_6dof.urdf.xacro (robot description, xacro)
@@ -3,5 +3,5 @@
        name="igus_rebel_6dof" >
   <!-- Controller settings, only enable a single one in the launch file -->
-  <xacro:arg name="controller_type" default="cprcanv2"/>
+  <xacro:arg name="hardware_protocol" default="cprcanv2"/>
   <!-- Rebel version selection  -->
   <xacro:arg name="rebel_version" default="01" />
@@ -18,5 +18,5 @@
   <!-- Include and call rebel macro -->
   <xacro:include filename="$(find irc_ros_description)/urdf/robots/igus_rebel_6dof.macro.xacro" />
-  <xacro:igus_rebel_6dof prefix="$(arg prefix)" continuous_last_joint="$(arg continuous_last_joint)" rebel_version="'$(arg rebel_version)'" controller_type="$(arg controller_type)" />
+  <xacro:igus_rebel_6dof prefix="$(arg prefix)" continuous_last_joint="$(arg continuous_last_joint)" rebel_version="'$(arg rebel_version)'" hardware_protocol="$(arg hardware_protocol)" />
   <!-- Add world link -->
   <link name="world" />

File: irc_ros_description/urdf/igus_robolink_rl_dp_5.urdf.xacro (robot description, xacro)
@@ -3,5 +3,5 @@
        name="igus_robolink_rl_dp_5" >
   <!-- Controller settings -->
-  <xacro:arg name="controller_type" default="cprcanv2"/>
+  <xacro:arg name="hardware_protocol" default="cprcanv2"/>
   <!-- Enable continuous rotation on the last join. While the last axis can turn continuously,
   it is limited here in case a tool with wiring is mounted. If you are certain that no wiring
@@ -16,5 +16,5 @@
   <!-- Include and call relevant macro -->
   <xacro:include filename="$(find irc_ros_description)/urdf/robots/igus_robolink_rl_dp_5.macro.xacro" />
-  <xacro:igus_robolink_rl_dp_5 prefix="$(arg prefix)" continuous_last_joint="$(arg continuous_last_joint)" controller_type="$(arg controller_type)"/>
+  <xacro:igus_robolink_rl_dp_5 prefix="$(arg prefix)" continuous_last_joint="$(arg continuous_last_joint)" hardware_protocol="$(arg hardware_protocol)"/>
   <!-- Add world link -->
   <link name="world" />

File: irc_ros_description/urdf/modules/din_rail.ros2_control.xacro (robot description, xacro)
@@ -18,5 +18,5 @@
       <param name="can_id">${can_id}</param>
       <param name="gear_scale">${gear_scale}</param>
-      <param name="controller_type">open_loop</param>
+      <param name="hardware_protocol">open_loop</param>
       <param name="referencing_required">${referencing_required}</param>
       <param name="referencing_priority">${referencing_priority}</param>

File: irc_ros_description/urdf/modules/rebel.ros2_control.xacro (robot description, xacro)
@@ -18,5 +18,5 @@
       <param name="can_id">${can_id}</param>
       <param name="gear_scale">${gear_scale}</param>
-      <param name="controller_type">closed_loop</param>
+      <param name="hardware_protocol">closed_loop</param>
     </joint>
   </xacro:macro>

File: irc_ros_description/urdf/platforms/cpr_platform_medium.macro.xacro (robot description, xacro)
@@ -5,8 +5,8 @@
   <xacro:include filename="$(find irc_ros_description)/urdf/platforms/cpr_platform_medium.description.xacro" />
   <xacro:include filename="$(find irc_ros_description)/urdf/platforms/cpr_platform_medium.ros2_control.xacro" />
-  <xacro:macro name="cpr_platform_medium" params="prefix controller_type">
+  <xacro:macro name="cpr_platform_medium" params="prefix hardware_protocol">
     <!-- Call macros once -->
     <xacro:cpr_platform_medium_description prefix="${prefix}"/>
-    <xacro:cpr_platform_medium_ros2_control prefix="${prefix}" controller_type="${controller_type}"/>
+    <xacro:cpr_platform_medium_ros2_control prefix="${prefix}" hardware_protocol="${hardware_protocol}"/>
   </xacro:macro>
 </robot>

File: irc_ros_description/urdf/platforms/cpr_platform_medium.ros2_control.xacro (robot description, xacro)
@@ -1,19 +1,19 @@
 <?xml version="1.0" ?>
 <robot xmlns:xacro="http://www.ros.org/wiki/xacro">
-  <xacro:macro name="cpr_platform_medium_ros2_control" params="prefix controller_type">
+  <xacro:macro name="cpr_platform_medium_ros2_control" params="prefix hardware_protocol">
     <ros2_control name="cpr_platform_medium" type="system">
       <hardware>
-        <xacro:if value="${controller_type == 'mock_hardware'}">
+        <xacro:if value="${hardware_protocol == 'mock_hardware'}">
           <plugin>mock_components/GenericSystem</plugin>
         </xacro:if>
-        <xacro:if value="${controller_type == 'gazebo'}">
+        <xacro:if value="${hardware_protocol == 'gazebo'}">
             <plugin>gazebo_ros2_control/GazeboSystem</plugin>
         </xacro:if>
-        <xacro:unless value="${controller_type == 'mock_hardware'}">
-          <xacro:if value="${controller_type == 'cprcanv2'}">
+        <xacro:unless value="${hardware_protocol == 'mock_hardware'}">
+          <xacro:if value="${hardware_protocol == 'cprcanv2'}">
             <plugin>irc_hardware/IrcRosCan</plugin>
             <param name="can_socket">can0</param>
           </xacro:if>
-          <xacro:if value="${controller_type == 'cri'}">
+          <xacro:if value="${hardware_protocol == 'cri'}">
             <plugin>irc_hardware/IrcRosCri</plugin>
             <param name="ip">192.168.3.11</param>

File: irc_ros_description/urdf/rebel_on_platform.urdf.xacro (robot description, xacro)
@@ -3,5 +3,5 @@
        name="rebel_on_platform" >
   <!-- Controller settings -->
-  <xacro:arg name="controller_type" default="cprcanv2"/>
+  <xacro:arg name="hardware_protocol" default="cprcanv2"/>
   <!-- Enable continuous rotation on the last join. While the last axis can turn continuously,
   it is limited here in case a tool with wiring is mounted. If you are certain that no wiring
@@ -10,6 +10,6 @@
   <xacro:include filename="$(find irc_ros_description)/urdf/robots/igus_rebel_6dof.macro.xacro"/>
   <xacro:include filename="$(find irc_ros_description)/urdf/platforms/cpr_platform_medium.macro.xacro"/>
-  <xacro:cpr_platform_medium prefix="" controller_type="$(arg controller_type)" />
-  <xacro:igus_rebel_6dof prefix="rebel_1_" continuous_last_joint="$(arg continuous_last_joint)" rebel_version="'00'"  controller_type="$(arg controller_type)" />
+  <xacro:cpr_platform_medium prefix="" hardware_protocol="$(arg hardware_protocol)" />
+  <xacro:igus_rebel_6dof prefix="rebel_1_" continuous_last_joint="$(arg continuous_last_joint)" rebel_version="'00'"  hardware_protocol="$(arg hardware_protocol)" />
   <joint name="platform_to_rebel" type="fixed">
     <parent link="base_link" />

File: irc_ros_description/urdf/robots/igus_rebel_4dof.macro.xacro (robot description, xacro)
@@ -7,13 +7,13 @@
   <xacro:include filename="$(find irc_ros_description)/urdf/robots/igus_rebel_4dof_01.description.xacro" />
   <xacro:include filename="$(find irc_ros_description)/urdf/robots/igus_rebel_4dof_01.ros2_control.xacro" />
-  <xacro:macro name="igus_rebel_4dof" params="prefix controller_type continuous_last_joint=false rebel_version">
+  <xacro:macro name="igus_rebel_4dof" params="prefix hardware_protocol continuous_last_joint=false rebel_version">
     <!-- Call macros once -->
     <xacro:if value="${rebel_version == '00'}">
       <xacro:igus_rebel_4dof_00_description prefix="${prefix}" continuous_last_joint="${continuous_last_joint}" />
-      <xacro:igus_rebel_4dof_00_ros2_control prefix="${prefix}" controller_type="${controller_type}" continuous_last_joint="${continuous_last_joint}" />
+      <xacro:igus_rebel_4dof_00_ros2_control prefix="${prefix}" hardware_protocol="${hardware_protocol}" continuous_last_joint="${continuous_last_joint}" />
     </xacro:if>
     <xacro:if value="${rebel_version == '01'}">
       <xacro:igus_rebel_4dof_00_description prefix="${prefix}" continuous_last_joint="${continuous_last_joint}" />
-      <xacro:igus_rebel_4dof_01_ros2_control prefix="${prefix}" controller_type="${controller_type}" continuous_last_joint="${continuous_last_joint}" />
+      <xacro:igus_rebel_4dof_01_ros2_control prefix="${prefix}" hardware_protocol="${hardware_protocol}" continuous_last_joint="${continuous_last_joint}" />
     </xacro:if>
   </xacro:macro>

File: irc_ros_description/urdf/robots/igus_rebel_4dof_00.ros2_control.xacro (robot description, xacro)
@@ -1,19 +1,19 @@
 <?xml version="1.0" ?>
 <robot xmlns:xacro="http://www.ros.org/wiki/xacro">
-  <xacro:macro name="igus_rebel_4dof_00_ros2_control" params="prefix controller_type continuous_last_joint">
+  <xacro:macro name="igus_rebel_4dof_00_ros2_control" params="prefix hardware_protocol continuous_last_joint">
     <ros2_control name="igus_rebel_4dof" type="system">
       <hardware>
-        <xacro:if value="${controller_type == 'mock_hardware'}">
+        <xacro:if value="${hardware_protocol == 'mock_hardware'}">
           <plugin>mock_components/GenericSystem</plugin>
         </xacro:if>
-        <xacro:if value="${controller_type == 'gazebo'}">
+        <xacro:if value="${hardware_protocol == 'gazebo'}">
             <plugin>gazebo_ros2_control/GazeboSystem</plugin>
         </xacro:if>
-        <xacro:unless value="${controller_type == 'mock_hardware'}">
-          <xacro:if value="${controller_type == 'cprcanv2'}">
+        <xacro:unless value="${hardware_protocol == 'mock_hardware'}">
+          <xacro:if value="${hardware_protocol == 'cprcanv2'}">
             <plugin>irc_hardware/IrcRosCan</plugin>
             <param name="can_socket">can0</param>
           </xacro:if>
-          <xacro:if value="${controller_type == 'cri'}">
+          <xacro:if value="${hardware_protocol == 'cri'}">
             <plugin>irc_hardware/IrcRosCri</plugin>
             <param name="ip">192.168.3.11</param>

File: irc_ros_description/urdf/robots/igus_rebel_4dof_01.ros2_control.xacro (robot description, xacro)
@@ -1,19 +1,19 @@
 <?xml version="1.0" ?>
 <robot xmlns:xacro="http://www.ros.org/wiki/xacro">
-  <xacro:macro name="igus_rebel_4dof_01_ros2_control" params="prefix controller_type continuous_last_joint">
+  <xacro:macro name="igus_rebel_4dof_01_ros2_control" params="prefix hardware_protocol continuous_last_joint">
     <ros2_control name="igus_rebel_4dof" type="system">
       <hardware>
-        <xacro:if value="${controller_type == 'mock_hardware'}">
+        <xacro:if value="${hardware_protocol == 'mock_hardware'}">
           <plugin>mock_components/GenericSystem</plugin>
         </xacro:if>
-        <xacro:if value="${controller_type == 'gazebo'}">
+        <xacro:if value="${hardware_protocol == 'gazebo'}">
             <plugin>gazebo_ros2_control/GazeboSystem</plugin>
         </xacro:if>
-        <xacro:unless value="${controller_type == 'mock_hardware'}">
-          <xacro:if value="${controller_type == 'cprcanv2'}">
+        <xacro:unless value="${hardware_protocol == 'mock_hardware'}">
+          <xacro:if value="${hardware_protocol == 'cprcanv2'}">
             <plugin>irc_hardware/IrcRosCan</plugin>
             <param name="can_socket">can0</param>
           </xacro:if>
-          <xacro:if value="${controller_type == 'cri'}">
+          <xacro:if value="${hardware_protocol == 'cri'}">
             <plugin>irc_hardware/IrcRosCri</plugin>
             <param name="ip">192.168.3.11</param>

File: irc_ros_description/urdf/robots/igus_rebel_6dof.macro.xacro (robot description, xacro)
@@ -9,17 +9,17 @@
   <xacro:include filename="$(find irc_ros_description)/urdf/robots/igus_rebel_6dof_01.description.xacro" />
   <xacro:include filename="$(find irc_ros_description)/urdf/robots/igus_rebel_6dof_01.ros2_control.xacro" />
-  <xacro:macro name="igus_rebel_6dof" params="prefix controller_type continuous_last_joint=false rebel_version">
+  <xacro:macro name="igus_rebel_6dof" params="prefix hardware_protocol continuous_last_joint=false rebel_version">
     <!-- Call macros once -->
     <xacro:if value="${rebel_version == 'pre'}">
       <xacro:igus_rebel_6dof_pre_description prefix="${prefix}" continuous_last_joint="${continuous_last_joint}" />
-      <xacro:igus_rebel_6dof_pre_ros2_control prefix="${prefix}" controller_type="${controller_type}" continuous_last_joint="${continuous_last_joint}" />
+      <xacro:igus_rebel_6dof_pre_ros2_control prefix="${prefix}" hardware_protocol="${hardware_protocol}" continuous_last_joint="${continuous_last_joint}" />
     </xacro:if>
     <xacro:if value="${rebel_version == '00'}">
       <xacro:igus_rebel_6dof_00_description prefix="${prefix}" continuous_last_joint="${continuous_last_joint}" />
-      <xacro:igus_rebel_6dof_00_ros2_control prefix="${prefix}" controller_type="${controller_type}" continuous_last_joint="${continuous_last_joint}" />
+      <xacro:igus_rebel_6dof_00_ros2_control prefix="${prefix}" hardware_protocol="${hardware_protocol}" continuous_last_joint="${continuous_last_joint}" />
     </xacro:if>
     <xacro:if value="${rebel_version == '01'}">
       <xacro:igus_rebel_6dof_00_description prefix="${prefix}" continuous_last_joint="${continuous_last_joint}" />
-      <xacro:igus_rebel_6dof_01_ros2_control prefix="${prefix}" controller_type="${controller_type}" continuous_last_joint="${continuous_last_joint}" />
+      <xacro:igus_rebel_6dof_01_ros2_control prefix="${prefix}" hardware_protocol="${hardware_protocol}" continuous_last_joint="${continuous_last_joint}" />
     </xacro:if>
   </xacro:macro>

File: irc_ros_description/urdf/robots/igus_rebel_6dof_00.ros2_control.xacro (robot description, xacro)
@@ -1,19 +1,19 @@
 <?xml version="1.0" ?>
 <robot xmlns:xacro="http://www.ros.org/wiki/xacro">
-  <xacro:macro name="igus_rebel_6dof_00_ros2_control" params="prefix controller_type continuous_last_joint">
+  <xacro:macro name="igus_rebel_6dof_00_ros2_control" params="prefix hardware_protocol continuous_last_joint">
     <ros2_control name="igus_rebel_6dof" type="system">
       <hardware>
-        <xacro:if value="${controller_type == 'mock_hardware'}">
+        <xacro:if value="${hardware_protocol == 'mock_hardware'}">
           <plugin>mock_components/GenericSystem</plugin>
         </xacro:if>
-        <xacro:if value="${controller_type == 'gazebo'}">
+        <xacro:if value="${hardware_protocol == 'gazebo'}">
             <plugin>gazebo_ros2_control/GazeboSystem</plugin>
         </xacro:if>
-        <xacro:unless value="${controller_type == 'mock_hardware'}">
-          <xacro:if value="${controller_type == 'cprcanv2'}">
+        <xacro:unless value="${hardware_protocol == 'mock_hardware'}">
+          <xacro:if value="${hardware_protocol == 'cprcanv2'}">
             <plugin>irc_hardware/IrcRosCan</plugin>
             <param name="can_socket">can0</param>
           </xacro:if>
-          <xacro:if value="${controller_type == 'cri'}">
+          <xacro:if value="${hardware_protocol == 'cri'}">
             <plugin>irc_hardware/IrcRosCri</plugin>
             <param name="ip">192.168.3.11</param>

File: irc_ros_description/urdf/robots/igus_rebel_6dof_01.ros2_control.xacro (robot description, xacro)
@@ -1,19 +1,19 @@
 <?xml version="1.0" ?>
 <robot xmlns:xacro="http://www.ros.org/wiki/xacro">
-  <xacro:macro name="igus_rebel_6dof_01_ros2_control" params="prefix controller_type continuous_last_joint">
+  <xacro:macro name="igus_rebel_6dof_01_ros2_control" params="prefix hardware_protocol continuous_last_joint">
     <ros2_control name="igus_rebel_6dof" type="system">
       <hardware>
-        <xacro:if value="${controller_type == 'mock_hardware'}">
+        <xacro:if value="${hardware_protocol == 'mock_hardware'}">
           <plugin>mock_components/GenericSystem</plugin>
         </xacro:if>
-        <xacro:if value="${controller_type == 'gazebo'}">
+        <xacro:if value="${hardware_protocol == 'gazebo'}">
             <plugin>gazebo_ros2_control/GazeboSystem</plugin>
         </xacro:if>
-        <xacro:unless value="${controller_type == 'mock_hardware'}">
-          <xacro:if value="${controller_type == 'cprcanv2'}">
+        <xacro:unless value="${hardware_protocol == 'mock_hardware'}">
+          <xacro:if value="${hardware_protocol == 'cprcanv2'}">
             <plugin>irc_hardware/IrcRosCan</plugin>
             <param name="can_socket">can0</param>
           </xacro:if>
-          <xacro:if value="${controller_type == 'cri'}">
+          <xacro:if value="${hardware_protocol == 'cri'}">
             <plugin>irc_hardware/IrcRosCri</plugin>
             <param name="ip">192.168.3.11</param>

File: irc_ros_description/urdf/robots/igus_rebel_6dof_pre.ros2_control.xacro (robot description, xacro)
@@ -1,19 +1,19 @@
 <?xml version="1.0" ?>
 <robot xmlns:xacro="http://www.ros.org/wiki/xacro">
-  <xacro:macro name="igus_rebel_6dof_pre_ros2_control" params="prefix controller_type continuous_last_joint">
+  <xacro:macro name="igus_rebel_6dof_pre_ros2_control" params="prefix hardware_protocol continuous_last_joint">
     <ros2_control name="igus_rebel_6dof" type="system">
       <hardware>
-        <xacro:if value="${controller_type == 'mock_hardware'}">
+        <xacro:if value="${hardware_protocol == 'mock_hardware'}">
           <plugin>mock_components/GenericSystem</plugin>
         </xacro:if>
-        <xacro:if value="${controller_type == 'gazebo'}">
+        <xacro:if value="${hardware_protocol == 'gazebo'}">
             <plugin>gazebo_ros2_control/GazeboSystem</plugin>
         </xacro:if>
-        <xacro:unless value="${controller_type == 'mock_hardware'}">
-          <xacro:if value="${controller_type == 'cprcanv2'}">
+        <xacro:unless value="${hardware_protocol == 'mock_hardware'}">
+          <xacro:if value="${hardware_protocol == 'cprcanv2'}">
             <plugin>irc_hardware/IrcRosCan</plugin>
             <param name="can_socket">can0</param>
           </xacro:if>
-          <xacro:if value="${controller_type == 'cri'}">
+          <xacro:if value="${hardware_protocol == 'cri'}">
             <plugin>irc_hardware/IrcRosCri</plugin>
             <param name="ip">192.168.3.11</param>

File: irc_ros_description/urdf/robots/igus_robolink_rl_dp_5.macro.xacro (robot description, xacro)
@@ -5,8 +5,8 @@
   <xacro:include filename="$(find irc_ros_description)/urdf/robots/igus_robolink_rl_dp_5.description.xacro" />
   <xacro:include filename="$(find irc_ros_description)/urdf/robots/igus_robolink_rl_dp_5.ros2_control.xacro" />
-  <xacro:macro name="igus_robolink_rl_dp_5" params="prefix controller_type continuous_last_joint=false">
+  <xacro:macro name="igus_robolink_rl_dp_5" params="prefix hardware_protocol continuous_last_joint=false">
     <!-- Call macros once -->
     <xacro:igus_robolink_rl_dp_5_description prefix="${prefix}" continuous_last_joint="${continuous_last_joint}" />
-    <xacro:igus_robolink_rl_dp_5_ros2_control prefix="${prefix}" controller_type="${controller_type}" continuous_last_joint="${continuous_last_joint}" />
+    <xacro:igus_robolink_rl_dp_5_ros2_control prefix="${prefix}" hardware_protocol="${hardware_protocol}" continuous_last_joint="${continuous_last_joint}" />
   </xacro:macro>
 </robot>

File: irc_ros_description/urdf/robots/igus_robolink_rl_dp_5.ros2_control.xacro (robot description, xacro)
@@ -3,19 +3,19 @@
   <!-- Include the joint module macro -->
   <xacro:include filename="$(find irc_ros_description)/urdf/modules/din_rail.ros2_control.xacro" />
-  <xacro:macro name="igus_robolink_rl_dp_5_ros2_control" params="prefix controller_type continuous_last_joint">
+  <xacro:macro name="igus_robolink_rl_dp_5_ros2_control" params="prefix hardware_protocol continuous_last_joint">
     <ros2_control name="igus_robolink_rl_dp_5" type="system">
       <hardware>
-        <xacro:if value="${controller_type == 'mock_hardware'}">
+        <xacro:if value="${hardware_protocol == 'mock_hardware'}">
           <plugin>mock_components/GenericSystem</plugin>
         </xacro:if>
-        <xacro:if value="${controller_type == 'gazebo'}">
+        <xacro:if value="${hardware_protocol == 'gazebo'}">
             <plugin>gazebo_ros2_control/GazeboSystem</plugin>
         </xacro:if>
-        <xacro:unless value="${controller_type == 'mock_hardware'}">
-          <xacro:if value="${controller_type == 'cprcanv2'}">
+        <xacro:unless value="${hardware_protocol == 'mock_hardware'}">
+          <xacro:if value="${hardware_protocol == 'cprcanv2'}">
             <plugin>irc_hardware/IrcRosCan</plugin>
             <param name="can_socket">can0</param>
           </xacro:if>
-          <xacro:if value="${controller_type == 'cri'}">
+          <xacro:if value="${hardware_protocol == 'cri'}">
             <plugin>irc_hardware/IrcRosCri</plugin>
             <param name="ip">192.168.3.11</param>

File: irc_ros_moveit_config/config/igus_rebel_6dof.urdf.xacro (robot description, xacro)
@@ -3,5 +3,5 @@
        name="igus_rebel_6dof" >
   <!-- Controller settings -->
-  <xacro:arg name="controller_type" default="cprcanv2"/>
+  <xacro:arg name="hardware_protocol" default="cprcanv2"/>
   <!-- (Internal) hardware selection  -->
   <xacro:arg name="rebel_version" default="00" />
@@ -18,5 +18,5 @@
   <xacro:arg name="root_link" default="true" />
   <xacro:include filename="$(find irc_ros_description)/urdf/robots/igus_rebel_6dof.macro.xacro" />
-  <xacro:igus_rebel_6dof prefix="$(arg prefix)" continuous_last_joint="$(arg continuous_last_joint)" rebel_version="'$(arg rebel_version)'"  controller_type="$(arg controller_type)" />
+  <xacro:igus_rebel_6dof prefix="$(arg prefix)" continuous_last_joint="$(arg continuous_last_joint)" rebel_version="'$(arg rebel_version)'"  hardware_protocol="$(arg hardware_protocol)" />
   <xacro:if value="$(arg root_link)">
     <link name="world" />
