Commit message: Allow multi-robot setups (#51)
* Add prefixe and namespace support

* Change chassis to base_link for the platform

* Reordered urdfs, divided urdfs into macros

* Add new documentation for the urdf structure

* Change hand to flange link

* Add launch argument for controller type selection

* Simplified protocol selection

* Add namespace, prefix, controller_manager_name arguments

* Add prefix to controller config

* Combine laser scanner nodes into seperate launch file

File: irc_ros_description/urdf/cpr_platform_medium.urdf.xacro (robot description, xacro)
@@ -3,10 +3,7 @@
        name="cpr_platform_medium" >
   <!-- Controller settings -->
-  <xacro:arg name="use_mock_hardware" default="false"/>
-  <xacro:arg name="use_gazebo" default="false"/>
-  <xacro:arg name="use_cprcanv2" default="false"/>
-  <xacro:arg name="use_cri" default="false"/>
-  <xacro:include filename="$(find irc_ros_description)/urdf/din_rail_module.ros2_control.xacro" />
-  <xacro:include filename="$(find irc_ros_description)/urdf/cpr_platform_medium.xacro" />
-  <xacro:include filename="$(find irc_ros_description)/urdf/cpr_platform_medium.ros2_control.xacro" />
+  <xacro:arg name="hardware_protocol" default="cprcanv2"/>
+  <xacro:arg name="prefix" default="" />
+  <xacro:include filename="$(find irc_ros_description)/urdf/platforms/cpr_platform_medium.macro.xacro" />
+  <xacro:cpr_platform_medium prefix="$(arg prefix)" hardware_protocol="$(arg hardware_protocol)" />
 </robot>

File: irc_ros_description/urdf/igus_rebel_4dof.urdf.xacro (robot description, xacro)
@@ -2,34 +2,30 @@
 <robot xmlns:xacro="http://www.ros.org/wiki/xacro"
        name="igus_rebel_4dof" >
-  <!-- Controller settings -->
-  <xacro:arg name="use_mock_hardware" default="false"/>
-  <xacro:arg name="use_gazebo" default="false"/>
-  <xacro:arg name="use_cprcanv2" default="false"/>
-  <xacro:arg name="use_cri" default="false"/>
-  <xacro:include filename="$(find irc_ros_description)/urdf/rebel_joint.ros2_control.xacro" />
-  <!-- (Internal) hardware selection  -->
+  <!-- Controller settings, only enable a single one in the launch file -->
+  <xacro:arg name="hardware_protocol" default="cprcanv2"/>
+  <!-- Rebel version selection  -->
   <xacro:arg name="rebel_version" default="01" />
-  <!-- Gripper selection -->
-  <xacro:arg name="gripper" default="schmalz_ecbpmi" />
   <!-- Enable continuous rotation on the last join. While the last axis can turn continuously,
   it is limited here in case a tool with wiring is mounted. If you are certain that no wiring
   issues can arise you may enable this -->
   <xacro:arg name="continuous_last_joint" default="false" />
-  <!-- TODO -->
-  <xacro:arg name="root_link" default="false" />
-  <xacro:include filename="$(find irc_ros_description)/urdf/igus_rebel_4dof_$(arg rebel_version).xacro" />
-  <xacro:include filename="$(find irc_ros_description)/urdf/igus_rebel_4dof_$(arg rebel_version).ros2_control.xacro" />
+  <!-- Prefix used for all joints and links, required for multi-robot setups!
+  Only change this over the launch file parameters, so the rest of the stack
+  knows what joint names to look for. -->
+  <xacro:arg name="prefix" default="" />
+  <!-- Gripper selection -->
+  <xacro:arg name="gripper" default="none" />
+  <!-- Include and call relevant macro -->
+  <xacro:include filename="$(find irc_ros_description)/urdf/robots/igus_rebel_4dof.macro.xacro" />
+  <xacro:igus_rebel_4dof prefix="$(arg prefix)" continuous_last_joint="$(arg continuous_last_joint)" rebel_version="'$(arg rebel_version)'" hardware_protocol="$(arg hardware_protocol)" />
+  <!-- Add world link -->
   <link name="world" />
-  <joint name="world_joint" type="fixed">
+  <joint name="world_to_$(arg prefix)base" type="fixed">
     <parent link="world" />
-    <child link = "base_link" />
+    <child link = "$(arg prefix)base_link" />
     <origin xyz="0.0 0.0 0.0" rpy="0.0 0.0 0.0" />
   </joint>
   <!-- Grippers -->
-  <joint name="hand_to_gripper" type="fixed">
-    <parent link="hand" />
-    <child link = "gripper_mount" />
-    <origin xyz="0.0 0.0 0.0" rpy="0.0 ${-pi/2} 0.0" />
-  </joint>
-  <xacro:include filename="$(find irc_ros_description)/urdf/gripper_$(arg gripper).urdf.xacro" />
+  <xacro:include filename="$(find irc_ros_description)/urdf/grippers/grippers.macro.xacro" />
+  <xacro:gripper prefix="$(arg prefix)" gripper_type="$(arg gripper)" parent_link="$(arg prefix)flange" />
 </robot>

File: irc_ros_description/urdf/igus_rebel_6dof.urdf.xacro (robot description, xacro)
@@ -2,36 +2,30 @@
 <robot xmlns:xacro="http://www.ros.org/wiki/xacro"
        name="igus_rebel_6dof" >
-  <!-- Controller settings -->
-  <xacro:arg name="use_mock_hardware" default="false"/>
-  <xacro:arg name="use_gazebo" default="false"/>
-  <xacro:arg name="use_cprcanv2" default="false"/>
-  <xacro:arg name="use_cri" default="false"/>
-  <xacro:include filename="$(find irc_ros_description)/urdf/rebel_joint.ros2_control.xacro" />
-  <!-- (Internal) hardware selection  -->
-  <xacro:arg name="rebel_version" default="00" />
-  <!-- Gripper selection -->
-  <xacro:arg name="gripper" default="none" />
+  <!-- Controller settings, only enable a single one in the launch file -->
+  <xacro:arg name="hardware_protocol" default="cprcanv2"/>
+  <!-- Rebel version selection  -->
+  <xacro:arg name="rebel_version" default="01" />
   <!-- Enable continuous rotation on the last join. While the last axis can turn continuously,
   it is limited here in case a tool with wiring is mounted. If you are certain that no wiring
   issues can arise you may enable this -->
   <xacro:arg name="continuous_last_joint" default="false" />
-  <!-- TODO -->
-  <xacro:arg name="root_link" default="false" />
-  <xacro:include filename="$(find irc_ros_description)/urdf/igus_rebel_6dof_$(arg rebel_version).xacro" />
-  <xacro:include filename="$(find irc_ros_description)/urdf/igus_rebel_6dof_$(arg rebel_version).ros2_control.xacro" />
-  <xacro:if value="$(arg root_link)">
-    <link name="world" />
-    <joint name="world_joint" type="fixed">
-      <parent link="world" />
-      <child link = "base_link" />
-      <origin xyz="0.0 0.0 0.0" rpy="0.0 0.0 0.0" />
-    </joint>
-  </xacro:if>
+  <!-- Prefix used for all joints and links, required for multi-robot setups!
+  Only change this over the launch file parameters, so the rest of the stack
+  knows what joint names to look for. -->
+  <xacro:arg name="prefix" default="" />
+  <!-- Gripper selection -->
+  <xacro:arg name="gripper" default="none" />
+  <!-- Include and call rebel macro -->
+  <xacro:include filename="$(find irc_ros_description)/urdf/robots/igus_rebel_6dof.macro.xacro" />
+  <xacro:igus_rebel_6dof prefix="$(arg prefix)" continuous_last_joint="$(arg continuous_last_joint)" rebel_version="'$(arg rebel_version)'" hardware_protocol="$(arg hardware_protocol)" />
+  <!-- Add world link -->
+  <link name="world" />
+  <joint name="world_to_$(arg prefix)base" type="fixed">
+    <parent link="world" />
+    <child link = "$(arg prefix)base_link" />
+    <origin xyz="0.0 0.0 0.0" rpy="0.0 0.0 0.0" />
+  </joint>
   <!-- Grippers -->
-  <joint name="hand_to_gripper" type="fixed">
-    <parent link="hand" />
-    <child link = "gripper_mount" />
-    <origin xyz="0.0 0.0 0.0" rpy="0.0 ${-pi/2} 0.0" />
-  </joint>
-  <xacro:include filename="$(find irc_ros_description)/urdf/gripper_$(arg gripper).urdf.xacro" />
+  <xacro:include filename="$(find irc_ros_description)/urdf/grippers/grippers.macro.xacro" />
+  <xacro:gripper prefix="$(arg prefix)" gripper_type="$(arg gripper)" parent_link="$(arg prefix)flange" />
 </robot>

File: irc_ros_description/urdf/igus_robolink_rl_dp_5.urdf.xacro (robot description, xacro)
@@ -3,32 +3,27 @@
        name="igus_robolink_rl_dp_5" >
   <!-- Controller settings -->
-  <xacro:arg name="use_mock_hardware" default="false"/>
-  <xacro:arg name="use_gazebo" default="false"/>
-  <xacro:arg name="use_cprcanv2" default="false"/>
-  <xacro:arg name="use_cri" default="false"/>
-  <xacro:include filename="$(find irc_ros_description)/urdf/din_rail_module.ros2_control.xacro" />
-  <!-- Gripper selection -->
-  <xacro:arg name="use_gripper" default="false" />
-  <xacro:arg name="gripper" default="schmalz_ecbpmi" />
+  <xacro:arg name="hardware_protocol" default="cprcanv2"/>
   <!-- Enable continuous rotation on the last join. While the last axis can turn continuously,
   it is limited here in case a tool with wiring is mounted. If you are certain that no wiring
   issues can arise you may enable this -->
   <xacro:arg name="continuous_last_joint" default="false" />
-  <xacro:include filename="$(find irc_ros_description)/urdf/igus_robolink_rl_dp_5.xacro" />
-  <xacro:include filename="$(find irc_ros_description)/urdf/igus_robolink_rl_dp_5.ros2_control.xacro" />
+  <!-- Prefix used for all joints and links, required for multi-robot setups!
+  Only change this over the launch file parameters, so the rest of the stack
+  knows what joint names to look for. -->
+  <xacro:arg name="prefix" default="" />
+  <!-- Gripper selection -->
+  <xacro:arg name="gripper" default="none" />
+  <!-- Include and call relevant macro -->
+  <xacro:include filename="$(find irc_ros_description)/urdf/robots/igus_robolink_rl_dp_5.macro.xacro" />
+  <xacro:igus_robolink_rl_dp_5 prefix="$(arg prefix)" continuous_last_joint="$(arg continuous_last_joint)" hardware_protocol="$(arg hardware_protocol)"/>
+  <!-- Add world link -->
   <link name="world" />
-  <joint name="world_joint" type="fixed">
+  <joint name="world_to_$(arg prefix)base" type="fixed">
     <parent link="world" />
-    <child link = "base_link" />
+    <child link = "$(arg prefix)base_link" />
     <origin xyz="0.0 0.0 0.0" rpy="0.0 0.0 0.0" />
   </joint>
   <!-- Grippers -->
-  <xacro:if value="$(arg use_gripper)">
-    <joint name="hand_to_gripper" type="fixed">
-      <parent link="hand" />
-      <child link = "gripper_mount" />
-      <origin xyz="0.0 0.0 0.0" rpy="0.0 ${-pi/2} 0.0" />
-    </joint>
-    <xacro:include filename="$(find irc_ros_description)/urdf/gripper_$(arg gripper).urdf.xacro" />
-  </xacro:if>
+  <xacro:include filename="$(find irc_ros_description)/urdf/grippers/grippers.macro.xacro" />
+  <xacro:gripper prefix="$(arg prefix)" gripper_type="$(arg gripper)" parent_link="$(arg prefix)flange" />
 </robot>

File: irc_ros_description/urdf/modules/din_rail.ros2_control.xacro (robot description, xacro)
@@ -1,5 +1,5 @@
 <?xml version="1.0"?>
 <robot xmlns:xacro="http://www.ros.org/wiki/xacro">
-  <xacro:macro name="rebel_joint" params="name can_id position_min position_max gear_scale continuous_joint=false">
+  <xacro:macro name="din_rail_module" params="name can_id position_min=0 position_max=0 gear_scale continuous_joint=false referencing_required=false referencing_priority=0" >
     <joint name="${name}">
       <command_interface name="position">
@@ -18,5 +18,7 @@
       <param name="can_id">${can_id}</param>
       <param name="gear_scale">${gear_scale}</param>
-      <param name="controller_type">closed_loop</param>
+      <param name="controller_type">open_loop</param>
+      <param name="referencing_required">${referencing_required}</param>
+      <param name="referencing_priority">${referencing_priority}</param>
     </joint>
   </xacro:macro>

File: irc_ros_description/urdf/modules/rebel.ros2_control.xacro (robot description, xacro)
@@ -1,5 +1,5 @@
 <?xml version="1.0"?>
 <robot xmlns:xacro="http://www.ros.org/wiki/xacro">
-  <xacro:macro name="din_rail_module" params="name can_id position_min=0 position_max=0 gear_scale continuous_joint=false referencing_required=false referencing_priority=0" >
+  <xacro:macro name="rebel_joint" params="name can_id position_min=0 position_max=0 gear_scale=1 continuous_joint=false">
     <joint name="${name}">
       <command_interface name="position">
@@ -18,7 +18,5 @@
       <param name="can_id">${can_id}</param>
       <param name="gear_scale">${gear_scale}</param>
-      <param name="controller_type">open_loop</param>
-      <param name="referencing_required">"${referencing_required}"</param>
-      <param name="referencing_priority">${referencing_priority}</param>
+      <param name="controller_type">closed_loop</param>
     </joint>
   </xacro:macro>

File: irc_ros_description/urdf/rebel_on_platform.urdf.xacro (robot description, xacro)
@@ -2,9 +2,17 @@
 <robot xmlns:xacro="http://www.ros.org/wiki/xacro"
        name="rebel_on_platform" >
-  <xacro:include filename="$(find irc_ros_description)/urdf/igus_rebel_6dof.urdf.xacro"/>
-  <xacro:include filename="$(find irc_ros_description)/urdf/cpr_platform_medium.urdf.xacro"/>
+  <!-- Controller settings -->
+  <xacro:arg name="hardware_protocol" default="cprcanv2"/>
+  <!-- Enable continuous rotation on the last join. While the last axis can turn continuously,
+  it is limited here in case a tool with wiring is mounted. If you are certain that no wiring
+  issues can arise you may enable this -->
+  <xacro:arg name="continuous_last_joint" default="false" />
+  <xacro:include filename="$(find irc_ros_description)/urdf/robots/igus_rebel_6dof.macro.xacro"/>
+  <xacro:include filename="$(find irc_ros_description)/urdf/platforms/cpr_platform_medium.macro.xacro"/>
+  <xacro:cpr_platform_medium prefix="" hardware_protocol="$(arg hardware_protocol)" />
+  <xacro:igus_rebel_6dof prefix="rebel_1_" continuous_last_joint="$(arg continuous_last_joint)" rebel_version="'00'"  hardware_protocol="$(arg hardware_protocol)" />
   <joint name="platform_to_rebel" type="fixed">
-    <parent link="chassis" />
-    <child link = "base_link" />
+    <parent link="base_link" />
+    <child link="rebel_1_base_link" />
     <origin xyz="0.0 0.0 ${0.7-0.1}" rpy="0.0 0.0 ${-pi/6}" />
   </joint>

File: irc_ros_moveit_config/config/igus_rebel_6dof.urdf.xacro (robot description, xacro)
@@ -3,11 +3,11 @@
        name="igus_rebel_6dof" >
   <!-- Controller settings -->
-  <xacro:arg name="use_mock_hardware" default="false"/>
-  <xacro:arg name="use_gazebo" default="false"/>
-  <xacro:arg name="use_cprcanv2" default="true"/>  <!-- Default differs in this launch file -->
-  <xacro:arg name="use_cri" default="false"/>
-  <xacro:include filename="$(find irc_ros_description)/urdf/rebel_joint.ros2_control.xacro" />
+  <xacro:arg name="hardware_protocol" default="cprcanv2"/>
   <!-- (Internal) hardware selection  -->
   <xacro:arg name="rebel_version" default="00" />
+  <!-- Prefix used for all joints and links, required for multi-robot setups!
+  Only change this over the launch file parameters, so the rest of the stack
+  knows what joint names to look for. -->
+  <xacro:arg name="prefix" default="" />
   <!-- Gripper selection -->
   <xacro:arg name="gripper" default="none" />
@@ -17,6 +17,6 @@
   <xacro:arg name="continuous_last_joint" default="false" />
   <xacro:arg name="root_link" default="true" />
-  <xacro:include filename="$(find irc_ros_description)/urdf/igus_rebel_6dof_$(arg rebel_version).xacro" />
-  <xacro:include filename="$(find irc_ros_description)/urdf/igus_rebel_6dof_$(arg rebel_version).ros2_control.xacro" />
+  <xacro:include filename="$(find irc_ros_description)/urdf/robots/igus_rebel_6dof.macro.xacro" />
+  <xacro:igus_rebel_6dof prefix="$(arg prefix)" continuous_last_joint="$(arg continuous_last_joint)" rebel_version="'$(arg rebel_version)'"  hardware_protocol="$(arg hardware_protocol)" />
   <xacro:if value="$(arg root_link)">
     <link name="world" />
@@ -28,9 +28,5 @@
   </xacro:if>
   <!-- Grippers -->
-  <joint name="hand_to_gripper" type="fixed">
-    <parent link="hand" />
-    <child link = "gripper_mount" />
-    <origin xyz="0.0 0.0 0.0" rpy="0.0 ${-pi/2} 0.0" />
-  </joint>
-  <xacro:include filename="$(find irc_ros_description)/urdf/gripper_$(arg gripper).urdf.xacro" />
+  <xacro:include filename="$(find irc_ros_description)/urdf/grippers/grippers.macro.xacro" />
+  <xacro:gripper prefix="$(arg prefix)" gripper_type="$(arg gripper)" parent_link="$(arg prefix)flange" />
 </robot>
