Commit message: Remove rotational offset for rebel on platform

File: irc_ros_description/urdf/rebel_on_platform.urdf.xacro (robot description, xacro)
@@ -15,5 +15,5 @@
     <parent link="base_link" />
     <child link="rebel_1_base_link" />
-    <origin xyz="0.0 0.0 ${0.7-0.1}" rpy="0.0 0.0 ${-pi/6}" />
+    <origin xyz="0.0 0.0 ${0.7-0.1}" rpy="0.0 0.0 0.0" />
   </joint>
 </robot>
