Commit message: Rename joint from lidar_back to laser_back

File: irc_ros_description/urdf/platforms/cpr_platform_medium.description.xacro (robot description, xacro)
@@ -79,5 +79,5 @@
     <link name="${prefix}laser_front">
     </link>
-    <joint name="${prefix}joint_lidar_back" type="fixed">
+    <joint name="${prefix}joint_laser_back" type="fixed">
       <parent link="base_link"/>
       <child link="laser_back"/>

Commit message: Fix missing prefixes

File: irc_ros_description/urdf/platforms/cpr_platform_medium.description.xacro (robot description, xacro)
@@ -56,5 +56,5 @@
       <!-- <limit effort="330.0" lower="-3.12414" upper="3.12414" velocity="2.16"/> -->
     </joint>
-    <link name="wheel_2">
+    <link name="${prefix}wheel_2">
       <visual>
         <geometry>
@@ -80,6 +80,6 @@
     </link>
     <joint name="${prefix}joint_laser_back" type="fixed">
-      <parent link="base_link"/>
-      <child link="laser_back"/>
+      <parent link="${prefix}base_link"/>
+      <child link="${prefix}laser_back"/>
       <origin rpy="0.0 0.0 ${pi}" xyz="-0.54 0 0"/>
     </joint>
