Commit message: initial commit

File: irc_ros_description/urdf/platforms/cpr_platform_medium.ros2_control.xacro (robot description, xacro)
@@ -23,4 +23,37 @@
       <xacro:din_rail_module name="${prefix}joint_wheel_1" can_id="0x18" gear_scale="33.33" continuous_joint="true" />
       <xacro:din_rail_module name="${prefix}joint_wheel_2" can_id="0x28" gear_scale="-33.33" continuous_joint="true" />
+      <!-- Added for Dio Control for enable/reset -->
+      <gpio name="${prefix}dio_base">
+        <param name="can_id">0x70</param>
+        <command_interface name="digital_output_0" data_type="bool" />
+        <command_interface name="digital_output_1" data_type="bool" />
+        <command_interface name="digital_output_2" data_type="bool" />
+        <command_interface name="digital_output_3" data_type="bool" />
+        <command_interface name="digital_output_4" data_type="bool" />
+        <command_interface name="digital_output_5" data_type="bool" />
+        <command_interface name="digital_output_6" data_type="bool" />
+        <state_interface name="digital_input_0" data_type="bool" />
+        <state_interface name="digital_input_1" data_type="bool" />
+        <state_interface name="digital_input_2" data_type="bool" />
+        <state_interface name="digital_input_3" data_type="bool" />
+        <state_interface name="digital_input_4" data_type="bool" />
+        <state_interface name="digital_input_5" data_type="bool" />
+        <state_interface name="digital_input_6" data_type="bool" />
+      </gpio>
+      <!-- <gpio name="${prefix}enable">
+        <command_interface name="digital_output_enable" data_type="bool" />
+        <state_interface name="digital_input_enable" data_type="bool" />
+      </gpio>
+      <gpio name="${prefix}reset">
+        <command_interface name="digital_output_reset" data_type="bool" />
+        <state_interface name="digital_input_reset" data_type="bool" />
+      </gpio> -->
+      <!-- <gpio name="${prefix}dio_arm">
+        <param name="can_id">0x80</param>
+        <command_interface name="digital_output_0" data_type="bool" />
+        <command_interface name="digital_output_1" data_type="bool" />
+        <state_interface name="digital_input_0" data_type="bool" />
+        <state_interface name="digital_input_1" data_type="bool" />
+      </gpio> -->
     </ros2_control>
   </xacro:macro>

File: irc_ros_description/urdf/rebel_on_platform.urdf.xacro (robot description, xacro)
@@ -3,17 +3,18 @@
        name="rebel_on_platform" >
   <!-- Controller settings -->
-  <xacro:arg name="hardware_protocol" default="cprcanv2"/>
+  <xacro:arg name="hardware_protocol" default="cri"/>
+  <xacro:arg name="rebel_version" default="01" />
   <!-- Enable continuous rotation on the last join. While the last axis can turn continuously,
   it is limited here in case a tool with wiring is mounted. If you are certain that no wiring
   issues can arise you may enable this -->
   <xacro:arg name="continuous_last_joint" default="false" />
-  <xacro:include filename="$(find irc_ros_description)/urdf/robots/igus_rebel_6dof.macro.xacro"/>
-  <xacro:include filename="$(find irc_ros_description)/urdf/platforms/cpr_platform_medium.macro.xacro"/>
-  <xacro:cpr_platform_medium prefix="" hardware_protocol="$(arg hardware_protocol)" />
-  <xacro:igus_rebel_6dof prefix="rebel_1_" continuous_last_joint="$(arg continuous_last_joint)" rebel_version="'00'"  hardware_protocol="$(arg hardware_protocol)" />
-  <joint name="platform_to_rebel" type="fixed">
+  <xacro:arg name="prefix" default="" />
+  <xacro:arg name="gripper" default="none" />
+  <xacro:include filename="$(find irc_ros_description)/urdf/serviceRobots/rebel_on_platform.macro.xacro"/>
+  <xacro:rebel_on_platform prefix="" continuous_last_joint="$(arg continuous_last_joint)" rebel_version="'01'"  hardware_protocol="$(arg hardware_protocol)" />
+  <!-- <joint name="platform_to_rebel" type="fixed">
     <parent link="base_link" />
     <child link="rebel_1_base_link" />
     <origin xyz="0.0 0.0 ${0.7-0.1}" rpy="0.0 0.0 0.0" />
-  </joint>
+  </joint> -->
 </robot>
