Commit message: Add tcp joint for no gripper case

File: irc_ros_description/urdf/grippers/grippers.macro.xacro (robot description, xacro)
@@ -16,4 +16,17 @@
     </xacro:if>
     <xacro:if value="${gripper_type == 'none'}">
+      <!-- Make sure tcp exists even if no tool is attached -->
+      <joint name="${prefix}flange_to_tcp" type="fixed">
+        <parent link="${prefix}flange"/>
+        <child link="${prefix}tcp"/>
+        <origin rpy="0.0 0.0 0.0" xyz="0.0 0.0 0.0"/>
+        <axis xyz="0 0 0"/>
+      </joint>
+      <link name="${prefix}tcp">
+        <inertial>
+          <mass value="0.1"/>
+          <inertia ixx="0.03" ixy="0.0" ixz="0.0" iyy="0.03" iyz="0.0" izz="0.03"/>
+        </inertial>
+      </link>
     </xacro:if>
   </xacro:macro>
