Commit message: Add hardware_protocol arguments to gripper macros

File: irc_ros_description/urdf/grippers/ext_dio_gripper.ros2_control.xacro (robot description, xacro)
@@ -2,5 +2,5 @@
 <robot xmlns:xacro="http://www.ros.org/wiki/xacro"
        name="ext_dio_gripper">
-  <xacro:macro name="ext_dio_gripper_ros2_control" params="prefix parent_link">
+  <xacro:macro name="ext_dio_gripper_ros2_control" params="prefix parent_link hardware_protocol">
     <!-- This gripper only works via CAN -->
     <xacro:if value="${hardware_protocol == 'cprcanv2'}">

File: irc_ros_description/urdf/grippers/grippers.macro.xacro (robot description, xacro)
@@ -6,9 +6,9 @@
   <xacro:include filename="$(find irc_ros_description)/urdf/grippers/ext_dio_gripper.ros2_control.xacro" />
   <xacro:include filename="$(find irc_ros_description)/urdf/grippers/schmalz_ecbpmi.description.xacro" />
-  <xacro:macro name="gripper" params="prefix gripper_type parent_link">
+  <xacro:macro name="gripper" params="prefix gripper_type parent_link hardware_protocol">
     <!-- Call macros once -->
     <xacro:if value="${gripper_type == 'ext_dio_gripper'}">
       <xacro:ext_dio_gripper_description prefix="${prefix}" parent_link="${parent_link}" />
-      <xacro:ext_dio_gripper_ros2_control prefix="${prefix}" parent_link="${parent_link}" />
+      <xacro:ext_dio_gripper_ros2_control prefix="${prefix}" parent_link="${parent_link}" hardware_protocol="${hardware_protocol}" />
     </xacro:if>
     <xacro:if value="${gripper_type == 'schmalz_ecbpmi'}">

File: irc_ros_description/urdf/igus_rebel_4dof.urdf.xacro (robot description, xacro)
@@ -28,4 +28,4 @@
   <!-- Grippers -->
   <xacro:include filename="$(find irc_ros_description)/urdf/grippers/grippers.macro.xacro" />
-  <xacro:gripper prefix="$(arg prefix)" gripper_type="$(arg gripper)" parent_link="$(arg prefix)flange" />
+  <xacro:gripper prefix="$(arg prefix)" gripper_type="$(arg gripper)" parent_link="$(arg prefix)flange" hardware_protocol="$(arg hardware_protocol)" />
 </robot>

File: irc_ros_description/urdf/igus_rebel_6dof.urdf.xacro (robot description, xacro)
@@ -28,4 +28,4 @@
   <!-- Grippers -->
   <xacro:include filename="$(find irc_ros_description)/urdf/grippers/grippers.macro.xacro" />
-  <xacro:gripper prefix="$(arg prefix)" gripper_type="$(arg gripper)" parent_link="$(arg prefix)flange" />
+  <xacro:gripper prefix="$(arg prefix)" gripper_type="$(arg gripper)" parent_link="$(arg prefix)flange" hardware_protocol="$(arg hardware_protocol)" />
 </robot>

File: irc_ros_description/urdf/igus_robolink_rl_dp_5.urdf.xacro (robot description, xacro)
@@ -26,4 +26,4 @@
   <!-- Grippers -->
   <xacro:include filename="$(find irc_ros_description)/urdf/grippers/grippers.macro.xacro" />
-  <xacro:gripper prefix="$(arg prefix)" gripper_type="$(arg gripper)" parent_link="$(arg prefix)flange" />
+  <xacro:gripper prefix="$(arg prefix)" gripper_type="$(arg gripper)" parent_link="$(arg prefix)flange" hardware_protocol="$(arg hardware_protocol)" />
 </robot>

Commit message: Only start ros2_control part of ext_dio_gripper with CPRCANv2 (#92)

File: irc_ros_description/urdf/grippers/ext_dio_gripper.ros2_control.xacro (robot description, xacro)
@@ -2,17 +2,19 @@
 <robot xmlns:xacro="http://www.ros.org/wiki/xacro"
        name="ext_dio_gripper">
-  <xacro:macro name="ext_dio_gripper_ros2_control" params="prefix parent_link">
-    <ros2_control name="gripper_ext_dio_gripper" type="system">
-      <hardware>
-        <!-- This gripper only works via CAN -->
-        <plugin>irc_hardware/IrcRosCan</plugin>
-        <param name="can_socket">can0</param>
-      </hardware>
-      <gpio name="${prefix}dio_ext">
-        <param name="can_id">0x90</param>
-        <command_interface name="digital_output" size="7" data_type="bool" />
-        <state_interface name="digital_input" size="7" data_type="bool" />
-      </gpio>
-    </ros2_control>
+  <xacro:macro name="ext_dio_gripper_ros2_control" params="prefix parent_link hardware_protocol">
+    <!-- This gripper only works via CAN -->
+    <xacro:if value="${hardware_protocol == 'cprcanv2'}">
+      <ros2_control name="gripper_ext_dio_gripper" type="system">
+        <hardware>
+          <plugin>irc_hardware/IrcRosCan</plugin>
+          <param name="can_socket">can0</param>
+        </hardware>
+        <gpio name="${prefix}dio_ext">
+          <param name="can_id">0x90</param>
+          <command_interface name="digital_output" size="7" data_type="bool" />
+          <state_interface name="digital_input" size="7" data_type="bool" />
+        </gpio>
+      </ros2_control>
+    </xacro:if>
   </xacro:macro>
 </robot>
