Commit message: Create gripper macro

File: irc_ros_description/urdf/grippers/ext_dio_gripper.description.xacro (robot description, xacro)
@@ -2,5 +2,10 @@
 <robot xmlns:xacro="http://www.ros.org/wiki/xacro"
        name="gripper_ext_dio_gripper">
-  <xacro:macro name="gripper_ext_dio_gripper" params="prefix">
+  <xacro:macro name="ext_dio_gripper_description" params="prefix parent_link">
+    <joint name="${prefix}flange_to_gripper" type="fixed">
+      <parent link="${parent_link}" />
+      <child link = "${prefix}gripper_mount" />
+      <origin xyz="0.0 0.0 0.0" rpy="0.0 ${-pi/2} 0.0" />
+    </joint>
     <link name="${prefix}gripper_mount">
       <visual>

File: irc_ros_description/urdf/grippers/ext_dio_gripper.ros2_control.xacro (robot description, xacro)
@@ -1,15 +1,18 @@
 <?xml version="1.0" ?>
-<robot xmlns:xacro="http://www.ros.org/wiki/xacro">
-<ros2_control name="gripper_ext_dio_gripper" type="system">
-  <hardware>
-    <!-- This gripper only works via CAN -->
-    <plugin>irc_hardware/IrcRosCan</plugin>
-    <param name="can_socket">can0</param>
-  </hardware>
-  <gpio name="${prefix}dio_ext">
-    <param name="can_id">0x90</param>
-    <command_interface name="digital_output" size="7" data_type="bool" />
-    <state_interface name="digital_input" size="7" data_type="bool" />
-  </gpio>
-</ros2_control>
+<robot xmlns:xacro="http://www.ros.org/wiki/xacro"
+       name="ext_dio_gripper">
+  <xacro:macro name="ext_dio_gripper_ros2_control" params="prefix parent_link">
+    <ros2_control name="gripper_ext_dio_gripper" type="system">
+      <hardware>
+        <!-- This gripper only works via CAN -->
+        <plugin>irc_hardware/IrcRosCan</plugin>
+        <param name="can_socket">can0</param>
+      </hardware>
+      <gpio name="${prefix}dio_ext">
+        <param name="can_id">0x90</param>
+        <command_interface name="digital_output" size="7" data_type="bool" />
+        <state_interface name="digital_input" size="7" data_type="bool" />
+      </gpio>
+    </ros2_control>
+  </xacro:macro>
 </robot>

Commit message: Fix gripper coordinate system rotation

File: irc_ros_description/urdf/grippers/ext_dio_gripper.description.xacro (robot description, xacro)
@@ -36,5 +36,5 @@
           <mesh filename="package://irc_ros_description/meshes/gripper_schmalz_ecbpmi/Joint0.dae"/>
         </geometry>
-        <origin rpy="${pi/2} ${-pi/2} 0.0" xyz="0.07 0.0 0.0"/>
+        <origin rpy="0.0 0.0 0.0" xyz="0.07 0.0 0.0"/>
       </visual>
       <collision>
@@ -42,5 +42,6 @@
           <mesh filename="package://irc_ros_description/meshes/gripper_schmalz_ecbpmi/Joint0Coll.dae"/>
         </geometry>
-        <origin rpy="${pi/2} ${-pi/2} 0.0" xyz="0.07 0.0 0.0"/>
+        <origin rpy="0.0 0.0 0.0" xyz="0.07 0.0 0.0"/>
+      </visual>
       </collision>
       <inertial>
@@ -49,5 +50,5 @@
       </inertial>
     </link>
-    <joint name="${prefix}joint99" type="fixed">
+    <joint name="${prefix}gripper_base_to_tcp" type="fixed">
       <parent link="${prefix}gripper_base"/>
       <child link="${prefix}tcp"/>

File: irc_ros_description/urdf/grippers/schmalz_ecbpmi.description.xacro (robot description, xacro)
@@ -36,5 +36,5 @@
           <mesh filename="package://irc_ros_description/meshes/gripper_schmalz_ecbpmi/Joint0.dae"/>
         </geometry>
-        <origin rpy="${pi/2} ${-pi/2} 0.0" xyz="0.07 0.0 0.0"/>
+        <origin rpy="0.0 0.0 0.0" xyz="0.07 0.0 0.0"/>
       </visual>
       <collision>
@@ -42,5 +42,5 @@
           <mesh filename="package://irc_ros_description/meshes/gripper_schmalz_ecbpmi/Joint0Coll.dae"/>
         </geometry>
-        <origin rpy="${pi/2} ${-pi/2} 0.0" xyz="0.07 0.0 0.0"/>
+        <origin rpy="0.0 0.0 0.0" xyz="0.07 0.0 0.0"/>
       </collision>
       <inertial>
@@ -49,5 +49,5 @@
       </inertial>
     </link>
-    <joint name="${prefix}joint99" type="fixed">
+    <joint name="${prefix}gripper_base_to_tcp" type="fixed">
       <parent link="${prefix}gripper_base"/>
       <child link="${prefix}tcp"/>

Commit message: Fix missmatched blocks

File: irc_ros_description/urdf/grippers/ext_dio_gripper.description.xacro (robot description, xacro)
@@ -43,5 +43,4 @@
         </geometry>
         <origin rpy="0.0 0.0 0.0" xyz="0.07 0.0 0.0"/>
-      </visual>
       </collision>
       <inertial>

Commit message: Align grippers with new flange frame orientation

File: irc_ros_description/urdf/grippers/ext_dio_gripper.description.xacro (robot description, xacro)
@@ -6,5 +6,5 @@
       <parent link="${parent_link}" />
       <child link = "${prefix}gripper_mount" />
-      <origin xyz="0.0 0.0 0.0" rpy="0.0 ${-pi/2} 0.0" />
+      <origin xyz="0.0 0.0 0.0" rpy="0.0 0.0 0.0" />
     </joint>
     <link name="${prefix}gripper_mount">
@@ -13,5 +13,5 @@
           <cylinder radius="0.035" length="0.01"/>
         </geometry>
-        <origin rpy="0.0 ${-pi/2} 0.0" xyz="0.005 0.0 0.0"/>
+        <origin rpy="0.0 ${pi/2} 0.0" xyz="0.005 0.0 0.0"/>
       </visual>
       <collision>
@@ -19,5 +19,5 @@
           <cylinder radius="0.035" length="0.01"/>
         </geometry>
-        <origin rpy="0.0 ${-pi/2} 0.0" xyz="0.005 0.0 0.0"/>
+        <origin rpy="0.0 ${pi/2} 0.0" xyz="0.005 0.0 0.0"/>
       </collision>
       <inertial>
@@ -36,5 +36,5 @@
           <mesh filename="package://irc_ros_description/meshes/gripper_schmalz_ecbpmi/Joint0.dae"/>
         </geometry>
-        <origin rpy="0.0 0.0 0.0" xyz="0.07 0.0 0.0"/>
+        <origin rpy="0.0 0.0 ${pi/2}" xyz="0.07 0.0 0.0"/>
       </visual>
       <collision>
@@ -42,5 +42,5 @@
           <mesh filename="package://irc_ros_description/meshes/gripper_schmalz_ecbpmi/Joint0Coll.dae"/>
         </geometry>
-        <origin rpy="0.0 0.0 0.0" xyz="0.07 0.0 0.0"/>
+        <origin rpy="0.0 0.0 ${pi/2}" xyz="0.07 0.0 0.0"/>
       </collision>
       <inertial>

File: irc_ros_description/urdf/grippers/schmalz_ecbpmi.description.xacro (robot description, xacro)
@@ -6,5 +6,5 @@
       <parent link="${parent_link}" />
       <child link = "${prefix}gripper_mount" />
-      <origin xyz="0.0 0.0 0.0" rpy="0.0 ${-pi/2} 0.0" />
+      <origin xyz="0.0 0.0 0.0" rpy="0.0 0.0 0.0" />
     </joint>
     <link name="${prefix}gripper_mount">
@@ -13,5 +13,5 @@
           <cylinder radius="0.035" length="0.01"/>
         </geometry>
-        <origin rpy="0.0 ${-pi/2} 0.0" xyz="0.005 0.0 0.0"/>
+        <origin rpy="0.0 ${pi/2} 0.0" xyz="0.005 0.0 0.0"/>
       </visual>
       <collision>
@@ -19,5 +19,5 @@
           <cylinder radius="0.035" length="0.01"/>
         </geometry>
-        <origin rpy="0.0 ${-pi/2} 0.0" xyz="0.005 0.0 0.0"/>
+        <origin rpy="0.0 ${pi/2} 0.0" xyz="0.005 0.0 0.0"/>
       </collision>
       <inertial>
@@ -36,5 +36,5 @@
           <mesh filename="package://irc_ros_description/meshes/gripper_schmalz_ecbpmi/Joint0.dae"/>
         </geometry>
-        <origin rpy="0.0 0.0 0.0" xyz="0.07 0.0 0.0"/>
+        <origin rpy="0.0 0.0 ${pi/2}" xyz="0.07 0.0 0.0"/>
       </visual>
       <collision>

Commit message: Make coordinate frames conform with convention, fix examples (#91)
* Fix gripper coordinate system rotation

* Add tool0 joints, add mock_hardware to macros

* Align grippers with new flange frame orientation

* PNP Example: Rename eef link, adjust its rotation

* PNP_Vacuum: Adjust rotation, rename variable

* Load joint limits for scaling the velocity/acceleration of linear movements

* Fix the rest of the example while we are at it

File: irc_ros_description/urdf/grippers/ext_dio_gripper.description.xacro (robot description, xacro)
@@ -6,5 +6,5 @@
       <parent link="${parent_link}" />
       <child link = "${prefix}gripper_mount" />
-      <origin xyz="0.0 0.0 0.0" rpy="0.0 ${-pi/2} 0.0" />
+      <origin xyz="0.0 0.0 0.0" rpy="0.0 0.0 0.0" />
     </joint>
     <link name="${prefix}gripper_mount">
@@ -13,5 +13,5 @@
           <cylinder radius="0.035" length="0.01"/>
         </geometry>
-        <origin rpy="0.0 ${-pi/2} 0.0" xyz="0.005 0.0 0.0"/>
+        <origin rpy="0.0 ${pi/2} 0.0" xyz="0.005 0.0 0.0"/>
       </visual>
       <collision>
@@ -19,5 +19,5 @@
           <cylinder radius="0.035" length="0.01"/>
         </geometry>
-        <origin rpy="0.0 ${-pi/2} 0.0" xyz="0.005 0.0 0.0"/>
+        <origin rpy="0.0 ${pi/2} 0.0" xyz="0.005 0.0 0.0"/>
       </collision>
       <inertial>
@@ -36,5 +36,5 @@
           <mesh filename="package://irc_ros_description/meshes/gripper_schmalz_ecbpmi/Joint0.dae"/>
         </geometry>
-        <origin rpy="${pi/2} ${-pi/2} 0.0" xyz="0.07 0.0 0.0"/>
+        <origin rpy="0.0 0.0 ${pi/2}" xyz="0.07 0.0 0.0"/>
       </visual>
       <collision>
@@ -42,5 +42,5 @@
           <mesh filename="package://irc_ros_description/meshes/gripper_schmalz_ecbpmi/Joint0Coll.dae"/>
         </geometry>
-        <origin rpy="${pi/2} ${-pi/2} 0.0" xyz="0.07 0.0 0.0"/>
+        <origin rpy="0.0 0.0 ${pi/2}" xyz="0.07 0.0 0.0"/>
       </collision>
       <inertial>
@@ -49,5 +49,5 @@
       </inertial>
     </link>
-    <joint name="${prefix}joint99" type="fixed">
+    <joint name="${prefix}gripper_base_to_tcp" type="fixed">
       <parent link="${prefix}gripper_base"/>
       <child link="${prefix}tcp"/>

File: irc_ros_description/urdf/grippers/schmalz_ecbpmi.description.xacro (robot description, xacro)
@@ -6,5 +6,5 @@
       <parent link="${parent_link}" />
       <child link = "${prefix}gripper_mount" />
-      <origin xyz="0.0 0.0 0.0" rpy="0.0 ${-pi/2} 0.0" />
+      <origin xyz="0.0 0.0 0.0" rpy="0.0 0.0 0.0" />
     </joint>
     <link name="${prefix}gripper_mount">
@@ -13,5 +13,5 @@
           <cylinder radius="0.035" length="0.01"/>
         </geometry>
-        <origin rpy="0.0 ${-pi/2} 0.0" xyz="0.005 0.0 0.0"/>
+        <origin rpy="0.0 ${pi/2} 0.0" xyz="0.005 0.0 0.0"/>
       </visual>
       <collision>
@@ -19,5 +19,5 @@
           <cylinder radius="0.035" length="0.01"/>
         </geometry>
-        <origin rpy="0.0 ${-pi/2} 0.0" xyz="0.005 0.0 0.0"/>
+        <origin rpy="0.0 ${pi/2} 0.0" xyz="0.005 0.0 0.0"/>
       </collision>
       <inertial>
@@ -36,5 +36,5 @@
           <mesh filename="package://irc_ros_description/meshes/gripper_schmalz_ecbpmi/Joint0.dae"/>
         </geometry>
-        <origin rpy="${pi/2} ${-pi/2} 0.0" xyz="0.07 0.0 0.0"/>
+        <origin rpy="0.0 0.0 ${pi/2}" xyz="0.07 0.0 0.0"/>
       </visual>
       <collision>
@@ -42,5 +42,5 @@
           <mesh filename="package://irc_ros_description/meshes/gripper_schmalz_ecbpmi/Joint0Coll.dae"/>
         </geometry>
-        <origin rpy="${pi/2} ${-pi/2} 0.0" xyz="0.07 0.0 0.0"/>
+        <origin rpy="0.0 0.0 0.0" xyz="0.07 0.0 0.0"/>
       </collision>
       <inertial>
@@ -49,5 +49,5 @@
       </inertial>
     </link>
-    <joint name="${prefix}joint99" type="fixed">
+    <joint name="${prefix}gripper_base_to_tcp" type="fixed">
       <parent link="${prefix}gripper_base"/>
       <child link="${prefix}tcp"/>

File: irc_ros_description/urdf/robots/igus_rebel_4dof_00.description.xacro (robot description, xacro)
@@ -135,12 +135,16 @@
       <parent link="${prefix}link_4"/>
       <child link="${prefix}flange"/>
-      <origin rpy="0.0 0.0 0.0" xyz="0.0 0.0 0.062"/>
+      <origin rpy="0.0 ${-pi/2} 0.0" xyz="0.0 0.0 0.062"/>
       <axis xyz="0 -1 0"/>
     </joint>
     <link name="${prefix}flange">
-      <inertial>
-        <mass value="0.1"/>
-        <inertia ixx="0.03" ixy="0.0" ixz="0.0" iyy="0.03" iyz="0.0" izz="0.03"/>
-      </inertial>
+    </link>
+    <joint name="${prefix}flange_to_tool0" type="fixed">
+      <parent link="${prefix}flange"/>
+      <child link="${prefix}tool0"/>
+      <origin rpy="0.0 0.0 0.0" xyz="0.0 0.0 0.0"/>
+      <axis xyz="0 0 0"/>
+    </joint>
+    <link name="${prefix}tool0">
     </link>
   </xacro:macro>

File: irc_ros_description/urdf/robots/igus_rebel_6dof_00.description.xacro (robot description, xacro)
@@ -187,13 +187,16 @@
       <parent link="${prefix}link_8"/>
       <child link="${prefix}flange"/>
-      <origin rpy="0.0 0.0 0.0" xyz="0.0 0 0.0012"/>
-      <axis xyz="0 0 1"/>
-      <limit effort="330.0" lower="-3.12414" upper="3.12414" velocity="${pi*45/180}"/>
+      <origin rpy="0.0 ${-pi/2} 0.0" xyz="0.0 0 0.0012"/>
+      <axis xyz="0 0 0"/>
     </joint>
     <link name="${prefix}flange">
-      <inertial>
-        <mass value="0.1"/>
-        <inertia ixx="0.03" ixy="0.0" ixz="0.0" iyy="0.03" iyz="0.0" izz="0.03"/>
-      </inertial>
+    </link>
+    <joint name="${prefix}flange_to_tool0" type="fixed">
+      <parent link="${prefix}flange"/>
+      <child link="${prefix}tool0"/>
+      <origin rpy="0.0 0.0 0.0" xyz="0.0 0.0 0.0"/>
+      <axis xyz="0 0 0"/>
+    </joint>
+    <link name="${prefix}tool0">
     </link>
   </xacro:macro>

File: irc_ros_description/urdf/robots/igus_rebel_6dof_pre.description.xacro (robot description, xacro)
@@ -188,13 +188,16 @@
       <parent link="${prefix}link_8"/>
       <child link="${prefix}flange"/>
-      <origin rpy="0.0 0.0 0.0" xyz="0.0 0 0.0012"/>
-      <axis xyz="0 0 1"/>
-      <limit effort="330.0" lower="-3.12414" upper="3.12414" velocity="${pi*45/180}"/>
+      <origin rpy="0.0 ${-pi/2} 0.0" xyz="0.0 0 0.0012"/>
+      <axis xyz="0 0 0"/>
     </joint>
     <link name="${prefix}flange">
-      <inertial>
-        <mass value="0.1"/>
-        <inertia ixx="0.03" ixy="0.0" ixz="0.0" iyy="0.03" iyz="0.0" izz="0.03"/>
-      </inertial>
+    </link>
+    <joint name="${prefix}flange_to_tool0" type="fixed">
+      <parent link="${prefix}flange"/>
+      <child link="${prefix}tool0"/>
+      <origin rpy="0.0 0.0 0.0" xyz="0.0 0.0 0.0"/>
+      <axis xyz="0 0 0"/>
+    </joint>
+    <link name="${prefix}tool0">
     </link>
   </xacro:macro>

File: irc_ros_description/urdf/robots/igus_robolink_rl_dp_5.description.xacro (robot description, xacro)
@@ -158,13 +158,17 @@
       <parent link="${prefix}link_7"/>
       <child link="${prefix}flange"/>
-      <origin rpy="0.0 0.0 0.0" xyz="0.0 0 0.0115"/>
+      <origin rpy="0.0 ${-pi/2} 0.0" xyz="0.0 0 0.0115"/>
       <axis xyz="0 0 1"/>
       <limit effort="330.0" lower="-1.65806" upper="1.65806" velocity="2.16"/>
     </joint>
     <link name="${prefix}flange">
-      <inertial>
-        <mass value="0.1"/>
-        <inertia ixx="0.03" ixy="0.0" ixz="0.0" iyy="0.03" iyz="0.0" izz="0.03"/>
-      </inertial>
+    </link>
+    <joint name="${prefix}flange_to_tool0" type="fixed">
+      <parent link="${prefix}flange"/>
+      <child link="${prefix}tool0"/>
+      <origin rpy="0.0 0.0 0.0" xyz="0.0 0.0 0.0"/>
+      <axis xyz="0 0 0"/>
+    </joint>
+    <link name="${prefix}tool0">
     </link>
   </xacro:macro>
