Commit message: Replace package with file uri

File: irc_ros_description/urdf/grippers/ext_dio_gripper.description.xacro (robot description, xacro)
@@ -34,5 +34,5 @@
       <visual>
         <geometry>
-          <mesh filename="package://irc_ros_description/meshes/gripper_schmalz_ecbpmi/Joint0.dae"/>
+          <mesh filename="file://$(find irc_ros_description)/meshes/gripper_schmalz_ecbpmi/Joint0.dae"/>
         </geometry>
         <origin rpy="0.0 0.0 ${pi/2}" xyz="0.07 0.0 0.0"/>
@@ -40,5 +40,5 @@
       <collision>
         <geometry>
-          <mesh filename="package://irc_ros_description/meshes/gripper_schmalz_ecbpmi/Joint0Coll.dae"/>
+          <mesh filename="file://$(find irc_ros_description)/meshes/gripper_schmalz_ecbpmi/Joint0Coll.dae"/>
         </geometry>
         <origin rpy="0.0 0.0 ${pi/2}" xyz="0.07 0.0 0.0"/>

File: irc_ros_description/urdf/grippers/schmalz_ecbpmi.description.xacro (robot description, xacro)
@@ -34,5 +34,5 @@
       <visual>
         <geometry>
-          <mesh filename="package://irc_ros_description/meshes/gripper_schmalz_ecbpmi/Joint0.dae"/>
+          <mesh filename="file://$(find irc_ros_description)/meshes/gripper_schmalz_ecbpmi/Joint0.dae"/>
         </geometry>
         <origin rpy="0.0 0.0 ${pi/2}" xyz="0.07 0.0 0.0"/>
@@ -40,5 +40,5 @@
       <collision>
         <geometry>
-          <mesh filename="package://irc_ros_description/meshes/gripper_schmalz_ecbpmi/Joint0Coll.dae"/>
+          <mesh filename="file://$(find irc_ros_description)/meshes/gripper_schmalz_ecbpmi/Joint0Coll.dae"/>
         </geometry>
         <origin rpy="0.0 0.0 0.0" xyz="0.07 0.0 0.0"/>

File: irc_ros_description/urdf/platforms/cpr_platform_medium.description.xacro (robot description, xacro)
@@ -9,5 +9,5 @@
       <visual>
         <geometry>
-          <mesh filename="package://irc_ros_description/meshes/cpr_platform_medium/body.dae"/>
+          <mesh filename="file://$(find irc_ros_description)/meshes/cpr_platform_medium/body.dae"/>
         </geometry>
         <origin rpy="0 0 3.14" xyz="0 0 0"/>
@@ -15,5 +15,5 @@
       <collision>
         <geometry>
-          <mesh filename="package://irc_ros_description/meshes/cpr_platform_medium/bodyColl.dae"/>
+          <mesh filename="file://$(find irc_ros_description)/meshes/cpr_platform_medium/bodyColl.dae"/>
         </geometry>
         <origin rpy="0 0 ${pi}" xyz="0 0 0"/>
@@ -35,10 +35,10 @@
       <visual>
         <geometry>
-          <mesh filename="package://irc_ros_description/meshes/cpr_platform_medium/wheel.dae"/>
+          <mesh filename="file://$(find irc_ros_description)/meshes/cpr_platform_medium/wheel.dae"/>
         </geometry>
       </visual>
       <collision>
         <geometry>
-          <mesh filename="package://irc_ros_description/meshes/cpr_platform_medium/wheelColl.dae"/>
+          <mesh filename="file://$(find irc_ros_description)/meshes/cpr_platform_medium/wheelColl.dae"/>
         </geometry>
       </collision>
@@ -59,10 +59,10 @@
       <visual>
         <geometry>
-          <mesh filename="package://irc_ros_description/meshes/cpr_platform_medium/wheel.dae"/>
+          <mesh filename="file://$(find irc_ros_description)/meshes/cpr_platform_medium/wheel.dae"/>
         </geometry>
       </visual>
       <collision>
         <geometry>
-          <mesh filename="package://irc_ros_description/meshes/cpr_platform_medium/wheelColl.dae"/>
+          <mesh filename="file://$(find irc_ros_description)/meshes/cpr_platform_medium/wheelColl.dae"/>
         </geometry>
       </collision>

File: irc_ros_description/urdf/robots/igus_rebel_4dof_00.description.xacro (robot description, xacro)
@@ -6,10 +6,10 @@
       <visual>
         <geometry>
-          <mesh filename="package://irc_ros_description/meshes/igus_rebel_4dof_00/Joint0.dae"/>
+          <mesh filename="file://$(find irc_ros_description)/meshes/igus_rebel_4dof_00/Joint0.dae"/>
         </geometry>
       </visual>
       <collision>
         <geometry>
-          <mesh filename="package://irc_ros_description/meshes/igus_rebel_4dof_00/Joint0Coll.dae"/>
+          <mesh filename="file://$(find irc_ros_description)/meshes/igus_rebel_4dof_00/Joint0Coll.dae"/>
         </geometry>
       </collision>
@@ -29,5 +29,5 @@
       <visual>
         <geometry>
-          <mesh filename="package://irc_ros_description/meshes/igus_rebel_4dof_00/Joint1.dae"/>
+          <mesh filename="file://$(find irc_ros_description)/meshes/igus_rebel_4dof_00/Joint1.dae"/>
         </geometry>
         <origin rpy="0 0 0" xyz="0.0 0.0 0"/>
@@ -35,5 +35,5 @@
       <collision>
         <geometry>
-          <mesh filename="package://irc_ros_description/meshes/igus_rebel_4dof_00/Joint1Coll.dae"/>
+          <mesh filename="file://$(find irc_ros_description)/meshes/igus_rebel_4dof_00/Joint1Coll.dae"/>
         </geometry>
         <origin rpy="0 0 0" xyz="0.0 0.0 0"/>
@@ -55,5 +55,5 @@
       <visual>
         <geometry>
-          <mesh filename="package://irc_ros_description/meshes/igus_rebel_4dof_00/Joint2.dae"/>
+          <mesh filename="file://$(find irc_ros_description)/meshes/igus_rebel_4dof_00/Joint2.dae"/>
         </geometry>
         <origin rpy="0 0 0" xyz="0 0 0"/>
@@ -61,5 +61,5 @@
       <collision>
         <geometry>
-          <mesh filename="package://irc_ros_description/meshes/igus_rebel_4dof_00/Joint2Coll.dae"/>
+          <mesh filename="file://$(find irc_ros_description)/meshes/igus_rebel_4dof_00/Joint2Coll.dae"/>
         </geometry>
         <origin rpy="0 0 0" xyz="0 0 0"/>
@@ -81,5 +81,5 @@
       <visual>
         <geometry>
-          <mesh filename="package://irc_ros_description/meshes/igus_rebel_4dof_00/Joint3.dae"/>
+          <mesh filename="file://$(find irc_ros_description)/meshes/igus_rebel_4dof_00/Joint3.dae"/>
         </geometry>
         <origin rpy="0 0 0" xyz="0 0 0"/>
@@ -87,5 +87,5 @@
       <collision>
         <geometry>
-          <mesh filename="package://irc_ros_description/meshes/igus_rebel_4dof_00/Joint3Coll.dae"/>
+          <mesh filename="file://$(find irc_ros_description)/meshes/igus_rebel_4dof_00/Joint3Coll.dae"/>
         </geometry>
         <origin rpy="0 0 0" xyz="0 0 0"/>
@@ -117,5 +117,5 @@
       <visual>
         <geometry>
-          <mesh filename="package://irc_ros_description/meshes/igus_rebel_4dof_00/Joint4.dae"/>
+          <mesh filename="file://$(find irc_ros_description)/meshes/igus_rebel_4dof_00/Joint4.dae"/>
         </geometry>
         <origin rpy="0 0 0" xyz="0 0 0"/>
@@ -123,5 +123,5 @@
       <collision>
         <geometry>
-          <mesh filename="package://irc_ros_description/meshes/igus_rebel_4dof_00/Joint4Coll.dae"/>
+          <mesh filename="file://$(find irc_ros_description)/meshes/igus_rebel_4dof_00/Joint4Coll.dae"/>
         </geometry>
         <origin rpy="0 0 0" xyz="0 0 0"/>

File: irc_ros_description/urdf/robots/igus_rebel_6dof_00.description.xacro (robot description, xacro)
@@ -6,10 +6,10 @@
       <visual>
         <geometry>
-          <mesh filename="package://irc_ros_description/meshes/igus_rebel_6dof_00/Joint0.dae"/>
-        </geometry>
-      </visual>
-      <collision>
-        <geometry>
-          <mesh filename="package://irc_ros_description/meshes/igus_rebel_6dof_00/Joint0Coll.dae"/>
+          <mesh filename="file://$(find irc_ros_description)/meshes/igus_rebel_6dof_00/Joint0.dae"/>
+        </geometry>
+      </visual>
+      <collision>
+        <geometry>
+          <mesh filename="file://$(find irc_ros_description)/meshes/igus_rebel_6dof_00/Joint0Coll.dae"/>
         </geometry>
       </collision>
@@ -29,11 +29,11 @@
       <visual>
         <geometry>
-          <mesh filename="package://irc_ros_description/meshes/igus_rebel_6dof_00/Joint1.dae"/>
-        </geometry>
-        <origin rpy="0 0 0" xyz="0 0 0"/>
-      </visual>
-      <collision>
-        <geometry>
-          <mesh filename="package://irc_ros_description/meshes/igus_rebel_6dof_00/Joint1Coll.dae"/>
+          <mesh filename="file://$(find irc_ros_description)/meshes/igus_rebel_6dof_00/Joint1.dae"/>
+        </geometry>
+        <origin rpy="0 0 0" xyz="0 0 0"/>
+      </visual>
+      <collision>
+        <geometry>
+          <mesh filename="file://$(find irc_ros_description)/meshes/igus_rebel_6dof_00/Joint1Coll.dae"/>
         </geometry>
         <origin rpy="0 0 0" xyz="0 0 0"/>
@@ -55,11 +55,11 @@
       <visual>
         <geometry>
-          <mesh filename="package://irc_ros_description/meshes/igus_rebel_6dof_00/Joint2.dae"/>
-        </geometry>
-        <origin rpy="0 0 0" xyz="0 0 0"/>
-      </visual>
-      <collision>
-        <geometry>
-          <mesh filename="package://irc_ros_description/meshes/igus_rebel_6dof_00/Joint2Coll.dae"/>
+          <mesh filename="file://$(find irc_ros_description)/meshes/igus_rebel_6dof_00/Joint2.dae"/>
+        </geometry>
+        <origin rpy="0 0 0" xyz="0 0 0"/>
+      </visual>
+      <collision>
+        <geometry>
+          <mesh filename="file://$(find irc_ros_description)/meshes/igus_rebel_6dof_00/Joint2Coll.dae"/>
         </geometry>
         <origin rpy="0 0 0" xyz="0 0 0"/>
@@ -81,11 +81,11 @@
       <visual>
         <geometry>
-          <mesh filename="package://irc_ros_description/meshes/igus_rebel_6dof_00/Joint3.dae"/>
-        </geometry>
-        <origin rpy="0 0 0" xyz="0 0 0"/>
-      </visual>
-      <collision>
-        <geometry>
-          <mesh filename="package://irc_ros_description/meshes/igus_rebel_6dof_00/Joint3Coll.dae"/>
+          <mesh filename="file://$(find irc_ros_description)/meshes/igus_rebel_6dof_00/Joint3.dae"/>
+        </geometry>
+        <origin rpy="0 0 0" xyz="0 0 0"/>
+      </visual>
+      <collision>
+        <geometry>
+          <mesh filename="file://$(find irc_ros_description)/meshes/igus_rebel_6dof_00/Joint3Coll.dae"/>
         </geometry>
         <origin rpy="0 0 0" xyz="0 0 0"/>
@@ -107,11 +107,11 @@
       <visual>
         <geometry>
-          <mesh filename="package://irc_ros_description/meshes/igus_rebel_6dof_00/Joint4.dae"/>
-        </geometry>
-        <origin rpy="0 0 0" xyz="0 0 0"/>
-      </visual>
-      <collision>
-        <geometry>
-          <mesh filename="package://irc_ros_description/meshes/igus_rebel_6dof_00/Joint4Coll.dae"/>
+          <mesh filename="file://$(find irc_ros_description)/meshes/igus_rebel_6dof_00/Joint4.dae"/>
+        </geometry>
+        <origin rpy="0 0 0" xyz="0 0 0"/>
+      </visual>
+      <collision>
+        <geometry>
+          <mesh filename="file://$(find irc_ros_description)/meshes/igus_rebel_6dof_00/Joint4Coll.dae"/>
         </geometry>
         <origin rpy="0 0 0" xyz="0 0 0"/>
@@ -133,11 +133,11 @@
       <visual>
         <geometry>
-          <mesh filename="package://irc_ros_description/meshes/igus_rebel_6dof_00/Joint5.dae"/>
-        </geometry>
-        <origin rpy="0 0 0" xyz="0 0 0"/>
-      </visual>
-      <collision>
-        <geometry>
-          <mesh filename="package://irc_ros_description/meshes/igus_rebel_6dof_00/Joint5Coll.dae"/>
+          <mesh filename="file://$(find irc_ros_description)/meshes/igus_rebel_6dof_00/Joint5.dae"/>
+        </geometry>
+        <origin rpy="0 0 0" xyz="0 0 0"/>
+      </visual>
+      <collision>
+        <geometry>
+          <mesh filename="file://$(find irc_ros_description)/meshes/igus_rebel_6dof_00/Joint5Coll.dae"/>
         </geometry>
         <origin rpy="0 0 0" xyz="0 0 0"/>
@@ -169,5 +169,5 @@
       <visual>
         <geometry>
-          <mesh filename="package://irc_ros_description/meshes/igus_rebel_6dof_00/Joint6.dae"/>
+          <mesh filename="file://$(find irc_ros_description)/meshes/igus_rebel_6dof_00/Joint6.dae"/>
         </geometry>
         <origin rpy="0 0 0" xyz="0.0 0 0"/>
@@ -175,5 +175,5 @@
       <collision>
         <geometry>
-          <mesh filename="package://irc_ros_description/meshes/igus_rebel_6dof_00/Joint6Coll.dae"/>
+          <mesh filename="file://$(find irc_ros_description)/meshes/igus_rebel_6dof_00/Joint6Coll.dae"/>
         </geometry>
         <origin rpy="0 0 0" xyz="0.0 0 0"/>

File: irc_ros_description/urdf/robots/igus_rebel_6dof_pre.description.xacro (robot description, xacro)
@@ -6,10 +6,10 @@
       <visual>
         <geometry>
-          <mesh filename="package://irc_ros_description/meshes/igus_rebel_6dof_pre/Joint0.dae"/>
-        </geometry>
-      </visual>
-      <collision>
-        <geometry>
-          <mesh filename="package://irc_ros_description/meshes/igus_rebel_6dof_pre/Joint0Coll.dae"/>
+          <mesh filename="file://$(find irc_ros_description)/meshes/igus_rebel_6dof_pre/Joint0.dae"/>
+        </geometry>
+      </visual>
+      <collision>
+        <geometry>
+          <mesh filename="file://$(find irc_ros_description)/meshes/igus_rebel_6dof_pre/Joint0Coll.dae"/>
         </geometry>
       </collision>
@@ -29,11 +29,11 @@
       <visual>
         <geometry>
-          <mesh filename="package://irc_ros_description/meshes/igus_rebel_6dof_pre/Joint1.dae"/>
-        </geometry>
-        <origin rpy="0 0 0" xyz="0 0 0"/>
-      </visual>
-      <collision>
-        <geometry>
-          <mesh filename="package://irc_ros_description/meshes/igus_rebel_6dof_pre/Joint1Coll.dae"/>
+          <mesh filename="file://$(find irc_ros_description)/meshes/igus_rebel_6dof_pre/Joint1.dae"/>
+        </geometry>
+        <origin rpy="0 0 0" xyz="0 0 0"/>
+      </visual>
+      <collision>
+        <geometry>
+          <mesh filename="file://$(find irc_ros_description)/meshes/igus_rebel_6dof_pre/Joint1Coll.dae"/>
         </geometry>
         <origin rpy="0 0 0" xyz="0 0 0"/>
@@ -55,11 +55,11 @@
       <visual>
         <geometry>
-          <mesh filename="package://irc_ros_description/meshes/igus_rebel_6dof_pre/Joint2.dae"/>
-        </geometry>
-        <origin rpy="0 0 0" xyz="0 0 0"/>
-      </visual>
-      <collision>
-        <geometry>
-          <mesh filename="package://irc_ros_description/meshes/igus_rebel_6dof_pre/Joint2Coll.dae"/>
+          <mesh filename="file://$(find irc_ros_description)/meshes/igus_rebel_6dof_pre/Joint2.dae"/>
+        </geometry>
+        <origin rpy="0 0 0" xyz="0 0 0"/>
+      </visual>
+      <collision>
+        <geometry>
+          <mesh filename="file://$(find irc_ros_description)/meshes/igus_rebel_6dof_pre/Joint2Coll.dae"/>
         </geometry>
         <origin rpy="0 0 0" xyz="0 0 0"/>
@@ -81,11 +81,11 @@
       <visual>
         <geometry>
-          <mesh filename="package://irc_ros_description/meshes/igus_rebel_6dof_pre/Joint3.dae"/>
-        </geometry>
-        <origin rpy="0 0 0" xyz="0 0 0"/>
-      </visual>
-      <collision>
-        <geometry>
-          <mesh filename="package://irc_ros_description/meshes/igus_rebel_6dof_pre/Joint3Coll.dae"/>
+          <mesh filename="file://$(find irc_ros_description)/meshes/igus_rebel_6dof_pre/Joint3.dae"/>
+        </geometry>
+        <origin rpy="0 0 0" xyz="0 0 0"/>
+      </visual>
+      <collision>
+        <geometry>
+          <mesh filename="file://$(find irc_ros_description)/meshes/igus_rebel_6dof_pre/Joint3Coll.dae"/>
         </geometry>
         <origin rpy="0 0 0" xyz="0 0 0"/>
@@ -108,11 +108,11 @@
       <visual>
         <geometry>
-          <mesh filename="package://irc_ros_description/meshes/igus_rebel_6dof_pre/Joint4.dae"/>
-        </geometry>
-        <origin rpy="0 0 0" xyz="0 0 0"/>
-      </visual>
-      <collision>
-        <geometry>
-          <mesh filename="package://irc_ros_description/meshes/igus_rebel_6dof_pre/Joint4Coll.dae"/>
+          <mesh filename="file://$(find irc_ros_description)/meshes/igus_rebel_6dof_pre/Joint4.dae"/>
+        </geometry>
+        <origin rpy="0 0 0" xyz="0 0 0"/>
+      </visual>
+      <collision>
+        <geometry>
+          <mesh filename="file://$(find irc_ros_description)/meshes/igus_rebel_6dof_pre/Joint4Coll.dae"/>
         </geometry>
         <origin rpy="0 0 0" xyz="0 0 0"/>
@@ -134,11 +134,11 @@
       <visual>
         <geometry>
-          <mesh filename="package://irc_ros_description/meshes/igus_rebel_6dof_pre/Joint5.dae"/>
-        </geometry>
-        <origin rpy="0 0 0" xyz="0 0 0"/>
-      </visual>
-      <collision>
-        <geometry>
-          <mesh filename="package://irc_ros_description/meshes/igus_rebel_6dof_pre/Joint5Coll.dae"/>
+          <mesh filename="file://$(find irc_ros_description)/meshes/igus_rebel_6dof_pre/Joint5.dae"/>
+        </geometry>
+        <origin rpy="0 0 0" xyz="0 0 0"/>
+      </visual>
+      <collision>
+        <geometry>
+          <mesh filename="file://$(find irc_ros_description)/meshes/igus_rebel_6dof_pre/Joint5Coll.dae"/>
         </geometry>
         <origin rpy="0 0 0" xyz="0 0 0"/>
@@ -170,5 +170,5 @@
       <visual>
         <geometry>
-          <mesh filename="package://irc_ros_description/meshes/igus_rebel_6dof_pre/Joint6.dae"/>
+          <mesh filename="file://$(find irc_ros_description)/meshes/igus_rebel_6dof_pre/Joint6.dae"/>
         </geometry>
         <origin rpy="0 0 0" xyz="0.0 0 0"/>
@@ -176,5 +176,5 @@
       <collision>
         <geometry>
-          <mesh filename="package://irc_ros_description/meshes/igus_rebel_6dof_pre/Joint6Coll.dae"/>
+          <mesh filename="file://$(find irc_ros_description)/meshes/igus_rebel_6dof_pre/Joint6Coll.dae"/>
         </geometry>
         <origin rpy="0 0 0" xyz="0.0 0 0"/>

File: irc_ros_description/urdf/robots/igus_robolink_rl_dp_5.description.xacro (robot description, xacro)
@@ -6,10 +6,10 @@
       <visual>
         <geometry>
-          <mesh filename="package://irc_ros_description/meshes/igus_robolink_rl_dp_5/Joint0.dae"/>
+          <mesh filename="file://$(find irc_ros_description)/meshes/igus_robolink_rl_dp_5/Joint0.dae"/>
         </geometry>
       </visual>
       <collision>
         <geometry>
-          <mesh filename="package://irc_ros_description/meshes/igus_robolink_rl_dp_5/Joint0Coll.dae"/>
+          <mesh filename="file://$(find irc_ros_description)/meshes/igus_robolink_rl_dp_5/Joint0Coll.dae"/>
         </geometry>
       </collision>
@@ -29,5 +29,5 @@
       <visual>
         <geometry>
-          <mesh filename="package://irc_ros_description/meshes/igus_robolink_rl_dp_5/Joint1.dae"/>
+          <mesh filename="file://$(find irc_ros_description)/meshes/igus_robolink_rl_dp_5/Joint1.dae"/>
         </geometry>
         <origin rpy="0 0 0" xyz="0 0 0"/>
@@ -35,5 +35,5 @@
       <collision>
         <geometry>
-          <mesh filename="package://irc_ros_description/meshes/igus_robolink_rl_dp_5/Joint1Coll.dae"/>
+          <mesh filename="file://$(find irc_ros_description)/meshes/igus_robolink_rl_dp_5/Joint1Coll.dae"/>
         </geometry>
         <origin rpy="0 0 0" xyz="0 0 0"/>
@@ -54,5 +54,5 @@
       <visual>
         <geometry>
-          <mesh filename="package://irc_ros_description/meshes/igus_robolink_rl_dp_5/Joint2.dae"/>
+          <mesh filename="file://$(find irc_ros_description)/meshes/igus_robolink_rl_dp_5/Joint2.dae"/>
         </geometry>
         <origin rpy="0 0 0" xyz="0 0 0"/>
@@ -60,5 +60,5 @@
       <collision>
         <geometry>
-          <mesh filename="package://irc_ros_description/meshes/igus_robolink_rl_dp_5/Joint2Coll.dae"/>
+          <mesh filename="file://$(find irc_ros_description)/meshes/igus_robolink_rl_dp_5/Joint2Coll.dae"/>
         </geometry>
         <origin rpy="0 0 0" xyz="0 0 0"/>
@@ -79,5 +79,5 @@
       <visual>
         <geometry>
-          <mesh filename="package://irc_ros_description/meshes/igus_robolink_rl_dp_5/Joint3.dae"/>
+          <mesh filename="file://$(find irc_ros_description)/meshes/igus_robolink_rl_dp_5/Joint3.dae"/>
         </geometry>
         <origin rpy="0 0 0" xyz="0 0 0"/>
@@ -85,5 +85,5 @@
       <collision>
         <geometry>
-          <mesh filename="package://irc_ros_description/meshes/igus_robolink_rl_dp_5/Joint3Coll.dae"/>
+          <mesh filename="file://$(find irc_ros_description)/meshes/igus_robolink_rl_dp_5/Joint3Coll.dae"/>
         </geometry>
         <origin rpy="0 0 0" xyz="0 0 0"/>
@@ -104,5 +104,5 @@
       <visual>
         <geometry>
-          <mesh filename="package://irc_ros_description/meshes/igus_robolink_rl_dp_5/Joint4.dae"/>
+          <mesh filename="file://$(find irc_ros_description)/meshes/igus_robolink_rl_dp_5/Joint4.dae"/>
         </geometry>
         <origin rpy="0 0 0" xyz="0 0 0"/>
@@ -110,5 +110,5 @@
       <collision>
         <geometry>
-          <mesh filename="package://irc_ros_description/meshes/igus_robolink_rl_dp_5/Joint4Coll.dae"/>
+          <mesh filename="file://$(find irc_ros_description)/meshes/igus_robolink_rl_dp_5/Joint4Coll.dae"/>
         </geometry>
         <origin rpy="0 0 0" xyz="0 0 0"/>
@@ -140,5 +140,5 @@
       <visual>
         <geometry>
-          <mesh filename="package://irc_ros_description/meshes/igus_robolink_rl_dp_5/Joint5.dae"/>
+          <mesh filename="file://$(find irc_ros_description)/meshes/igus_robolink_rl_dp_5/Joint5.dae"/>
         </geometry>
         <origin rpy="0 0 0" xyz="0 0 0"/>
@@ -146,5 +146,5 @@
       <collision>
         <geometry>
-          <mesh filename="package://irc_ros_description/meshes/igus_robolink_rl_dp_5/Joint5Coll.dae"/>
+          <mesh filename="file://$(find irc_ros_description)/meshes/igus_robolink_rl_dp_5/Joint5Coll.dae"/>
         </geometry>
         <origin rpy="0 0 0" xyz="0 0 0"/>
