Commit message: Add tool0 joints, add mock_hardware to macros

File: irc_ros_description/urdf/robots/igus_rebel_4dof_00.description.xacro (robot description, xacro)
@@ -137,8 +137,12 @@
     </joint>
     <link name="${prefix}flange">
-      <inertial>
-        <mass value="0.1"/>
-        <inertia ixx="0.03" ixy="0.0" ixz="0.0" iyy="0.03" iyz="0.0" izz="0.03"/>
-      </inertial>
+    </link>
+    <joint name="${prefix}flange_to_tool0" type="fixed">
+      <parent link="${prefix}flange"/>
+      <child link="${prefix}tool0"/>
+      <origin rpy="0.0 0.0 0.0" xyz="0.0 0.0 0.062"/>
+      <axis xyz="0 0 0"/>
+    </joint>
+    <link name="${prefix}tool0">
     </link>
   </xacro:macro>

File: irc_ros_description/urdf/robots/igus_rebel_6dof_00.description.xacro (robot description, xacro)
@@ -190,8 +190,12 @@
     </joint>
     <link name="${prefix}flange">
-      <inertial>
-        <mass value="0.1"/>
-        <inertia ixx="0.03" ixy="0.0" ixz="0.0" iyy="0.03" iyz="0.0" izz="0.03"/>
-      </inertial>
+    </link>
+    <joint name="${prefix}flange_to_tool0" type="fixed">
+      <parent link="${prefix}flange"/>
+      <child link="${prefix}tool0"/>
+      <origin rpy="0.0 0.0 0.0" xyz="0.0 0.0 0.062"/>
+      <axis xyz="0 0 0"/>
+    </joint>
+    <link name="${prefix}tool0">
     </link>
   </xacro:macro>

File: irc_ros_description/urdf/robots/igus_rebel_6dof_pre.description.xacro (robot description, xacro)
@@ -190,8 +190,12 @@
     </joint>
     <link name="${prefix}flange">
-      <inertial>
-        <mass value="0.1"/>
-        <inertia ixx="0.03" ixy="0.0" ixz="0.0" iyy="0.03" iyz="0.0" izz="0.03"/>
-      </inertial>
+    </link>
+    <joint name="${prefix}flange_to_tool0" type="fixed">
+      <parent link="${prefix}flange"/>
+      <child link="${prefix}tool0"/>
+      <origin rpy="0.0 0.0 0.0" xyz="0.0 0.0 0.062"/>
+      <axis xyz="0 0 0"/>
+    </joint>
+    <link name="${prefix}tool0">
     </link>
   </xacro:macro>

File: irc_ros_description/urdf/robots/igus_robolink_rl_dp_5.description.xacro (robot description, xacro)
@@ -163,8 +163,12 @@
     </joint>
     <link name="${prefix}flange">
-      <inertial>
-        <mass value="0.1"/>
-        <inertia ixx="0.03" ixy="0.0" ixz="0.0" iyy="0.03" iyz="0.0" izz="0.03"/>
-      </inertial>
+    </link>
+    <joint name="${prefix}flange_to_tool0" type="fixed">
+      <parent link="${prefix}flange"/>
+      <child link="${prefix}tool0"/>
+      <origin rpy="0.0 0.0 0.0" xyz="0.0 0.0 0.062"/>
+      <axis xyz="0 0 0"/>
+    </joint>
+    <link name="${prefix}tool0">
     </link>
   </xacro:macro>

Commit message: Fix flange/tool0 coordinate systems

File: irc_ros_description/urdf/robots/igus_rebel_4dof_00.description.xacro (robot description, xacro)
@@ -133,5 +133,5 @@
       <parent link="${prefix}link_4"/>
       <child link="${prefix}flange"/>
-      <origin rpy="0.0 0.0 0.0" xyz="0.0 0.0 0.062"/>
+      <origin rpy="0.0 ${-pi/2} 0.0" xyz="0.0 0.0 0.062"/>
       <axis xyz="0 -1 0"/>
     </joint>
@@ -141,5 +141,5 @@
       <parent link="${prefix}flange"/>
       <child link="${prefix}tool0"/>
-      <origin rpy="0.0 0.0 0.0" xyz="0.0 0.0 0.062"/>
+      <origin rpy="0.0 0.0 0.0" xyz="0.0 0.0 0.0"/>
       <axis xyz="0 0 0"/>
     </joint>

File: irc_ros_description/urdf/robots/igus_rebel_6dof_00.description.xacro (robot description, xacro)
@@ -185,7 +185,6 @@
       <parent link="${prefix}link_8"/>
       <child link="${prefix}flange"/>
-      <origin rpy="0.0 0.0 0.0" xyz="0.0 0 0.0012"/>
-      <axis xyz="0 0 1"/>
-      <limit effort="330.0" lower="-3.12414" upper="3.12414" velocity="2.16"/>
+      <origin rpy="0.0 ${-pi/2} 0.0" xyz="0.0 0 0.0012"/>
+      <axis xyz="0 0 0"/>
     </joint>
     <link name="${prefix}flange">
@@ -194,5 +193,5 @@
       <parent link="${prefix}flange"/>
       <child link="${prefix}tool0"/>
-      <origin rpy="0.0 0.0 0.0" xyz="0.0 0.0 0.062"/>
+      <origin rpy="0.0 0.0 0.0" xyz="0.0 0.0 0.0"/>
       <axis xyz="0 0 0"/>
     </joint>

File: irc_ros_description/urdf/robots/igus_rebel_6dof_pre.description.xacro (robot description, xacro)
@@ -185,7 +185,6 @@
       <parent link="${prefix}link_8"/>
       <child link="${prefix}flange"/>
-      <origin rpy="0.0 0.0 0.0" xyz="0.0 0 0.0012"/>
-      <axis xyz="0 0 1"/>
-      <limit effort="330.0" lower="-3.12414" upper="3.12414" velocity="2.16"/>
+      <origin rpy="0.0 ${-pi/2} 0.0" xyz="0.0 0 0.0012"/>
+      <axis xyz="0 0 0"/>
     </joint>
     <link name="${prefix}flange">
@@ -194,5 +193,5 @@
       <parent link="${prefix}flange"/>
       <child link="${prefix}tool0"/>
-      <origin rpy="0.0 0.0 0.0" xyz="0.0 0.0 0.062"/>
+      <origin rpy="0.0 0.0 0.0" xyz="0.0 0.0 0.0"/>
       <axis xyz="0 0 0"/>
     </joint>

File: irc_ros_description/urdf/robots/igus_robolink_rl_dp_5.description.xacro (robot description, xacro)
@@ -158,5 +158,5 @@
       <parent link="${prefix}link_7"/>
       <child link="${prefix}flange"/>
-      <origin rpy="0.0 0.0 0.0" xyz="0.0 0 0.0115"/>
+      <origin rpy="0.0 ${-pi/2} 0.0" xyz="0.0 0 0.0115"/>
       <axis xyz="0 0 1"/>
       <limit effort="330.0" lower="-1.65806" upper="1.65806" velocity="2.16"/>
@@ -167,5 +167,5 @@
       <parent link="${prefix}flange"/>
       <child link="${prefix}tool0"/>
-      <origin rpy="0.0 0.0 0.0" xyz="0.0 0.0 0.062"/>
+      <origin rpy="0.0 0.0 0.0" xyz="0.0 0.0 0.0"/>
       <axis xyz="0 0 0"/>
     </joint>

Commit message: Lower joint limits on axis 2 and 3

File: irc_ros_description/urdf/robots/igus_rebel_4dof_00.description.xacro (robot description, xacro)
@@ -49,5 +49,6 @@
       <origin rpy="0.0 ${pi/6} 0.0" xyz="0.0 0 0.149"/>
       <axis xyz="0 1 0"/>
-      <limit effort="330.0" lower="${-pi*2/3}" upper="${pi*2/3}" velocity="2.16"/>
+      <!-- pi*2/3 are the physical limits, but to avoid any collisions we set the actual limits lower -->
+      <limit effort="330.0" lower="${-pi*11/18}" upper="${pi*11/18}" velocity="2.16"/>
     </joint>
     <link name="${prefix}link_2">
@@ -74,5 +75,6 @@
       <origin rpy="0.0 ${pi/6} 0.0" xyz="0.0 0.0 0.2384"/>
       <axis xyz="0 1 0"/>
-      <limit effort="330.0" lower="${-pi*2/3}" upper="${pi*2/3}" velocity="2.16"/>
+      <!-- pi*2/3 are the physical limits, but to avoid any collisions we set the actual limits lower -->
+      <limit effort="330.0" lower="${-pi*11/18}" upper="${pi*11/18}" velocity="2.16"/>
     </joint>
     <link name="${prefix}link_3">

File: irc_ros_description/urdf/robots/igus_rebel_6dof_00.description.xacro (robot description, xacro)
@@ -49,5 +49,6 @@
       <origin rpy="0.0 ${pi/6} 0.0" xyz="0.0 0 0.149"/>
       <axis xyz="0 1 0"/>
-      <limit effort="330.0" lower="${-pi*2/3}" upper="${pi*2/3}" velocity="2.16"/>
+      <!-- pi*2/3 are the physical limits, but to avoid any collisions we set the actual limits lower -->
+      <limit effort="330.0" lower="${-pi*11/18}" upper="${pi*11/18}" velocity="2.16"/>
     </joint>
     <link name="${prefix}link_2">
@@ -74,5 +75,6 @@
       <origin rpy="0.0 ${pi/6} 0.0" xyz="0.0 0.0 0.2384"/>
       <axis xyz="0 1 0"/>
-      <limit effort="330.0" lower="${-pi*2/3}" upper="${pi*2/3}" velocity="2.16"/>
+      <!-- pi*2/3 are the physical limits, but to avoid any collisions we set the actual limits lower -->
+      <limit effort="330.0" lower="${-pi*11/18}" upper="${pi*11/18}" velocity="2.16"/>
     </joint>
     <link name="${prefix}link_5">

File: irc_ros_description/urdf/robots/igus_rebel_6dof_pre.description.xacro (robot description, xacro)
@@ -49,5 +49,6 @@
       <origin rpy="0.0 0.0 0.0" xyz="0.0 0 0.130"/>
       <axis xyz="0 1 0"/>
-      <limit effort="330.0" lower="${-pi*2/3 + pi/6}" upper="${pi*2/3 + pi/6}" velocity="2.16"/>
+      <!-- pi*2/3 are the physical limits, but to avoid any collisions we set the actual limits lower -->
+      <limit effort="330.0" lower="${-pi*11/18 + pi/6}" upper="${pi*11/18 + pi/6}" velocity="2.16"/>
     </joint>
     <link name="${prefix}link_2">
@@ -74,5 +75,6 @@
       <origin rpy="0.0 0.0 0.0" xyz="0.0 0.0 0.2384"/>
       <axis xyz="0 1 0"/>
-      <limit effort="330.0" lower="${-pi*2/3 + pi/6}" upper="${pi*2/3 + pi/6}" velocity="2.16"/>
+      <!-- pi*2/3 are the physical limits, but to avoid any collisions we set the actual limits lower -->
+      <limit effort="330.0" lower="${-pi*11/18 + pi/6}" upper="${pi*11/18 + pi/6}" velocity="2.16"/>
     </joint>
     <link name="${prefix}link_5">

Commit message: Fix joint offsets

File: irc_ros_description/urdf/robots/igus_rebel_4dof_00.description.xacro (robot description, xacro)
@@ -100,5 +100,5 @@
         <parent link="${prefix}link_3"/>
         <child link="${prefix}link_4"/>
-        <origin rpy="0.0 0.0 0.0" xyz="0.0 0.0 0.2423"/>
+        <origin rpy="0.0 ${pi/24} 0.0" xyz="0.0 0.0 0.2423"/>
         <axis xyz="0 -1 0"/>
         <limit effort="330.0" velocity="2.16"/>
@@ -109,5 +109,5 @@
         <parent link="${prefix}link_3"/>
         <child link="${prefix}link_4"/>
-        <origin rpy="0.0 0.0 0.0" xyz="0.0 0.0 0.2423"/>
+        <origin rpy="0.0 ${-pi/24} 0.0" xyz="0.0 0.0 0.2423"/>
         <axis xyz="0 -1 0"/>
         <limit effort="330.0" lower="${-pi*179/180}" upper="${pi*179/180}" velocity="2.16"/>

File: irc_ros_description/urdf/robots/igus_rebel_6dof_00.description.xacro (robot description, xacro)
@@ -126,5 +126,5 @@
       <child link="${prefix}link_7"/>
       <!-- TODO The 0.03m offset are most likely caused by the mesh file (Issue 15) -->
-      <origin rpy="0.0 0.0 0.0" xyz="0.0 0 ${0.14 + 0.03}"/>
+      <origin rpy="0.0 ${-pi/24} 0.0" xyz="0.0 0 ${0.14 + 0.03}"/>
       <axis xyz="0 1 0"/>
       <limit effort="330.0" lower="${-pi*19/36}" upper="${pi*19/36}" velocity="2.16"/>

File: irc_ros_description/urdf/robots/igus_rebel_6dof_pre.description.xacro (robot description, xacro)
@@ -100,4 +100,5 @@
       <child link="${prefix}link_6"/>
       <!-- TODO The 0.03m offset are most likely caused by the mesh file (Issue 15) -->
+      <!-- The irc config file specifies a rotational offset of 65 degrees, if someone has access to a pre version please verify if that is correct -->
       <origin rpy="0.0 0.0 0.0" xyz="0.0 0 ${0.149 - 0.03}"/>
       <axis xyz="0 0 1"/>

Commit message: Change velocities in urdf descriptions to match new defaults

File: irc_ros_description/urdf/robots/igus_rebel_4dof_00.description.xacro (robot description, xacro)
@@ -24,5 +24,5 @@
       <origin rpy="0.0 0.0 0.0" xyz="0.0 0.0 0.100"/>
       <axis xyz="0 0 -1"/>
-      <limit effort="330.0" lower="${-pi*179/180}" upper="${pi*179/180}" velocity="2.16"/>
+      <limit effort="330.0" lower="${-pi*179/180}" upper="${pi*179/180}" velocity="${pi*45/180}"/>
     </joint>
     <link name="${prefix}link_1">
@@ -50,5 +50,5 @@
       <axis xyz="0 1 0"/>
       <!-- pi*2/3 are the physical limits, but to avoid any collisions we set the actual limits lower -->
-      <limit effort="330.0" lower="${-pi*11/18}" upper="${pi*11/18}" velocity="2.16"/>
+      <limit effort="330.0" lower="${-pi*11/18}" upper="${pi*11/18}" velocity="${pi*45/180}"/>
     </joint>
     <link name="${prefix}link_2">
@@ -76,5 +76,5 @@
       <axis xyz="0 1 0"/>
       <!-- pi*2/3 are the physical limits, but to avoid any collisions we set the actual limits lower -->
-      <limit effort="330.0" lower="${-pi*11/18}" upper="${pi*11/18}" velocity="2.16"/>
+      <limit effort="330.0" lower="${-pi*11/18}" upper="${pi*11/18}" velocity="${pi*45/180}"/>
     </joint>
     <link name="${prefix}link_3">
@@ -102,5 +102,5 @@
         <origin rpy="0.0 ${pi/24} 0.0" xyz="0.0 0.0 0.2423"/>
         <axis xyz="0 -1 0"/>
-        <limit effort="330.0" velocity="2.16"/>
+        <limit effort="330.0" velocity="${pi*45/180}"/>
       </joint>
     </xacro:if>
@@ -111,5 +111,5 @@
         <origin rpy="0.0 ${-pi/24} 0.0" xyz="0.0 0.0 0.2423"/>
         <axis xyz="0 -1 0"/>
-        <limit effort="330.0" lower="${-pi*179/180}" upper="${pi*179/180}" velocity="2.16"/>
+        <limit effort="330.0" lower="${-pi*179/180}" upper="${pi*179/180}" velocity="${pi*45/180}"/>
       </joint>
     </xacro:unless>

File: irc_ros_description/urdf/robots/igus_rebel_6dof_00.description.xacro (robot description, xacro)
@@ -24,5 +24,5 @@
       <origin rpy="0.0 0.0 0.0" xyz="0.0 0 0.100"/>
       <axis xyz="0 0 -1"/>
-      <limit effort="330.0" lower="${-pi*179/180}" upper="${pi*179/180}" velocity="2.16"/>
+      <limit effort="330.0" lower="${-pi*179/180}" upper="${pi*179/180}" velocity="${pi*45/180}"/>
     </joint>
     <link name="${prefix}link_1">
@@ -50,5 +50,5 @@
       <axis xyz="0 1 0"/>
       <!-- pi*2/3 are the physical limits, but to avoid any collisions we set the actual limits lower -->
-      <limit effort="330.0" lower="${-pi*11/18}" upper="${pi*11/18}" velocity="2.16"/>
+      <limit effort="330.0" lower="${-pi*11/18}" upper="${pi*11/18}" velocity="${pi*45/180}"/>
     </joint>
     <link name="${prefix}link_2">
@@ -76,5 +76,5 @@
       <axis xyz="0 1 0"/>
       <!-- pi*2/3 are the physical limits, but to avoid any collisions we set the actual limits lower -->
-      <limit effort="330.0" lower="${-pi*11/18}" upper="${pi*11/18}" velocity="2.16"/>
+      <limit effort="330.0" lower="${-pi*11/18}" upper="${pi*11/18}" velocity="${pi*45/180}"/>
     </joint>
     <link name="${prefix}link_5">
@@ -102,5 +102,5 @@
       <origin rpy="0.0 0.0 0.0" xyz="0.0 0 ${0.149 - 0.03}"/>
       <axis xyz="0 0 1"/>
-      <limit effort="330.0" lower="${-pi*179/180}" upper="${pi*179/180}" velocity="2.16"/>
+      <limit effort="330.0" lower="${-pi*179/180}" upper="${pi*179/180}" velocity="${pi*45/180}"/>
     </joint>
     <link name="${prefix}link_6">
@@ -128,5 +128,5 @@
       <origin rpy="0.0 ${-pi/24} 0.0" xyz="0.0 0 ${0.14 + 0.03}"/>
       <axis xyz="0 1 0"/>
-      <limit effort="330.0" lower="${-pi*19/36}" upper="${pi*19/36}" velocity="2.16"/>
+      <limit effort="330.0" lower="${-pi*19/36}" upper="${pi*19/36}" velocity="${pi*45/180}"/>
     </joint>
     <link name="${prefix}link_7">
@@ -154,5 +154,5 @@
         <origin rpy="0.0 0.0 0.0" xyz="0.0 0 0.1208"/>
         <axis xyz="0 0 1"/>
-        <limit effort="330.0" velocity="2.16"/>
+        <limit effort="330.0" velocity="${pi*45/180}"/>
       </joint>
     </xacro:if>
@@ -163,5 +163,5 @@
         <origin rpy="0.0 0.0 0.0" xyz="0.0 0 0.1208"/>
         <axis xyz="0 0 1"/>
-        <limit effort="330.0" lower="${-pi*179/180}" upper="${pi*179/180}" velocity="2.16"/>
+        <limit effort="330.0" lower="${-pi*179/180}" upper="${pi*179/180}" velocity="${pi*45/180}"/>
       </joint>
     </xacro:unless>
@@ -189,5 +189,5 @@
       <origin rpy="0.0 0.0 0.0" xyz="0.0 0 0.0012"/>
       <axis xyz="0 0 1"/>
-      <limit effort="330.0" lower="-3.12414" upper="3.12414" velocity="2.16"/>
+      <limit effort="330.0" lower="-3.12414" upper="3.12414" velocity="${pi*45/180}"/>
     </joint>
     <link name="${prefix}flange">

File: irc_ros_description/urdf/robots/igus_rebel_6dof_pre.description.xacro (robot description, xacro)
@@ -24,5 +24,5 @@
       <origin rpy="0.0 0.0 0.0" xyz="0.0 0 0.144"/>
       <axis xyz="0 0 -1"/>
-      <limit effort="330.0" lower="${-pi*179/180}" upper="${pi*179/180}" velocity="2.16"/>
+      <limit effort="330.0" lower="${-pi*179/180}" upper="${pi*179/180}" velocity="${pi*45/180}"/>
     </joint>
     <link name="${prefix}link_1">
@@ -50,5 +50,5 @@
       <axis xyz="0 1 0"/>
       <!-- pi*2/3 are the physical limits, but to avoid any collisions we set the actual limits lower -->
-      <limit effort="330.0" lower="${-pi*11/18 + pi/6}" upper="${pi*11/18 + pi/6}" velocity="2.16"/>
+      <limit effort="330.0" lower="${-pi*11/18 + pi/6}" upper="${pi*11/18 + pi/6}" velocity="${pi*45/180}"/>
     </joint>
     <link name="${prefix}link_2">
@@ -76,5 +76,5 @@
       <axis xyz="0 1 0"/>
       <!-- pi*2/3 are the physical limits, but to avoid any collisions we set the actual limits lower -->
-      <limit effort="330.0" lower="${-pi*11/18 + pi/6}" upper="${pi*11/18 + pi/6}" velocity="2.16"/>
+      <limit effort="330.0" lower="${-pi*11/18 + pi/6}" upper="${pi*11/18 + pi/6}" velocity="${pi*45/180}"/>
     </joint>
     <link name="${prefix}link_5">
@@ -103,5 +103,5 @@
       <origin rpy="0.0 0.0 0.0" xyz="0.0 0 ${0.149 - 0.03}"/>
       <axis xyz="0 0 1"/>
-      <limit effort="330.0" lower="${-pi*179/180}" upper="${pi*179/180}" velocity="2.16"/>
+      <limit effort="330.0" lower="${-pi*179/180}" upper="${pi*179/180}" velocity="${pi*45/180}"/>
     </joint>
     <link name="${prefix}link_6">
@@ -129,5 +129,5 @@
       <origin rpy="0.0 0.0 0.0" xyz="0.0 0 ${0.14 + 0.03}"/>
       <axis xyz="0 1 0"/>
-      <limit effort="330.0" lower="${-pi*19/36}" upper="${pi*19/36}" velocity="2.16"/>
+      <limit effort="330.0" lower="${-pi*19/36}" upper="${pi*19/36}" velocity="${pi*45/180}"/>
     </joint>
     <link name="${prefix}link_7">
@@ -155,5 +155,5 @@
         <origin rpy="0.0 0.0 0.0" xyz="0.0 0 0.1208"/>
         <axis xyz="0 0 1"/>
-        <limit effort="330.0" velocity="2.16"/>
+        <limit effort="330.0" velocity="${pi*45/180}"/>
       </joint>
     </xacro:if>
@@ -164,5 +164,5 @@
         <origin rpy="0.0 0.0 0.0" xyz="0.0 0 0.1208"/>
         <axis xyz="0 0 1"/>
-        <limit effort="330.0" lower="${-pi*179/180}" upper="${pi*179/180}" velocity="2.16"/>
+        <limit effort="330.0" lower="${-pi*179/180}" upper="${pi*179/180}" velocity="${pi*45/180}"/>
       </joint>
     </xacro:unless>
@@ -190,5 +190,5 @@
       <origin rpy="0.0 0.0 0.0" xyz="0.0 0 0.0012"/>
       <axis xyz="0 0 1"/>
-      <limit effort="330.0" lower="-3.12414" upper="3.12414" velocity="2.16"/>
+      <limit effort="330.0" lower="-3.12414" upper="3.12414" velocity="${pi*45/180}"/>
     </joint>
     <link name="${prefix}flange">

Commit message: Add missing - to offset

File: irc_ros_description/urdf/robots/igus_rebel_4dof_00.description.xacro (robot description, xacro)
@@ -24,5 +24,5 @@
       <origin rpy="0.0 0.0 0.0" xyz="0.0 0.0 0.100"/>
       <axis xyz="0 0 -1"/>
-      <limit effort="330.0" lower="${-pi*179/180}" upper="${pi*179/180}" velocity="${pi*45/180}"/>
+      <limit effort="330.0" lower="${-pi*179/180}" upper="${pi*179/180}" velocity="2.16"/>
     </joint>
     <link name="${prefix}link_1">
@@ -50,5 +50,5 @@
       <axis xyz="0 1 0"/>
       <!-- pi*2/3 are the physical limits, but to avoid any collisions we set the actual limits lower -->
-      <limit effort="330.0" lower="${-pi*11/18}" upper="${pi*11/18}" velocity="${pi*45/180}"/>
+      <limit effort="330.0" lower="${-pi*11/18}" upper="${pi*11/18}" velocity="2.16"/>
     </joint>
     <link name="${prefix}link_2">
@@ -76,5 +76,5 @@
       <axis xyz="0 1 0"/>
       <!-- pi*2/3 are the physical limits, but to avoid any collisions we set the actual limits lower -->
-      <limit effort="330.0" lower="${-pi*11/18}" upper="${pi*11/18}" velocity="${pi*45/180}"/>
+      <limit effort="330.0" lower="${-pi*11/18}" upper="${pi*11/18}" velocity="2.16"/>
     </joint>
     <link name="${prefix}link_3">
@@ -100,7 +100,7 @@
         <parent link="${prefix}link_3"/>
         <child link="${prefix}link_4"/>
-        <origin rpy="0.0 ${pi/24} 0.0" xyz="0.0 0.0 0.2423"/>
+        <origin rpy="0.0 ${-pi/24} 0.0" xyz="0.0 0.0 0.2423"/>
         <axis xyz="0 -1 0"/>
-        <limit effort="330.0" velocity="${pi*45/180}"/>
+        <limit effort="330.0" velocity="2.16"/>
       </joint>
     </xacro:if>
@@ -111,5 +111,5 @@
         <origin rpy="0.0 ${-pi/24} 0.0" xyz="0.0 0.0 0.2423"/>
         <axis xyz="0 -1 0"/>
-        <limit effort="330.0" lower="${-pi*179/180}" upper="${pi*179/180}" velocity="${pi*45/180}"/>
+        <limit effort="330.0" lower="${-pi*179/180}" upper="${pi*179/180}" velocity="2.16"/>
       </joint>
     </xacro:unless>

Commit message: Adjust joint limits to offset, adjust direction and velocity for 4dof

File: irc_ros_description/urdf/robots/igus_rebel_4dof_00.description.xacro (robot description, xacro)
@@ -24,5 +24,5 @@
       <origin rpy="0.0 0.0 0.0" xyz="0.0 0.0 0.100"/>
       <axis xyz="0 0 -1"/>
-      <limit effort="330.0" lower="${-pi*179/180}" upper="${pi*179/180}" velocity="2.16"/>
+      <limit effort="330.0" lower="${-pi*179/180}" upper="${pi*179/180}" velocity="${pi*45/180}"/>
     </joint>
     <link name="${prefix}link_1">
@@ -50,5 +50,5 @@
       <axis xyz="0 1 0"/>
       <!-- pi*2/3 are the physical limits, but to avoid any collisions we set the actual limits lower -->
-      <limit effort="330.0" lower="${-pi*11/18}" upper="${pi*11/18}" velocity="2.16"/>
+      <limit effort="330.0" lower="${-pi*11/18}" upper="${pi*11/18}" velocity="${pi*45/180}"/>
     </joint>
     <link name="${prefix}link_2">
@@ -76,5 +76,5 @@
       <axis xyz="0 1 0"/>
       <!-- pi*2/3 are the physical limits, but to avoid any collisions we set the actual limits lower -->
-      <limit effort="330.0" lower="${-pi*11/18}" upper="${pi*11/18}" velocity="2.16"/>
+      <limit effort="330.0" lower="${-pi*11/18}" upper="${pi*11/18}" velocity="${pi*45/180}"/>
     </joint>
     <link name="${prefix}link_3">
@@ -110,6 +110,6 @@
         <child link="${prefix}link_4"/>
         <origin rpy="0.0 ${-pi/24} 0.0" xyz="0.0 0.0 0.2423"/>
-        <axis xyz="0 -1 0"/>
-        <limit effort="330.0" lower="${-pi*179/180}" upper="${pi*179/180}" velocity="2.16"/>
+        <axis xyz="0 1 0"/>
+      <limit effort="330.0" lower="${-pi*19/36 + pi/24}" upper="${pi*19/36 + pi/24}" velocity="${pi*45/180}"/>
       </joint>
     </xacro:unless>

File: irc_ros_description/urdf/robots/igus_rebel_6dof_00.description.xacro (robot description, xacro)
@@ -128,5 +128,5 @@
       <origin rpy="0.0 ${-pi/24} 0.0" xyz="0.0 0 ${0.14 + 0.03}"/>
       <axis xyz="0 1 0"/>
-      <limit effort="330.0" lower="${-pi*19/36}" upper="${pi*19/36}" velocity="${pi*45/180}"/>
+      <limit effort="330.0" lower="${-pi*19/36 + pi/24}" upper="${pi*19/36 + pi/24}" velocity="${pi*45/180}"/>
     </joint>
     <link name="${prefix}link_7">
