Commit message: Fix joint offsets and limits (#99)
* Remove rotational offset for rebel on platform

* Lower joint limits on axis 2 and 3 from 120 to 110 degrees

* Fix joint4 (4dof)/joint 5 (6dof) offsets and offset the joint limits

* Change velocities in urdf descriptions to match new defaults

* Fix joint direction for 4dof

File: irc_ros_description/urdf/robots/igus_rebel_4dof_00.description.xacro (robot description, xacro)
@@ -24,5 +24,5 @@
       <origin rpy="0.0 0.0 0.0" xyz="0.0 0.0 0.100"/>
       <axis xyz="0 0 -1"/>
-      <limit effort="330.0" lower="${-pi*179/180}" upper="${pi*179/180}" velocity="2.16"/>
+      <limit effort="330.0" lower="${-pi*179/180}" upper="${pi*179/180}" velocity="${pi*45/180}"/>
     </joint>
     <link name="${prefix}link_1">
@@ -49,5 +49,6 @@
       <origin rpy="0.0 ${pi/6} 0.0" xyz="0.0 0 0.149"/>
       <axis xyz="0 1 0"/>
-      <limit effort="330.0" lower="${-pi*2/3}" upper="${pi*2/3}" velocity="2.16"/>
+      <!-- pi*2/3 are the physical limits, but to avoid any collisions we set the actual limits lower -->
+      <limit effort="330.0" lower="${-pi*11/18}" upper="${pi*11/18}" velocity="${pi*45/180}"/>
     </joint>
     <link name="${prefix}link_2">
@@ -74,5 +75,6 @@
       <origin rpy="0.0 ${pi/6} 0.0" xyz="0.0 0.0 0.2384"/>
       <axis xyz="0 1 0"/>
-      <limit effort="330.0" lower="${-pi*2/3}" upper="${pi*2/3}" velocity="2.16"/>
+      <!-- pi*2/3 are the physical limits, but to avoid any collisions we set the actual limits lower -->
+      <limit effort="330.0" lower="${-pi*11/18}" upper="${pi*11/18}" velocity="${pi*45/180}"/>
     </joint>
     <link name="${prefix}link_3">
@@ -98,5 +100,5 @@
         <parent link="${prefix}link_3"/>
         <child link="${prefix}link_4"/>
-        <origin rpy="0.0 0.0 0.0" xyz="0.0 0.0 0.2423"/>
+        <origin rpy="0.0 ${-pi/24} 0.0" xyz="0.0 0.0 0.2423"/>
         <axis xyz="0 -1 0"/>
         <limit effort="330.0" velocity="2.16"/>
@@ -107,7 +109,7 @@
         <parent link="${prefix}link_3"/>
         <child link="${prefix}link_4"/>
-        <origin rpy="0.0 0.0 0.0" xyz="0.0 0.0 0.2423"/>
-        <axis xyz="0 -1 0"/>
-        <limit effort="330.0" lower="${-pi*179/180}" upper="${pi*179/180}" velocity="2.16"/>
+        <origin rpy="0.0 ${-pi/24} 0.0" xyz="0.0 0.0 0.2423"/>
+        <axis xyz="0 1 0"/>
+      <limit effort="330.0" lower="${-pi*19/36 + pi/24}" upper="${pi*19/36 + pi/24}" velocity="${pi*45/180}"/>
       </joint>
     </xacro:unless>

File: irc_ros_description/urdf/robots/igus_rebel_6dof_00.description.xacro (robot description, xacro)
@@ -24,5 +24,5 @@
       <origin rpy="0.0 0.0 0.0" xyz="0.0 0 0.100"/>
       <axis xyz="0 0 -1"/>
-      <limit effort="330.0" lower="${-pi*179/180}" upper="${pi*179/180}" velocity="2.16"/>
+      <limit effort="330.0" lower="${-pi*179/180}" upper="${pi*179/180}" velocity="${pi*45/180}"/>
     </joint>
     <link name="${prefix}link_1">
@@ -49,5 +49,6 @@
       <origin rpy="0.0 ${pi/6} 0.0" xyz="0.0 0 0.149"/>
       <axis xyz="0 1 0"/>
-      <limit effort="330.0" lower="${-pi*2/3}" upper="${pi*2/3}" velocity="2.16"/>
+      <!-- pi*2/3 are the physical limits, but to avoid any collisions we set the actual limits lower -->
+      <limit effort="330.0" lower="${-pi*11/18}" upper="${pi*11/18}" velocity="${pi*45/180}"/>
     </joint>
     <link name="${prefix}link_2">
@@ -74,5 +75,6 @@
       <origin rpy="0.0 ${pi/6} 0.0" xyz="0.0 0.0 0.2384"/>
       <axis xyz="0 1 0"/>
-      <limit effort="330.0" lower="${-pi*2/3}" upper="${pi*2/3}" velocity="2.16"/>
+      <!-- pi*2/3 are the physical limits, but to avoid any collisions we set the actual limits lower -->
+      <limit effort="330.0" lower="${-pi*11/18}" upper="${pi*11/18}" velocity="${pi*45/180}"/>
     </joint>
     <link name="${prefix}link_5">
@@ -100,5 +102,5 @@
       <origin rpy="0.0 0.0 0.0" xyz="0.0 0 ${0.149 - 0.03}"/>
       <axis xyz="0 0 1"/>
-      <limit effort="330.0" lower="${-pi*179/180}" upper="${pi*179/180}" velocity="2.16"/>
+      <limit effort="330.0" lower="${-pi*179/180}" upper="${pi*179/180}" velocity="${pi*45/180}"/>
     </joint>
     <link name="${prefix}link_6">
@@ -124,7 +126,7 @@
       <child link="${prefix}link_7"/>
       <!-- TODO The 0.03m offset are most likely caused by the mesh file (Issue 15) -->
-      <origin rpy="0.0 0.0 0.0" xyz="0.0 0 ${0.14 + 0.03}"/>
+      <origin rpy="0.0 ${-pi/24} 0.0" xyz="0.0 0 ${0.14 + 0.03}"/>
       <axis xyz="0 1 0"/>
-      <limit effort="330.0" lower="${-pi*19/36}" upper="${pi*19/36}" velocity="2.16"/>
+      <limit effort="330.0" lower="${-pi*19/36 + pi/24}" upper="${pi*19/36 + pi/24}" velocity="${pi*45/180}"/>
     </joint>
     <link name="${prefix}link_7">
@@ -152,5 +154,5 @@
         <origin rpy="0.0 0.0 0.0" xyz="0.0 0 0.1208"/>
         <axis xyz="0 0 1"/>
-        <limit effort="330.0" velocity="2.16"/>
+        <limit effort="330.0" velocity="${pi*45/180}"/>
       </joint>
     </xacro:if>
@@ -161,5 +163,5 @@
         <origin rpy="0.0 0.0 0.0" xyz="0.0 0 0.1208"/>
         <axis xyz="0 0 1"/>
-        <limit effort="330.0" lower="${-pi*179/180}" upper="${pi*179/180}" velocity="2.16"/>
+        <limit effort="330.0" lower="${-pi*179/180}" upper="${pi*179/180}" velocity="${pi*45/180}"/>
       </joint>
     </xacro:unless>
@@ -187,5 +189,5 @@
       <origin rpy="0.0 0.0 0.0" xyz="0.0 0 0.0012"/>
       <axis xyz="0 0 1"/>
-      <limit effort="330.0" lower="-3.12414" upper="3.12414" velocity="2.16"/>
+      <limit effort="330.0" lower="-3.12414" upper="3.12414" velocity="${pi*45/180}"/>
     </joint>
     <link name="${prefix}flange">

File: irc_ros_description/urdf/robots/igus_rebel_6dof_pre.description.xacro (robot description, xacro)
@@ -24,5 +24,5 @@
       <origin rpy="0.0 0.0 0.0" xyz="0.0 0 0.144"/>
       <axis xyz="0 0 -1"/>
-      <limit effort="330.0" lower="${-pi*179/180}" upper="${pi*179/180}" velocity="2.16"/>
+      <limit effort="330.0" lower="${-pi*179/180}" upper="${pi*179/180}" velocity="${pi*45/180}"/>
     </joint>
     <link name="${prefix}link_1">
@@ -49,5 +49,6 @@
       <origin rpy="0.0 0.0 0.0" xyz="0.0 0 0.130"/>
       <axis xyz="0 1 0"/>
-      <limit effort="330.0" lower="${-pi*2/3 + pi/6}" upper="${pi*2/3 + pi/6}" velocity="2.16"/>
+      <!-- pi*2/3 are the physical limits, but to avoid any collisions we set the actual limits lower -->
+      <limit effort="330.0" lower="${-pi*11/18 + pi/6}" upper="${pi*11/18 + pi/6}" velocity="${pi*45/180}"/>
     </joint>
     <link name="${prefix}link_2">
@@ -74,5 +75,6 @@
       <origin rpy="0.0 0.0 0.0" xyz="0.0 0.0 0.2384"/>
       <axis xyz="0 1 0"/>
-      <limit effort="330.0" lower="${-pi*2/3 + pi/6}" upper="${pi*2/3 + pi/6}" velocity="2.16"/>
+      <!-- pi*2/3 are the physical limits, but to avoid any collisions we set the actual limits lower -->
+      <limit effort="330.0" lower="${-pi*11/18 + pi/6}" upper="${pi*11/18 + pi/6}" velocity="${pi*45/180}"/>
     </joint>
     <link name="${prefix}link_5">
@@ -98,7 +100,8 @@
       <child link="${prefix}link_6"/>
       <!-- TODO The 0.03m offset are most likely caused by the mesh file (Issue 15) -->
+      <!-- The irc config file specifies a rotational offset of 65 degrees, if someone has access to a pre version please verify if that is correct -->
       <origin rpy="0.0 0.0 0.0" xyz="0.0 0 ${0.149 - 0.03}"/>
       <axis xyz="0 0 1"/>
-      <limit effort="330.0" lower="${-pi*179/180}" upper="${pi*179/180}" velocity="2.16"/>
+      <limit effort="330.0" lower="${-pi*179/180}" upper="${pi*179/180}" velocity="${pi*45/180}"/>
     </joint>
     <link name="${prefix}link_6">
@@ -126,5 +129,5 @@
       <origin rpy="0.0 0.0 0.0" xyz="0.0 0 ${0.14 + 0.03}"/>
       <axis xyz="0 1 0"/>
-      <limit effort="330.0" lower="${-pi*19/36}" upper="${pi*19/36}" velocity="2.16"/>
+      <limit effort="330.0" lower="${-pi*19/36}" upper="${pi*19/36}" velocity="${pi*45/180}"/>
     </joint>
     <link name="${prefix}link_7">
@@ -152,5 +155,5 @@
         <origin rpy="0.0 0.0 0.0" xyz="0.0 0 0.1208"/>
         <axis xyz="0 0 1"/>
-        <limit effort="330.0" velocity="2.16"/>
+        <limit effort="330.0" velocity="${pi*45/180}"/>
       </joint>
     </xacro:if>
@@ -161,5 +164,5 @@
         <origin rpy="0.0 0.0 0.0" xyz="0.0 0 0.1208"/>
         <axis xyz="0 0 1"/>
-        <limit effort="330.0" lower="${-pi*179/180}" upper="${pi*179/180}" velocity="2.16"/>
+        <limit effort="330.0" lower="${-pi*179/180}" upper="${pi*179/180}" velocity="${pi*45/180}"/>
       </joint>
     </xacro:unless>
@@ -187,5 +190,5 @@
       <origin rpy="0.0 0.0 0.0" xyz="0.0 0 0.0012"/>
       <axis xyz="0 0 1"/>
-      <limit effort="330.0" lower="-3.12414" upper="3.12414" velocity="2.16"/>
+      <limit effort="330.0" lower="-3.12414" upper="3.12414" velocity="${pi*45/180}"/>
     </joint>
     <link name="${prefix}flange">
