Commit message: Add cri offset parameter to rebel axis and set them

File: irc_ros_description/urdf/modules/rebel.ros2_control.xacro (robot description, xacro)
@@ -1,5 +1,5 @@
 <?xml version="1.0"?>
 <robot xmlns:xacro="http://www.ros.org/wiki/xacro">
-  <xacro:macro name="rebel_joint" params="name can_id position_min=0 position_max=0 gear_scale=1 continuous_joint=false">
+  <xacro:macro name="rebel_joint" params="name can_id position_min=0 position_max=0 gear_scale=1 continuous_joint=false cri_position_offset=0">
     <joint name="${name}">
       <command_interface name="position">
@@ -21,7 +21,10 @@
         <param name="initial_value">0.0</param>
       </state_interface>
+      <!-- CPRCAN specific parameters -->
       <param name="can_id">${can_id}</param>
       <param name="gear_scale">${gear_scale}</param>
       <param name="controller_type">closed_loop</param>
+      <!-- CRI specific parameters -->
+      <param name="cri_position_offset">${cri_position_offset}</param>
     </joint>
   </xacro:macro>

File: irc_ros_description/urdf/robots/igus_rebel_4dof_00.ros2_control.xacro (robot description, xacro)
@@ -23,7 +23,7 @@
       <xacro:rebel_joint name="${prefix}joint1" can_id="0x10" position_min="${-pi*179/180}" position_max="${pi*179/180}" gear_scale="-1031.11" />
       <!-- Position limit difference with iRC files due to 30 degree offset in joint 2 and 3 -->
-      <xacro:rebel_joint name="${prefix}joint2" can_id="0x20" position_min="${-pi*2/3}" position_max="${pi*2/3}" gear_scale="1031.11" />
-      <xacro:rebel_joint name="${prefix}joint3" can_id="0x30" position_min="${-pi*2/3}" position_max="${pi*2/3}" gear_scale="1031.11" />
-      <xacro:rebel_joint name="${prefix}joint4" can_id="0x40" position_min="${-pi*19/36}" position_max="${pi*19/36}" gear_scale="1031.11" continuous_joint="${continuous_last_joint}" />
+      <xacro:rebel_joint name="${prefix}joint2" can_id="0x20" position_min="${-pi*2/3}" position_max="${pi*2/3}" gear_scale="1031.11" cri_position_offset="-30" />
+      <xacro:rebel_joint name="${prefix}joint3" can_id="0x30" position_min="${-pi*2/3}" position_max="${pi*2/3}" gear_scale="1031.11" cri_position_offset="-30" />
+      <xacro:rebel_joint name="${prefix}joint4" can_id="0x40" position_min="${-pi*19/36}" position_max="${pi*19/36}" gear_scale="1031.11" continuous_joint="${continuous_last_joint}" cri_position_offset="7.5" />
       <gpio name="${prefix}dio_base">
         <param name="can_id">0x70</param>

File: irc_ros_description/urdf/robots/igus_rebel_4dof_01.ros2_control.xacro (robot description, xacro)
@@ -22,7 +22,7 @@
       <xacro:include filename="$(find irc_ros_description)/urdf/modules/rebel.ros2_control.xacro" />
       <xacro:rebel_joint name="${prefix}joint1" can_id="0x10" position_min="${-pi*179/180}" position_max="${pi*179/180}" gear_scale="-1443.55" />
-      <xacro:rebel_joint name="${prefix}joint2" can_id="0x20" position_min="${-pi*2/3}" position_max="${pi*2/3}" gear_scale="1443.55" />
-      <xacro:rebel_joint name="${prefix}joint3" can_id="0x30" position_min="${-pi*2/3}" position_max="${pi*2/3}" gear_scale="1443.55" />
-      <xacro:rebel_joint name="${prefix}joint4" can_id="0x40" position_min="${-pi*19/36}" position_max="${pi*19/36}" gear_scale="1031.11" continuous_joint="${continuous_last_joint}" />
+      <xacro:rebel_joint name="${prefix}joint2" can_id="0x20" position_min="${-pi*2/3}" position_max="${pi*2/3}" gear_scale="1443.55" cri_position_offset="-30" />
+      <xacro:rebel_joint name="${prefix}joint3" can_id="0x30" position_min="${-pi*2/3}" position_max="${pi*2/3}" gear_scale="1443.55" cri_position_offset="-30" />
+      <xacro:rebel_joint name="${prefix}joint4" can_id="0x40" position_min="${-pi*19/36}" position_max="${pi*19/36}" gear_scale="1031.11" continuous_joint="${continuous_last_joint}" cri_position_offset="7.5" />
       <gpio name="${prefix}dio_base">
         <param name="can_id">0x70</param>

File: irc_ros_description/urdf/robots/igus_rebel_6dof_00.ros2_control.xacro (robot description, xacro)
@@ -23,8 +23,8 @@
       <xacro:rebel_joint name="${prefix}joint1" can_id="0x10" position_min="${-pi*179/180}" position_max="${pi*179/180}" gear_scale="1031.11" />
       <!-- Position limit difference with iRC files due to 30 degree offset in joint 2 and 3 -->
-      <xacro:rebel_joint name="${prefix}joint2" can_id="0x20" position_min="${-pi*2/3}" position_max="${pi*2/3}" gear_scale="1031.11" />
-      <xacro:rebel_joint name="${prefix}joint3" can_id="0x30" position_min="${-pi*2/3}" position_max="${pi*2/3}" gear_scale="1031.11" />
+      <xacro:rebel_joint name="${prefix}joint2" can_id="0x20" position_min="${-pi*2/3}" position_max="${pi*2/3}" gear_scale="1031.11" cri_position_offset="-30" />
+      <xacro:rebel_joint name="${prefix}joint3" can_id="0x30" position_min="${-pi*2/3}" position_max="${pi*2/3}" gear_scale="1031.11" cri_position_offset="-30" />
       <xacro:rebel_joint name="${prefix}joint4" can_id="0x40" position_min="${-pi*179/180}" position_max="${pi*179/180}" gear_scale="-1031.11" />
-      <xacro:rebel_joint name="${prefix}joint5" can_id="0x50" position_min="${-pi*19/36}" position_max="${pi*19/36}" gear_scale="1031.11" />
+      <xacro:rebel_joint name="${prefix}joint5" can_id="0x50" position_min="${-pi*19/36}" position_max="${pi*19/36}" gear_scale="1031.11" cri_position_offset="7.5" />
       <xacro:rebel_joint name="${prefix}joint6" can_id="0x60" position_min="${-pi*179/180}" position_max="${pi*179/180}" gear_scale="-1031.11" continuous_joint="${continuous_last_joint}" />
       <gpio name="${prefix}dio_base">

File: irc_ros_description/urdf/robots/igus_rebel_6dof_01.ros2_control.xacro (robot description, xacro)
@@ -23,8 +23,8 @@
       <xacro:rebel_joint name="${prefix}joint1" can_id="0x10" position_min="${-pi*179/180}" position_max="${pi*179/180}" gear_scale="1443.55" />
       <!-- Position limit difference with iRC files due to 30 degree offset in joint 2 and 3 -->
-      <xacro:rebel_joint name="${prefix}joint2" can_id="0x20" position_min="${-pi*2/3}" position_max="${pi*2/3}" gear_scale="1443.55" />
-      <xacro:rebel_joint name="${prefix}joint3" can_id="0x30" position_min="${-pi*2/3}" position_max="${pi*2/3}" gear_scale="1443.55" />
+      <xacro:rebel_joint name="${prefix}joint2" can_id="0x20" position_min="${-pi*2/3}" position_max="${pi*2/3}" gear_scale="1443.55" cri_position_offset="-30" />
+      <xacro:rebel_joint name="${prefix}joint3" can_id="0x30" position_min="${-pi*2/3}" position_max="${pi*2/3}" gear_scale="1443.55" cri_position_offset="-30" />
       <xacro:rebel_joint name="${prefix}joint4" can_id="0x40" position_min="${-pi*179/180}" position_max="${pi*179/180}" gear_scale="-1443.55" />
-      <xacro:rebel_joint name="${prefix}joint5" can_id="0x50" position_min="${-pi*19/36}" position_max="${pi*19/36}" gear_scale="1031.11" />
+      <xacro:rebel_joint name="${prefix}joint5" can_id="0x50" position_min="${-pi*19/36}" position_max="${pi*19/36}" gear_scale="1031.11" cri_position_offset="7.5" />
       <xacro:rebel_joint name="${prefix}joint6" can_id="0x60" position_min="${-pi*179/180}" position_max="${pi*179/180}" gear_scale="-1031.11" continuous_joint="${continuous_last_joint}" />
       <gpio name="${prefix}dio_base">

Commit message: Rename offset parameter

File: irc_ros_description/urdf/modules/rebel.ros2_control.xacro (robot description, xacro)
@@ -1,5 +1,5 @@
 <?xml version="1.0"?>
 <robot xmlns:xacro="http://www.ros.org/wiki/xacro">
-  <xacro:macro name="rebel_joint" params="name can_id position_min=0 position_max=0 gear_scale=1 continuous_joint=false cri_position_offset=0">
+  <xacro:macro name="rebel_joint" params="name can_id position_min=0 position_max=0 gear_scale=1 continuous_joint=false cri_joint_offset=0">
     <joint name="${name}">
       <command_interface name="position">
@@ -26,5 +26,5 @@
       <param name="controller_type">closed_loop</param>
       <!-- CRI specific parameters -->
-      <param name="cri_position_offset">${cri_position_offset}</param>
+      <param name="cri_joint_offset">${cri_joint_offset}</param>
     </joint>
   </xacro:macro>

File: irc_ros_description/urdf/robots/igus_rebel_4dof_00.ros2_control.xacro (robot description, xacro)
@@ -23,7 +23,7 @@
       <xacro:rebel_joint name="${prefix}joint1" can_id="0x10" position_min="${-pi*179/180}" position_max="${pi*179/180}" gear_scale="-1031.11" />
       <!-- Position limit difference with iRC files due to 30 degree offset in joint 2 and 3 -->
-      <xacro:rebel_joint name="${prefix}joint2" can_id="0x20" position_min="${-pi*2/3}" position_max="${pi*2/3}" gear_scale="1031.11" cri_position_offset="-30" />
-      <xacro:rebel_joint name="${prefix}joint3" can_id="0x30" position_min="${-pi*2/3}" position_max="${pi*2/3}" gear_scale="1031.11" cri_position_offset="-30" />
-      <xacro:rebel_joint name="${prefix}joint4" can_id="0x40" position_min="${-pi*19/36}" position_max="${pi*19/36}" gear_scale="1031.11" continuous_joint="${continuous_last_joint}" cri_position_offset="7.5" />
+      <xacro:rebel_joint name="${prefix}joint2" can_id="0x20" position_min="${-pi*2/3}" position_max="${pi*2/3}" gear_scale="1031.11" cri_joint_offset="-30" />
+      <xacro:rebel_joint name="${prefix}joint3" can_id="0x30" position_min="${-pi*2/3}" position_max="${pi*2/3}" gear_scale="1031.11" cri_joint_offset="-30" />
+      <xacro:rebel_joint name="${prefix}joint4" can_id="0x40" position_min="${-pi*19/36}" position_max="${pi*19/36}" gear_scale="1031.11" continuous_joint="${continuous_last_joint}" cri_joint_offset="7.5" />
       <gpio name="${prefix}dio_base">
         <param name="can_id">0x70</param>

File: irc_ros_description/urdf/robots/igus_rebel_4dof_01.ros2_control.xacro (robot description, xacro)
@@ -22,7 +22,7 @@
       <xacro:include filename="$(find irc_ros_description)/urdf/modules/rebel.ros2_control.xacro" />
       <xacro:rebel_joint name="${prefix}joint1" can_id="0x10" position_min="${-pi*179/180}" position_max="${pi*179/180}" gear_scale="-1443.55" />
-      <xacro:rebel_joint name="${prefix}joint2" can_id="0x20" position_min="${-pi*2/3}" position_max="${pi*2/3}" gear_scale="1443.55" cri_position_offset="-30" />
-      <xacro:rebel_joint name="${prefix}joint3" can_id="0x30" position_min="${-pi*2/3}" position_max="${pi*2/3}" gear_scale="1443.55" cri_position_offset="-30" />
-      <xacro:rebel_joint name="${prefix}joint4" can_id="0x40" position_min="${-pi*19/36}" position_max="${pi*19/36}" gear_scale="1031.11" continuous_joint="${continuous_last_joint}" cri_position_offset="7.5" />
+      <xacro:rebel_joint name="${prefix}joint2" can_id="0x20" position_min="${-pi*2/3}" position_max="${pi*2/3}" gear_scale="1443.55" cri_joint_offset="-30" />
+      <xacro:rebel_joint name="${prefix}joint3" can_id="0x30" position_min="${-pi*2/3}" position_max="${pi*2/3}" gear_scale="1443.55" cri_joint_offset="-30" />
+      <xacro:rebel_joint name="${prefix}joint4" can_id="0x40" position_min="${-pi*19/36}" position_max="${pi*19/36}" gear_scale="1031.11" continuous_joint="${continuous_last_joint}" cri_joint_offset="7.5" />
       <gpio name="${prefix}dio_base">
         <param name="can_id">0x70</param>

File: irc_ros_description/urdf/robots/igus_rebel_6dof_00.ros2_control.xacro (robot description, xacro)
@@ -23,8 +23,8 @@
       <xacro:rebel_joint name="${prefix}joint1" can_id="0x10" position_min="${-pi*179/180}" position_max="${pi*179/180}" gear_scale="1031.11" />
       <!-- Position limit difference with iRC files due to 30 degree offset in joint 2 and 3 -->
-      <xacro:rebel_joint name="${prefix}joint2" can_id="0x20" position_min="${-pi*2/3}" position_max="${pi*2/3}" gear_scale="1031.11" cri_position_offset="-30" />
-      <xacro:rebel_joint name="${prefix}joint3" can_id="0x30" position_min="${-pi*2/3}" position_max="${pi*2/3}" gear_scale="1031.11" cri_position_offset="-30" />
+      <xacro:rebel_joint name="${prefix}joint2" can_id="0x20" position_min="${-pi*2/3}" position_max="${pi*2/3}" gear_scale="1031.11" cri_joint_offset="-30" />
+      <xacro:rebel_joint name="${prefix}joint3" can_id="0x30" position_min="${-pi*2/3}" position_max="${pi*2/3}" gear_scale="1031.11" cri_joint_offset="-30" />
       <xacro:rebel_joint name="${prefix}joint4" can_id="0x40" position_min="${-pi*179/180}" position_max="${pi*179/180}" gear_scale="-1031.11" />
-      <xacro:rebel_joint name="${prefix}joint5" can_id="0x50" position_min="${-pi*19/36}" position_max="${pi*19/36}" gear_scale="1031.11" cri_position_offset="7.5" />
+      <xacro:rebel_joint name="${prefix}joint5" can_id="0x50" position_min="${-pi*19/36}" position_max="${pi*19/36}" gear_scale="1031.11" cri_joint_offset="7.5" />
       <xacro:rebel_joint name="${prefix}joint6" can_id="0x60" position_min="${-pi*179/180}" position_max="${pi*179/180}" gear_scale="-1031.11" continuous_joint="${continuous_last_joint}" />
       <gpio name="${prefix}dio_base">

File: irc_ros_description/urdf/robots/igus_rebel_6dof_01.ros2_control.xacro (robot description, xacro)
@@ -23,8 +23,8 @@
       <xacro:rebel_joint name="${prefix}joint1" can_id="0x10" position_min="${-pi*179/180}" position_max="${pi*179/180}" gear_scale="1443.55" />
       <!-- Position limit difference with iRC files due to 30 degree offset in joint 2 and 3 -->
-      <xacro:rebel_joint name="${prefix}joint2" can_id="0x20" position_min="${-pi*2/3}" position_max="${pi*2/3}" gear_scale="1443.55" cri_position_offset="-30" />
-      <xacro:rebel_joint name="${prefix}joint3" can_id="0x30" position_min="${-pi*2/3}" position_max="${pi*2/3}" gear_scale="1443.55" cri_position_offset="-30" />
+      <xacro:rebel_joint name="${prefix}joint2" can_id="0x20" position_min="${-pi*2/3}" position_max="${pi*2/3}" gear_scale="1443.55" cri_joint_offset="-30" />
+      <xacro:rebel_joint name="${prefix}joint3" can_id="0x30" position_min="${-pi*2/3}" position_max="${pi*2/3}" gear_scale="1443.55" cri_joint_offset="-30" />
       <xacro:rebel_joint name="${prefix}joint4" can_id="0x40" position_min="${-pi*179/180}" position_max="${pi*179/180}" gear_scale="-1443.55" />
-      <xacro:rebel_joint name="${prefix}joint5" can_id="0x50" position_min="${-pi*19/36}" position_max="${pi*19/36}" gear_scale="1031.11" cri_position_offset="7.5" />
+      <xacro:rebel_joint name="${prefix}joint5" can_id="0x50" position_min="${-pi*19/36}" position_max="${pi*19/36}" gear_scale="1031.11" cri_joint_offset="7.5" />
       <xacro:rebel_joint name="${prefix}joint6" can_id="0x60" position_min="${-pi*179/180}" position_max="${pi*179/180}" gear_scale="-1031.11" continuous_joint="${continuous_last_joint}" />
       <gpio name="${prefix}dio_base">

Commit message: Fix CRI joint missalignments (#82)
* Add cri offset parameter to rebel axis and set them

* Add mock gpios

* Stop command output spam

File: irc_ros_description/urdf/modules/rebel.ros2_control.xacro (robot description, xacro)
@@ -1,5 +1,5 @@
 <?xml version="1.0"?>
 <robot xmlns:xacro="http://www.ros.org/wiki/xacro">
-  <xacro:macro name="rebel_joint" params="name can_id position_min=0 position_max=0 gear_scale=1 continuous_joint=false">
+  <xacro:macro name="rebel_joint" params="name can_id position_min=0 position_max=0 gear_scale=1 continuous_joint=false cri_joint_offset=0">
     <joint name="${name}">
       <command_interface name="position">
@@ -21,7 +21,10 @@
         <param name="initial_value">0.0</param>
       </state_interface>
+      <!-- CPRCAN specific parameters -->
       <param name="can_id">${can_id}</param>
       <param name="gear_scale">${gear_scale}</param>
       <param name="controller_type">closed_loop</param>
+      <!-- CRI specific parameters -->
+      <param name="cri_joint_offset">${cri_joint_offset}</param>
     </joint>
   </xacro:macro>

File: irc_ros_description/urdf/robots/igus_rebel_4dof_00.ros2_control.xacro (robot description, xacro)
@@ -23,7 +23,7 @@
       <xacro:rebel_joint name="${prefix}joint1" can_id="0x10" position_min="${-pi*179/180}" position_max="${pi*179/180}" gear_scale="-1031.11" />
       <!-- Position limit difference with iRC files due to 30 degree offset in joint 2 and 3 -->
-      <xacro:rebel_joint name="${prefix}joint2" can_id="0x20" position_min="${-pi*2/3}" position_max="${pi*2/3}" gear_scale="1031.11" />
-      <xacro:rebel_joint name="${prefix}joint3" can_id="0x30" position_min="${-pi*2/3}" position_max="${pi*2/3}" gear_scale="1031.11" />
-      <xacro:rebel_joint name="${prefix}joint4" can_id="0x40" position_min="${-pi*19/36}" position_max="${pi*19/36}" gear_scale="1031.11" continuous_joint="${continuous_last_joint}" />
+      <xacro:rebel_joint name="${prefix}joint2" can_id="0x20" position_min="${-pi*2/3}" position_max="${pi*2/3}" gear_scale="1031.11" cri_joint_offset="-30" />
+      <xacro:rebel_joint name="${prefix}joint3" can_id="0x30" position_min="${-pi*2/3}" position_max="${pi*2/3}" gear_scale="1031.11" cri_joint_offset="-30" />
+      <xacro:rebel_joint name="${prefix}joint4" can_id="0x40" position_min="${-pi*19/36}" position_max="${pi*19/36}" gear_scale="1031.11" continuous_joint="${continuous_last_joint}" cri_joint_offset="7.5" />
       <gpio name="${prefix}dio_base">
         <param name="can_id">0x70</param>

File: irc_ros_description/urdf/robots/igus_rebel_4dof_01.ros2_control.xacro (robot description, xacro)
@@ -22,7 +22,7 @@
       <xacro:include filename="$(find irc_ros_description)/urdf/modules/rebel.ros2_control.xacro" />
       <xacro:rebel_joint name="${prefix}joint1" can_id="0x10" position_min="${-pi*179/180}" position_max="${pi*179/180}" gear_scale="-1443.55" />
-      <xacro:rebel_joint name="${prefix}joint2" can_id="0x20" position_min="${-pi*2/3}" position_max="${pi*2/3}" gear_scale="1443.55" />
-      <xacro:rebel_joint name="${prefix}joint3" can_id="0x30" position_min="${-pi*2/3}" position_max="${pi*2/3}" gear_scale="1443.55" />
-      <xacro:rebel_joint name="${prefix}joint4" can_id="0x40" position_min="${-pi*19/36}" position_max="${pi*19/36}" gear_scale="1031.11" continuous_joint="${continuous_last_joint}" />
+      <xacro:rebel_joint name="${prefix}joint2" can_id="0x20" position_min="${-pi*2/3}" position_max="${pi*2/3}" gear_scale="1443.55" cri_joint_offset="-30" />
+      <xacro:rebel_joint name="${prefix}joint3" can_id="0x30" position_min="${-pi*2/3}" position_max="${pi*2/3}" gear_scale="1443.55" cri_joint_offset="-30" />
+      <xacro:rebel_joint name="${prefix}joint4" can_id="0x40" position_min="${-pi*19/36}" position_max="${pi*19/36}" gear_scale="1031.11" continuous_joint="${continuous_last_joint}" cri_joint_offset="7.5" />
       <gpio name="${prefix}dio_base">
         <param name="can_id">0x70</param>

File: irc_ros_description/urdf/robots/igus_rebel_6dof_00.ros2_control.xacro (robot description, xacro)
@@ -23,8 +23,8 @@
       <xacro:rebel_joint name="${prefix}joint1" can_id="0x10" position_min="${-pi*179/180}" position_max="${pi*179/180}" gear_scale="1031.11" />
       <!-- Position limit difference with iRC files due to 30 degree offset in joint 2 and 3 -->
-      <xacro:rebel_joint name="${prefix}joint2" can_id="0x20" position_min="${-pi*2/3}" position_max="${pi*2/3}" gear_scale="1031.11" />
-      <xacro:rebel_joint name="${prefix}joint3" can_id="0x30" position_min="${-pi*2/3}" position_max="${pi*2/3}" gear_scale="1031.11" />
+      <xacro:rebel_joint name="${prefix}joint2" can_id="0x20" position_min="${-pi*2/3}" position_max="${pi*2/3}" gear_scale="1031.11" cri_joint_offset="-30" />
+      <xacro:rebel_joint name="${prefix}joint3" can_id="0x30" position_min="${-pi*2/3}" position_max="${pi*2/3}" gear_scale="1031.11" cri_joint_offset="-30" />
       <xacro:rebel_joint name="${prefix}joint4" can_id="0x40" position_min="${-pi*179/180}" position_max="${pi*179/180}" gear_scale="-1031.11" />
-      <xacro:rebel_joint name="${prefix}joint5" can_id="0x50" position_min="${-pi*19/36}" position_max="${pi*19/36}" gear_scale="1031.11" />
+      <xacro:rebel_joint name="${prefix}joint5" can_id="0x50" position_min="${-pi*19/36}" position_max="${pi*19/36}" gear_scale="1031.11" cri_joint_offset="7.5" />
       <xacro:rebel_joint name="${prefix}joint6" can_id="0x60" position_min="${-pi*179/180}" position_max="${pi*179/180}" gear_scale="-1031.11" continuous_joint="${continuous_last_joint}" />
       <gpio name="${prefix}dio_base">

File: irc_ros_description/urdf/robots/igus_rebel_6dof_01.ros2_control.xacro (robot description, xacro)
@@ -23,8 +23,8 @@
       <xacro:rebel_joint name="${prefix}joint1" can_id="0x10" position_min="${-pi*179/180}" position_max="${pi*179/180}" gear_scale="1443.55" />
       <!-- Position limit difference with iRC files due to 30 degree offset in joint 2 and 3 -->
-      <xacro:rebel_joint name="${prefix}joint2" can_id="0x20" position_min="${-pi*2/3}" position_max="${pi*2/3}" gear_scale="1443.55" />
-      <xacro:rebel_joint name="${prefix}joint3" can_id="0x30" position_min="${-pi*2/3}" position_max="${pi*2/3}" gear_scale="1443.55" />
+      <xacro:rebel_joint name="${prefix}joint2" can_id="0x20" position_min="${-pi*2/3}" position_max="${pi*2/3}" gear_scale="1443.55" cri_joint_offset="-30" />
+      <xacro:rebel_joint name="${prefix}joint3" can_id="0x30" position_min="${-pi*2/3}" position_max="${pi*2/3}" gear_scale="1443.55" cri_joint_offset="-30" />
       <xacro:rebel_joint name="${prefix}joint4" can_id="0x40" position_min="${-pi*179/180}" position_max="${pi*179/180}" gear_scale="-1443.55" />
-      <xacro:rebel_joint name="${prefix}joint5" can_id="0x50" position_min="${-pi*19/36}" position_max="${pi*19/36}" gear_scale="1031.11" />
+      <xacro:rebel_joint name="${prefix}joint5" can_id="0x50" position_min="${-pi*19/36}" position_max="${pi*19/36}" gear_scale="1031.11" cri_joint_offset="7.5" />
       <xacro:rebel_joint name="${prefix}joint6" can_id="0x60" position_min="${-pi*179/180}" position_max="${pi*179/180}" gear_scale="-1031.11" continuous_joint="${continuous_last_joint}" />
       <gpio name="${prefix}dio_base">
